File: Mosfet pre-regulator/Eagle files/EEZ Mosfet pre-regulator r3B3b (SS).sch (EAGLE design)
At the start: 87 parts, among them IC1 LP2951SO8, IC2 LP2951SO8, IC3 LM5574, IC4 LM337LZ, IC5 Si8610BC-B-IS, IC6 TLC555, P1 500K, Q1 MMBT5401, Q2 IRF5210PBF, Q3 IRF5210PBF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

Commit message: minor textual corrections
Other:
- note added: "Note 2.1: replace with 33K or 36K (to decrease frequency) to become slave in multiple devices sync configuration"
- note removed: "Note 2.1: replace with 33K (to decrease frequency) if sync with LM5574 on pre-regulator board is used"
Changed lines of the file:
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@@
 <text x="127" y="-99.06" size="1.778" layer="97" rot="MR180">V/F converter for temperature sensor (optional)</text>
 <wire x1="124.46" y1="-97.79" x2="262.255" y2="-97.79" width="0.1524" layer="97" style="shortdash"/>
-<text x="10.16" y="-170.18" size="1.27" layer="108">Note 2.1: replace with 33K (to decrease frequency) if sync with LM5574 on pre-regulator board is used</text>
 <text x="13.97" y="-78.74" size="1.27" layer="108">See note 2.1</text>
 <text x="66.04" y="-59.69" size="1.27" layer="96">or DFLS1100-7</text>
@@
 <text x="2.54" y="-185.42" size="1.778" layer="94">Repository: https://github.com/eez-open</text>
 <text x="2.54" y="-182.88" size="1.778" layer="94">More info at http://www.envox.hr/eez</text>
+<text x="10.16" y="-170.18" size="1.27" layer="108">Note 2.1: replace with 33K or 36K (to decrease frequency) to become slave in multiple devices sync configuration</text>
 </plain>
 <instances>
