File: Arduino shield/Eagle files/EEZ Arduino shield+BP r1B13a.brd (EAGLE design)
At the start: 175 x 105 mm, 191 parts, among them IC1 TLC5925, IC10 SN74LV125APW, IC11 SI8620EC-B-IS, IC12 SI8620EC-B-IS, IC13 Si8660EC-B-IS1, IC14 PCA21125, IC15 AT25256B, IC16 ENC28J60-I/SS, IC17 BC857BS, IC18 NE555D, IC19 BC857BS, IC2 SN74LVCC3245ADBRSSOP, IC20 NE555D, IC21 SN74LV1T34, IC3 SN74LVCC3245ADBRSSOP, IC4 SN74LVCC3245ADBRSSOP, IC5 SN74LVCC3245ADBRSSOP, IC6 LD1117ADT33TR, IC7 SN74LVCC3245ADBRSSOP, IC8 SN74LVCC3245ADBRSSOP, IC9 Si8660EC-B-IS1, J1 BS-244DSM-R, J2 BS-244DSM-B, J3 BS-244DSM-R, J4 BS-244DSM-G, J5 BS-244DSM-B, Q1 IRLML2246TRPBF, Q10 2N7002, Q11 2N7002, Q12 2N7002, Q13 2N7002, Q2 IRLML2246TRPBF, Q3 IRLML2246TRPBF, Q4 2N7002, Q5 IRLML2246TRPBF, Q6 2N7002, Q7 2N7002, Q8 2N7002, Q9 IRLML2246TRPBF, SW1 1301.9316, X1 282836-4, X10 LMJTAB881243M-L, X11 22-23-2021, X12 22-23-2021, X2 MC000005, X3 282836-4, X4 MC000005, X5 22-23-2021, X6 22-23-2041, X7 09185106324, X8 09185106324, X9 22-23-2021, Y1 32,768kHz, Y2 25MHz

Commit message: Arduino Shield r1B13a update
Connections:
- net EARTH: now also X4.4, X4.4.1; no longer X4.6, X4.6.1
- net SENSE2+: now also X4.5, X4.5.1; no longer X4.4, X4.4.1
- net SENSE2-: now also X4.6, X4.6.1; no longer X4.5, X4.5.1
Routing:
- net SENSE2-: track 17.7 -> 11.6 mm
- net SENSE2+: track 22.6 -> 19.9 mm
- net EARTH: track 377.1 -> 375.4 mm
Other:
- board text added: "EEZ Arduino shield+BP (03/2016 r1B13a)"
- board text removed: "EEZ Arduino shield+BP (03/2016 r1B13)"
Changed lines of the file:
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@@
 <text x="142.875" y="23.114" size="1.6764" layer="21" ratio="10">JP2 settings:</text>
 <wire x1="173.2915" y1="2.2225" x2="191.77" y2="2.2225" width="2.1844" layer="29"/>
-<text x="29.1465" y="2.3495" size="1.6764" layer="21" ratio="10" rot="SR0">EEZ Arduino shield+BP (03/2016 r1B13)</text>
+<text x="29.1465" y="2.3495" size="1.6764" layer="21" ratio="10" rot="SR0">EEZ Arduino shield+BP (03/2016 r1B13a)</text>
 <text x="139.065" y="20.193" size="2.54" layer="21" ratio="15">!</text>
 <wire x1="136.652" y1="19.431" x2="139.2555" y2="24.1935" width="0.3048" layer="21"/>
@@
 <text x="162.052" y="74.4855" size="1.6764" layer="21" ratio="10">PWML</text>
 <text x="124.587" y="74.4855" size="1.6764" layer="21" ratio="10">Comm</text>
-<text x="82.804" y="2.286" size="1.6764" layer="16" ratio="10" rot="SMR0">EEZ Arduino shield+BP (03/2016 r1B13)</text>
+<text x="84.3915" y="2.3495" size="1.6764" layer="16" ratio="10" rot="SMR0">EEZ Arduino shield+BP (03/2016 r1B13a)</text>
 <text x="29.4005" y="78.2955" size="1.524" layer="21" ratio="10">Ch#1</text>
 <text x="75.7555" y="94.234" size="1.016" layer="21" ratio="10">Temp out1</text>
@@
 <contactref element="J4" pad="P$1"/>
 <wire x1="27.3685" y1="20.6315" x2="27.3685" y2="76.7715" width="1.016" layer="1"/>
-<contactref element="X4" pad="3"/>
-<contactref element="X4" pad="3.1"/>
-<contactref element="X4" pad="6.1"/>
-<contactref element="X4" pad="6"/>
 <wire x1="49.9745" y1="12.697" x2="69.0235" y2="12.697" width="1.016" layer="1"/>
 <wire x1="69.0235" y1="12.697" x2="69.0265" y2="12.7" width="1.016" layer="1"/>
@@
 <wire x1="35.303" y1="12.697" x2="34" y2="14" width="1.016" layer="1"/>
 <wire x1="27.3685" y1="20.6315" x2="34" y2="14" width="1.016" layer="1"/>
-<wire x1="69.0265" y1="12.7" x2="72.5805" y2="12.7" width="0.8128" layer="1"/>
-<wire x1="72.5805" y1="12.7" x2="80.264" y2="20.3835" width="0.8128" layer="1"/>
-<wire x1="81.0895" y1="18.8595" x2="80.2005" y2="19.7485" width="0.4064" layer="1"/>
-<wire x1="80.2005" y1="19.7485" x2="80.2005" y2="20.32" width="0.4064" layer="1"/>
-<wire x1="80.2005" y1="20.32" x2="80.264" y2="20.3835" width="0.4064" layer="1"/>
-<wire x1="87.884" y1="20.3835" x2="87.884" y2="25.4" width="0.4064" layer="16"/>
-<wire x1="80.264" y1="25.4635" x2="80.264" y2="20.3835" width="0.4064" layer="16"/>
-<wire x1="81.0895" y1="18.8595" x2="86.36" y2="18.8595" width="0.4064" layer="1"/>
-<wire x1="86.36" y1="18.8595" x2="87.884" y2="20.3835" width="0.4064" layer="1"/>
 <wire x1="69.079" y1="89.029" x2="69.079" y2="96.4655" width="0.4064" layer="1"/>
 <via x="49.9745" y="98.171" extent="1-16" drill="0.6" shape="octagon"/>
@@
 <contactref element="X10" pad="SH1"/>
 <contactref element="X10" pad="SH2"/>
-<wire x1="87.884" y1="25.4" x2="87.884" y2="25.4635" width="0" layer="19" extent="16-16"/>
+<contactref element="X4" pad="4"/>
+<contactref element="X4" pad="4.1"/>
+<contactref element="X4" pad="3"/>
+<contactref element="X4" pad="3.1"/>
+<wire x1="85.344" y1="25.4635" x2="85.344" y2="20.3835" width="0.4064" layer="16"/>
+<wire x1="85.344" y1="20.3835" x2="87.884" y2="20.3835" width="0.4064" layer="16"/>
+<wire x1="87.884" y1="25.4635" x2="87.884" y2="20.3835" width="0.4064" layer="16"/>
+<wire x1="69.0265" y1="12.7" x2="77.6605" y2="12.7" width="0.8128" layer="1"/>
+<wire x1="77.6605" y1="12.7" x2="85.344" y2="20.3835" width="0.8128" layer="1"/>
 </signal>
 <signal name="SENSE1+">
@@
 </signal>
 <signal name="SENSE2+">
-<contactref element="X4" pad="4"/>
-<contactref element="X4" pad="4.1"/>
 <contactref element="K_S2" pad="4"/>
 <wire x1="77.978" y1="38.2075" x2="77.978" y2="33.9725" width="0.3048" layer="1"/>
 <wire x1="77.978" y1="33.9725" x2="79.1845" y2="32.766" width="0.3048" layer="1"/>
-<wire x1="79.1845" y1="32.766" x2="79.1845" y2="28.702" width="0.3048" layer="1"/>
-<wire x1="79.1845" y1="28.702" x2="80.391" y2="27.4955" width="0.3048" layer="1"/>
-<wire x1="80.391" y1="27.4955" x2="83.312" y2="27.4955" width="0.3048" layer="1"/>
-<wire x1="83.312" y1="27.4955" x2="85.344" y2="25.4635" width="0.3048" layer="1"/>
-<wire x1="85.344" y1="25.4635" x2="85.344" y2="20.3835" width="0.4064" layer="16"/>
+<wire x1="79.1845" y1="32.766" x2="79.1845" y2="28.956" width="0.3048" layer="1"/>
+<contactref element="X4" pad="5"/>
+<contactref element="X4" pad="5.1"/>
+<wire x1="82.804" y1="25.4635" x2="82.677" y2="25.4635" width="0.3048" layer="1"/>
+<wire x1="82.677" y1="25.4635" x2="79.1845" y2="28.956" width="0.3048" layer="1"/>
+<wire x1="82.804" y1="20.3835" x2="82.804" y2="25.4635" width="0.4064" layer="16"/>
 </signal>
 <signal name="SENSE2-">
-<contactref element="X4" pad="5.1"/>
-<contactref element="X4" pad="5"/>
 <contactref element="K_S2" pad="5"/>
-<wire x1="77.978" y1="31.0075" x2="77.978" y2="25.2095" width="0.3048" layer="1"/>
-<wire x1="77.978" y1="25.2095" x2="82.804" y2="20.3835" width="0.3048" layer="1"/>
-<wire x1="82.804" y1="25.4635" x2="82.804" y2="20.3835" width="0.4064" layer="16"/>
+<contactref element="X4" pad="6.1"/>
+<contactref element="X4" pad="6"/>
+<wire x1="77.978" y1="31.0075" x2="77.978" y2="27.7495" width="0.3048" layer="1"/>
+<wire x1="77.978" y1="27.7495" x2="80.264" y2="25.4635" width="0.3048" layer="1"/>
+<wire x1="80.264" y1="20.3835" x2="80.264" y2="25.4635" width="0.4064" layer="16"/>
 </signal>
 <signal name="OUT2-">
@@
 <wire x1="85.344" y1="71.882" x2="88.011" y2="69.215" width="0.4064" layer="1"/>
 <wire x1="88.011" y1="69.215" x2="104.8385" y2="69.215" width="0.4064" layer="1"/>
-<wire x1="104.8385" y1="69.215" x2="105.156" y2="69.5325" width="0" layer="19" extent="1-16"/>
 <wire x1="58.547" y1="94.869" x2="56.388" y2="92.71" width="0.4064" layer="16"/>
 <wire x1="50.1755" y1="34.29" x2="50.1755" y2="38.174" width="0.4064" layer="1"/>
