File: Arduino shield/Eagle files/EEZ Arduino shield+BP r1B13a.sch (EAGLE design)
At the start: 187 parts, among them IC1 TLC5925, IC10 SN74LV125APW, IC11 SI8620EC-B-IS, IC12 SI8620EC-B-IS, IC13 Si8660EC-B-IS1, IC14 PCA21125, IC15 AT25256B, IC16 ENC28J60-I/SS, IC17 BC857BS, IC18 NE555D, IC19 BC857BS, IC2 SN74LVCC3245ADBRSSOP, IC20 NE555D, IC21 SN74LV1T34, IC3 SN74LVCC3245ADBRSSOP, IC4 SN74LVCC3245ADBRSSOP, IC5 SN74LVCC3245ADBRSSOP, IC6 LD1117ADT33TR, IC7 SN74LVCC3245ADBRSSOP, IC8 SN74LVCC3245ADBRSSOP, IC9 Si8660EC-B-IS1, J1 BS-244DSM-R, J2 BS-244DSM-B, J3 BS-244DSM-R, J4 BS-244DSM-G, J5 BS-244DSM-B, Q1 IRLML2246TRPBF, Q10 2N7002, Q11 2N7002, Q12 2N7002, Q13 2N7002, Q2 IRLML2246TRPBF, Q3 IRLML2246TRPBF, Q4 2N7002, Q5 IRLML2246TRPBF, Q6 2N7002, Q7 2N7002, Q8 2N7002, Q9 IRLML2246TRPBF, SW1 1301.9316, X1 282836-4, X10 LMJTAB881243M-L, X11 22-23-2021, X12 22-23-2021, X2 MC000005, X3 282836-4, X4 MC000005, X5 22-23-2021, X6 22-23-2041, X7 09185106324, X8 09185106324, X9 22-23-2021, Y1 32,768kHz, Y2 25MHz

Commit message: Arduino Shield r1B13a update
Connections:
- net EARTH: now also X4-4.1; no longer X4-6.1
- net SENSE2+: now also X4-5.1; no longer X4-4.1
- net SENSE2-: now also X4-6.1; no longer X4-5.1
Other:
- note added: "3 Earth"
- note added: "4 Earth"
- note added: "6-pin push-in connector X3"
- note added: "6-pin push-in connector X4"
- note removed: "6-pin push-in connector X3, X4"
- moved on the sheet: X4-4, X4-5, X4-6
Changed lines of the file:
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@@
 <wire x1="113.03" y1="38.1" x2="113.03" y2="43.18" width="0.1524" layer="101"/>
 <wire x1="113.03" y1="43.18" x2="128.27" y2="43.18" width="0.1524" layer="101"/>
-<text x="109.22" y="60.325" size="2.1844" layer="101">6-pin push-in connector X3, X4</text>
+<text x="109.22" y="60.325" size="2.1844" layer="101">6-pin push-in connector X3</text>
 <circle x="119.38" y="39.37" radius="0.635" width="0.1524" layer="101"/>
 <text x="128.905" y="45.085" size="1.4224" layer="101">6 Battery NTC (Input)</text>
@@
 <wire x1="137.16" y1="22.225" x2="121.92" y2="22.225" width="0.1524" layer="103"/>
 <wire x1="111.76" y1="22.225" x2="121.92" y2="22.225" width="0.1524" layer="103"/>
+<circle x="167.64" y="39.37" radius="0.635" width="0.1524" layer="101"/>
+<circle x="165.1" y="39.37" radius="0.635" width="0.1524" layer="101"/>
+<wire x1="179.07" y1="43.18" x2="179.07" y2="38.1" width="0.1524" layer="101"/>
+<wire x1="179.07" y1="38.1" x2="163.83" y2="38.1" width="0.1524" layer="101"/>
+<wire x1="163.83" y1="38.1" x2="163.83" y2="43.18" width="0.1524" layer="101"/>
+<wire x1="163.83" y1="43.18" x2="179.07" y2="43.18" width="0.1524" layer="101"/>
+<text x="160.02" y="60.325" size="2.1844" layer="101">6-pin push-in connector X4</text>
+<circle x="170.18" y="39.37" radius="0.635" width="0.1524" layer="101"/>
+<text x="179.705" y="45.085" size="1.4224" layer="101">6 Battery NTC (Input)</text>
+<circle x="172.72" y="39.37" radius="0.635" width="0.1524" layer="101"/>
+<text x="179.705" y="47.625" size="1.4224" layer="101">5 Channel ground</text>
+<circle x="175.26" y="39.37" radius="0.635" width="0.1524" layer="101"/>
+<circle x="177.8" y="39.37" radius="0.635" width="0.1524" layer="101"/>
+<text x="179.705" y="57.785" size="1.4224" layer="101">1 Remote sense- (Input)</text>
+<text x="179.705" y="52.705" size="1.4224" layer="101">3 Earth</text>
+<wire x1="179.07" y1="55.88" x2="173.99" y2="55.88" width="0.1524" layer="101"/>
+<wire x1="173.99" y1="55.88" x2="167.64" y2="49.53" width="0.1524" layer="101"/>
+<wire x1="167.64" y1="49.53" x2="167.64" y2="44.45" width="0.1524" layer="101"/>
+<wire x1="179.07" y1="53.34" x2="175.26" y2="53.34" width="0.1524" layer="101"/>
+<wire x1="175.26" y1="53.34" x2="170.18" y2="48.26" width="0.1524" layer="101"/>
+<wire x1="170.18" y1="48.26" x2="170.18" y2="44.45" width="0.1524" layer="101"/>
+<wire x1="179.07" y1="50.8" x2="176.53" y2="50.8" width="0.1524" layer="101"/>
+<wire x1="176.53" y1="50.8" x2="172.72" y2="46.99" width="0.1524" layer="101"/>
+<wire x1="172.72" y1="46.99" x2="172.72" y2="44.45" width="0.1524" layer="101"/>
+<wire x1="177.8" y1="48.26" x2="175.26" y2="45.72" width="0.1524" layer="101"/>
+<wire x1="175.26" y1="45.72" x2="175.26" y2="44.45" width="0.1524" layer="101"/>
+<wire x1="179.07" y1="45.72" x2="177.8" y2="45.72" width="0.1524" layer="101"/>
+<wire x1="177.8" y1="44.45" x2="177.8" y2="45.72" width="0.1524" layer="101"/>
+<wire x1="177.8" y1="48.26" x2="179.07" y2="48.26" width="0.1524" layer="101"/>
+<wire x1="165.1" y1="44.45" x2="165.1" y2="50.8" width="0.1524" layer="101"/>
+<wire x1="165.1" y1="50.8" x2="172.72" y2="58.42" width="0.1524" layer="101"/>
+<wire x1="172.72" y1="58.42" x2="179.07" y2="58.42" width="0.1524" layer="101"/>
+<text x="179.705" y="50.165" size="1.4224" layer="101">4 Earth</text>
+<text x="179.705" y="55.245" size="1.4224" layer="101">2 Remote sense+ (Input)</text>
 </plain>
 <instances>
@@
 <attribute name="NAME" x="90.17" y="49.149" size="1.778" layer="95" rot="MR180"/>
 </instance>
-<instance part="X4" gate="-4" x="83.82" y="73.66" smashed="yes" rot="R180">
+<instance part="X4" gate="-4" x="83.82" y="45.72" smashed="yes" rot="R180">
+<attribute name="NAME" x="90.17" y="44.831" size="1.778" layer="95"/>
+</instance>
+<instance part="X4" gate="-5" x="83.82" y="73.66" smashed="yes" rot="R180">
 <attribute name="NAME" x="90.17" y="72.771" size="1.778" layer="95"/>
 </instance>
-<instance part="X4" gate="-5" x="83.82" y="35.56" smashed="yes" rot="R180">
-<attribute name="NAME" x="90.17" y="34.671" size="1.778" layer="95"/>
-</instance>
-<instance part="X4" gate="-6" x="83.82" y="45.72" smashed="yes" rot="MR0">
-<attribute name="NAME" x="90.17" y="46.609" size="1.778" layer="95" rot="MR180"/>
+<instance part="X4" gate="-6" x="83.82" y="35.56" smashed="yes" rot="MR0">
+<attribute name="NAME" x="90.17" y="36.449" size="1.778" layer="95" rot="MR180"/>
 </instance>
 <instance part="LED_01_POS" gate="-GREEN" x="243.84" y="129.54" smashed="yes" rot="R270">
@@
 <label x="88.9" y="55.88" size="1.27" layer="102" rot="R180"/>
 <pinref part="J4" gate="G$1" pin="P$1"/>
+<junction x="78.74" y="48.26"/>
+<wire x1="81.28" y1="48.26" x2="78.74" y2="48.26" width="0.1524" layer="91"/>
+<wire x1="81.28" y1="45.72" x2="81.28" y2="48.26" width="0.1524" layer="91"/>
+<pinref part="X4" gate="-4" pin="1"/>
+<wire x1="81.28" y1="45.72" x2="83.82" y2="45.72" width="0.1524" layer="91"/>
 <pinref part="X4" gate="-3" pin="1"/>
 <wire x1="83.82" y1="48.26" x2="81.28" y2="48.26" width="0.1524" layer="91"/>
-<junction x="78.74" y="48.26"/>
-<pinref part="X4" gate="-6" pin="1"/>
-<wire x1="81.28" y1="48.26" x2="78.74" y2="48.26" width="0.1524" layer="91"/>
-<wire x1="83.82" y1="45.72" x2="81.28" y2="45.72" width="0.1524" layer="91"/>
-<wire x1="81.28" y1="45.72" x2="81.28" y2="48.26" width="0.1524" layer="91"/>
 <junction x="81.28" y="48.26"/>
 </segment>
@@
 <label x="83.185" y="75.565" size="1.27" layer="102" rot="R180"/>
 <wire x1="40.64" y1="73.66" x2="83.82" y2="73.66" width="0.1524" layer="91"/>
-<pinref part="X4" gate="-4" pin="1"/>
 <pinref part="K_S2" gate="2" pin="S"/>
+<pinref part="X4" gate="-5" pin="1"/>
 </segment>
 </net>
@@
 <label x="83.185" y="37.465" size="1.27" layer="102" rot="R180"/>
 <wire x1="40.64" y1="35.56" x2="83.82" y2="35.56" width="0.1524" layer="91"/>
-<pinref part="X4" gate="-5" pin="1"/>
 <pinref part="K_S2" gate="3" pin="S"/>
-</segment>
-</net>
+<pinref part="X4" gate="-6" pin="1"/>
+</segment>
+</net>
