File: Arduino shield/Eagle files/EEZ Arduino shield+BP r1B14.brd (EAGLE design)
At the start: 175 x 105 mm, 190 parts, among them IC1 TLC5925, IC10 SN74LV125APW, IC11 SI8620EC-B-IS, IC12 SI8620EC-B-IS, IC13 Si8660EC-B-IS1, IC14 PCA21125, IC15 AT25256B, IC16 ENC28J60-I/SS, IC17 BC857BS, IC18 NE555D, IC19 BC857BS, IC2 SN74LVCC3245ADBRSSOP, IC20 NE555D, IC21 SN74LV1T34, IC3 SN74LVCC3245ADBRSSOP, IC4 SN74LVCC3245ADBRSSOP, IC5 SN74LVCC3245ADBRSSOP, IC6 LD1117ADT33TR, IC7 SN74LVCC3245ADBRSSOP, IC8 SN74LVCC3245ADBRSSOP, IC9 Si8660EC-B-IS1, J1 BS-244DSM-R, J2 BS-244DSM-B, J3 BS-244DSM-R, J4 BS-244DSM-G, J5 BS-244DSM-B, Q1 IRLML2246TRPBF, Q10 2N7002, Q11 2N7002, Q12 2N7002, Q13 2N7002, Q2 IRLML2246TRPBF, Q3 IRLML2246TRPBF, Q4 2N7002, Q5 IRLML2246TRPBF, Q6 2N7002, Q7 2N7002, Q8 2N7002, Q9 IRLML2246TRPBF, SW1 1301.9316, X1 282836-4, X10 22-23-2021, X11 22-23-2021, X2 MC000005, X3 282836-4, X4 MC000005, X5 09185067324, X6 09185106324, X7 09185106324, X8 22-23-2021, X9 LMJTAB881243M-L, Y1 32,768kHz, Y2 25MHz

Commit message: AUX PS r4B41 BOM update
Routing:
- net OUT1+: track 41.7 -> 39.4 mm
Changed lines of the file:
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@@
 <layer number="17" name="Pads" color="14" fill="1" visible="yes" active="yes"/>
 <layer number="18" name="Vias" color="14" fill="1" visible="yes" active="yes"/>
-<layer number="19" name="Unrouted" color="6" fill="1" visible="no" active="yes"/>
-<layer number="20" name="Dimension" color="15" fill="1" visible="yes" active="yes"/>
-<layer number="21" name="tPlace" color="7" fill="1" visible="yes" active="yes"/>
+<layer number="19" name="Unrouted" color="6" fill="1" visible="yes" active="yes"/>
+<layer number="20" name="Dimension" color="15" fill="1" visible="no" active="yes"/>
+<layer number="21" name="tPlace" color="7" fill="1" visible="no" active="yes"/>
 <layer number="22" name="bPlace" color="7" fill="1" visible="no" active="yes"/>
 <layer number="23" name="tOrigins" color="15" fill="1" visible="no" active="yes"/>
 <layer number="24" name="bOrigins" color="15" fill="1" visible="no" active="yes"/>
-<layer number="25" name="tNames" color="7" fill="1" visible="yes" active="yes"/>
+<layer number="25" name="tNames" color="7" fill="1" visible="no" active="yes"/>
 <layer number="26" name="bNames" color="7" fill="1" visible="no" active="yes"/>
 <layer number="27" name="tValues" color="10" fill="1" visible="no" active="yes"/>
 <layer number="28" name="bValues" color="3" fill="1" visible="no" active="yes"/>
 <layer number="29" name="tStop" color="15" fill="3" visible="no" active="yes"/>
-<layer number="30" name="bStop" color="7" fill="6" visible="yes" active="yes"/>
+<layer number="30" name="bStop" color="7" fill="6" visible="no" active="yes"/>
 <layer number="31" name="tCream" color="7" fill="4" visible="no" active="yes"/>
 <layer number="32" name="bCream" color="7" fill="5" visible="no" active="yes"/>
@@
 <layer number="37" name="tTest" color="7" fill="1" visible="no" active="yes"/>
 <layer number="38" name="bTest" color="7" fill="1" visible="no" active="yes"/>
-<layer number="39" name="tKeepout" color="15" fill="1" visible="yes" active="yes"/>
+<layer number="39" name="tKeepout" color="15" fill="1" visible="no" active="yes"/>
 <layer number="40" name="bKeepout" color="1" fill="11" visible="no" active="yes"/>
 <layer number="41" name="tRestrict" color="4" fill="10" visible="no" active="yes"/>
@@
 <attribute name="MF" value="OMRON COMPONENTS USA" x="60.198" y="81.026" size="1.778" layer="27" display="off"/>
 <attribute name="OC_FARNELL" value="1690427" x="60.198" y="81.026" size="1.778" layer="27" display="off"/>
-<attribute name="NAME" x="55.432" y="90.997" size="1.27" layer="25" ratio="10" rot="R90"/>
+<attribute name="NAME" x="54.421" y="92.3325" size="1.27" layer="25" ratio="10"/>
 <attribute name="VALUE" x="54.737" y="87.122" size="1.016" layer="27" ratio="10"/>
 </element>
@@
 </element>
 <element name="X4" library="EEZ_Lib1" package="MC000005_MIRROR" value="MC000005" x="92.964" y="25.4635" locked="yes" smashed="yes">
-<attribute name="NAME" x="78.994" y="29.2735" size="1.6764" layer="25" ratio="10"/>
+<attribute name="NAME" x="95.504" y="28.829" size="1.6764" layer="25" ratio="10"/>
 <attribute name="VALUE" x="82.4865" y="22.225" size="1.6764" layer="27" ratio="10"/>
 </element>
@@
 <wire x1="66.1855" y1="74.1355" x2="69.05" y2="77" width="0.6096" layer="1"/>
 <wire x1="69.079" y1="86.229" x2="69.079" y2="78.0325" width="0.4064" layer="1"/>
-<wire x1="69.079" y1="78.0325" x2="67.437" y2="76.3905" width="0.4064" layer="1"/>
 <wire x1="58.928" y1="90.976" x2="58.928" y2="89.7255" width="0.3048" layer="1"/>
 <wire x1="58.928" y1="89.7255" x2="60.198" y2="88.4555" width="0.3048" layer="1"/>
@@
 <contactref element="IC14" pad="5"/>
 <via x="156.21" y="64.008" extent="1-16" drill="0.6" shape="octagon"/>
-<wire x1="179.451" y1="63.8175" x2="190.4365" y2="63.8175" width="0.254" layer="16"/>
 <via x="191.262" y="61.9125" extent="1-16" drill="0.6" shape="octagon"/>
 <wire x1="193.4591" y1="58.8264" x2="193.4591" y2="60.3504" width="0.254" layer="1"/>
 <wire x1="191.262" y1="61.9125" x2="191.262" y2="62.992" width="0.254" layer="16"/>
-<wire x1="191.262" y1="62.992" x2="190.4365" y2="63.8175" width="0.254" layer="16"/>
+<wire x1="191.262" y1="62.992" x2="190.246" y2="64.008" width="0.254" layer="16"/>
 <wire x1="193.4591" y1="60.3504" x2="191.897" y2="61.9125" width="0.254" layer="1"/>
 <wire x1="191.262" y1="61.9125" x2="191.897" y2="61.9125" width="0.254" layer="1"/>
@@
 <wire x1="163.957" y1="62.6745" x2="157.5435" y2="62.6745" width="0.254" layer="16"/>
 <wire x1="157.5435" y1="62.6745" x2="156.21" y2="64.008" width="0.254" layer="16"/>
+<wire x1="190.246" y1="64.008" x2="180.848" y2="64.008" width="0.254" layer="16"/>
+<wire x1="180.848" y1="64.008" x2="180.6575" y2="63.8175" width="0.254" layer="16"/>
+<wire x1="180.6575" y1="63.8175" x2="179.451" y2="63.8175" width="0.254" layer="16"/>
 </signal>
 <signal name="N$97">
@@
 <contactref element="LCD1" pad="34"/>
 <via x="136.906" y="22.9235" extent="1-16" drill="0.6" shape="octagon"/>
-<via x="144.9705" y="32.512" extent="1-16" drill="0.6" shape="octagon"/>
+<via x="144.78" y="32.385" extent="1-16" drill="0.6" shape="octagon"/>
 <via x="145.669" y="69.1515" extent="1-16" drill="0.6" shape="octagon"/>
 <wire x1="148.1455" y1="28.0035" x2="148.1455" y2="24.13" width="0.254" layer="1"/>
@@
 <wire x1="144.907" y1="53.7845" x2="143.51" y2="52.3875" width="0.254" layer="16"/>
 <wire x1="145.288" y1="44.5135" x2="143.51" y2="46.2915" width="0.254" layer="16"/>
-<wire x1="147.32" y1="29.718" x2="144.9705" y2="32.0675" width="0.254" layer="1"/>
-<wire x1="144.9705" y1="32.512" x2="144.9705" y2="32.0675" width="0.254" layer="1"/>
+<wire x1="147.32" y1="29.718" x2="144.78" y2="32.258" width="0.254" layer="1"/>
 <wire x1="147.32" y1="28.829" x2="147.32" y2="29.718" width="0.254" layer="1"/>
-<wire x1="145.288" y1="44.5135" x2="145.288" y2="32.8295" width="0.254" layer="16"/>
-<wire x1="145.288" y1="32.8295" x2="144.9705" y2="32.512" width="0.254" layer="16"/>
+<wire x1="145.288" y1="44.5135" x2="145.288" y2="32.893" width="0.254" layer="16"/>
 <wire x1="146.05" y1="68.7705" x2="145.669" y2="69.1515" width="0.254" layer="1"/>
+<wire x1="145.288" y1="32.893" x2="144.78" y2="32.385" width="0.254" layer="16"/>
+<wire x1="144.78" y1="32.385" x2="144.78" y2="32.258" width="0.254" layer="1"/>
 </signal>
 <signal name="3V3LCD_WR">
@@
 <wire x1="159.004" y1="79.248" x2="159.004" y2="80.518" width="0.254" layer="16"/>
 <wire x1="159.004" y1="80.518" x2="154.8765" y2="84.6455" width="0.254" layer="16"/>
-<wire x1="179.197" y1="64.389" x2="180.2765" y2="64.389" width="0.254" layer="16"/>
-<wire x1="180.2765" y1="64.77" x2="180.2765" y2="64.389" width="0.254" layer="16"/>
-<wire x1="180.2765" y1="64.389" x2="190.6905" y2="64.389" width="0.254" layer="16"/>
 <via x="191.8335" y="57.2135" extent="1-16" drill="0.6" shape="octagon"/>
-<wire x1="190.6905" y1="64.389" x2="192.2145" y2="62.865" width="0.254" layer="16"/>
+<wire x1="190.5" y1="64.5795" x2="192.2145" y2="62.865" width="0.254" layer="16"/>
 <wire x1="192.2145" y1="62.865" x2="192.2145" y2="57.5945" width="0.254" layer="16"/>
 <wire x1="192.2145" y1="57.5945" x2="191.8335" y2="57.2135" width="0.254" layer="16"/>
@@
 <wire x1="132.08" y1="30.099" x2="132.08" y2="20.0025" width="0.254" layer="1"/>
 <wire x1="132.08" y1="20.0025" x2="132.588" y2="19.4945" width="0.254" layer="1"/>
+<wire x1="180.2765" y1="64.77" x2="180.467" y2="64.5795" width="0.254" layer="16"/>
+<wire x1="180.467" y1="64.5795" x2="190.5" y2="64.5795" width="0.254" layer="16"/>
+<wire x1="179.197" y1="64.389" x2="179.8955" y2="64.389" width="0.254" layer="16"/>
+<wire x1="179.8955" y1="64.389" x2="180.2765" y2="64.77" width="0.254" layer="16"/>
 </signal>
 <signal name="!ISOLATOR1_EN">
@@
 <via x="181.5465" y="69.977" extent="1-16" drill="0.6" shape="octagon"/>
 <wire x1="181.5465" y1="67.2465" x2="181.5465" y2="69.977" width="0.254" layer="1"/>
-<via x="182.5625" y="65.3415" extent="1-16" drill="0.6" shape="octagon"/>
+<via x="182.5625" y="65.532" extent="1-16" drill="0.6" shape="octagon"/>
 <wire x1="181.5592" y1="67.2592" x2="181.5465" y2="67.2465" width="0.254" layer="1"/>
 <wire x1="192.1637" y1="53.1876" x2="192.1637" y2="53.7718" width="0.254" layer="1"/>
@@
 <wire x1="192.1637" y1="54.0893" x2="191.77" y2="54.483" width="0.254" layer="1"/>
 <wire x1="181.5465" y1="67.2465" x2="181.5465" y2="65.7225" width="0.254" layer="1"/>
-<wire x1="181.5465" y1="65.7225" x2="181.9275" y2="65.3415" width="0.254" layer="1"/>
-<wire x1="182.5625" y1="65.3415" x2="181.9275" y2="65.3415" width="0.254" layer="1"/>
-<wire x1="182.5625" y1="65.3415" x2="182.9435" y2="64.9605" width="0.254" layer="16"/>
-<wire x1="182.9435" y1="64.9605" x2="190.9445" y2="64.9605" width="0.254" layer="16"/>
-<wire x1="190.9445" y1="64.9605" x2="192.786" y2="63.119" width="0.254" layer="16"/>
+<wire x1="190.754" y1="65.151" x2="192.786" y2="63.119" width="0.254" layer="16"/>
 <contactref element="IC8" pad="9"/>
 <wire x1="181.483" y1="69.9135" x2="181.5465" y2="69.977" width="0.254" layer="16"/>
@@
 <wire x1="136.8425" y1="15.0495" x2="141.351" y2="19.558" width="0.254" layer="1"/>
 <wire x1="141.351" y1="19.558" x2="153.162" y2="19.558" width="0.254" layer="1"/>
+<wire x1="190.754" y1="65.151" x2="182.9435" y2="65.151" width="0.254" layer="16"/>
+<wire x1="182.9435" y1="65.151" x2="182.5625" y2="65.532" width="0.254" layer="16"/>
+<wire x1="182.5625" y1="65.532" x2="181.737" y2="65.532" width="0.254" layer="1"/>
+<wire x1="181.737" y1="65.532" x2="181.5465" y2="65.7225" width="0.254" layer="1"/>
 </signal>
 <signal name="!3V3RESET">
@@
 </signal>
 </signals>
-<errors>
-</errors>
 </board>
 </drawing>
