File: Arduino shield/Eagle files/EEZ Arduino shield+BP r3B3.sch (EAGLE design)
At the start: 177 parts, among them IC1 TLC5925IDBQR, IC10 BC857BS, IC11 TLC555, IC12 SN74LVC2G08DCTR, IC13 TPS3705-33D, IC14 SN74LV1T34DBVR, IC15 SN74LVC2G02DCTR, IC2 Si8641EC-B-IS1, IC3 SI8651EC-B-IS1, IC4 SI8651EC-B-IS1, IC5 LD1117ADT33TR, IC6 Si8641EC-B-IS1, IC7 PCA21125, IC8 AT25256B, IC9 W5500, J1 BS-244DSM-R, J2 BS-244DSM-G, J3 BS-244DSM-B, J4 BS-244DSM-R, J5 BS-244DSM-B, Q1 IRLML2246TRPBF, Q2 IRLML2246TRPBF, Q3 IRLML2246TRPBF, Q4 IRLML2246TRPBF, Q5 2N7002, Q6 IRLML2246TRPBF, Q7 2N7002, Q8 2N7002, SW1 A101SYCQ04, SW2 1301.9316, X1 MC000006, X2 TSW-113-07-F-D, X3 MC000005, X4 TSW-113-07-F-D, X5 09185067324, X6 22-23-2021, X7 826629-8, X8 22-23-2041, X9 SSW-105-02-S-D, Y1 32,768kHz, Y2 25MHz

Commit message: AUX PS, Arduino Shield: removed Net class 1
Parts:
- C28, C32: device rcl:C-EUC0603 -> rcl:C-EUC0805
Changed lines of the file:
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@@
 <clearance class="0" value="0.254"/>
 </class>
-<class number="1" name="power" width="0.254" drill="0.5842">
-<clearance class="1" value="0.254"/>
-</class>
 <class number="2" name="gnd" width="0.254" drill="0.5842">
 <clearance class="2" value="0.254"/>
@@
 <part name="C31" library="rcl" deviceset="C-EU" device="C0603" value="6n8"/>
 <part name="C41" library="EEZ_Lib1" deviceset="ECAP" device="1206" value="10u"/>
-<part name="C28" library="rcl" deviceset="C-EU" device="C0603" value="18p"/>
-<part name="C32" library="rcl" deviceset="C-EU" device="C0603" value="18p"/>
+<part name="C28" library="rcl" deviceset="C-EU" device="C0805" value="18p"/>
+<part name="C32" library="rcl" deviceset="C-EU" device="C0805" value="18p"/>
 <part name="SH1" library="EEZ_Lib1" deviceset="SHORT" device="NOHOLE"/>
 <part name="SUPPLY3" library="supply2" deviceset="GND" device=""/>
@@
 </segment>
 </net>
-<net name="+3V3" class="1">
+<net name="+3V3" class="0">
 <segment>
 <pinref part="IC1" gate="A" pin="VDD"/>
@@
 </segment>
 </net>
-<net name="+3V3" class="1">
+<net name="+3V3" class="0">
 <segment>
 <junction x="25.4" y="124.46"/>
@@
 </segment>
 </net>
-<net name="+3V3" class="1">
+<net name="+3V3" class="0">
 <segment>
 <pinref part="+3V1" gate="G$1" pin="+3V3"/>
@@
 </segment>
 </net>
-<net name="N$10" class="1">
+<net name="N$10" class="0">
 <segment>
 <wire x1="226.06" y1="104.14" x2="246.38" y2="104.14" width="0.1524" layer="91"/>
@@
 </segment>
 </net>
-<net name="+3V3" class="1">
+<net name="+3V3" class="0">
 <segment>
 <pinref part="+3V6" gate="G$1" pin="+3V3"/>
@@
 </segment>
 </net>
-<net name="+3V3" class="1">
+<net name="+3V3" class="0">
 <segment>
 <pinref part="WIFI" gate="G$1" pin="3.3V"/>

Commit message: Arduino shield renumbering
Parts:
- removed D8: SKL16, diode:DIODE-DO214AC
- removed JP1: 826926-2, jumper:JP1E
- removed JP2: 0R-JUMPA, jump-0r-smd:0R-JUMPA
- added D29: SKL16, EEZ_Lib1:SCHOTTKYSOD123
- added JP6, JP7: 0R-JUMPA, jump-0r-smd:0R-JUMPA
- JP3: value 0R-JUMPA -> 826926-2; device jump-0r-smd:0R-JUMPA -> jumper:JP1E
- LED_CC1, LED_CC2, LED_CV1, LED_CV2, LED_O1, LED_O2, LED_PROG1, LED_PROG2, LED_PWR, LED_S1, LED_S2, LED_SP: device led:LEDCHIPLED_0805 -> EEZ_Lib1:LED0805
- renumbered C1 to C105, C10 to C114, C11 to C115, C12 to C116, C13 to C117, C14 to C119, C15 to C118, C16 to C120, C17 to C121, C18 to C122, C19 to C123, C2 to C106, C20 to C124, C21 to C125, C22 to C126, C23 to C127, C24 to C128, C25 to C129, C26 to C130, C27 to C131, C28 to C132, C29 to C133, C3 to C107, C30 to C134, C31 to C135, C32 to C136, C33 to C137, C34 to C138, C35 to C139, C36 to C140, C37 to C141, C38 to C142, C39 to C143, C4 to C108, C40 to C144, C41 to C145, C42 to C146, C43 to C147, C44 to C148, C45 to C149, C46 to C150, C47 to C151, C48 to C152, C49 to C153, C5 to C109, C50 to C154, C51 to C155, C52 to C156, C53 to C157, C6 to C110, C7 to C111, C8 to C112, C9 to C113, D1 to D22, D2 to D23, D3 to D24, D4 to D25, D5 to D26, D6 to D27, D7 to D28, FB to FB8, IC1 to IC21, IC10 to IC30, IC11 to IC31, IC12 to IC32, IC13 to IC33, IC14 to IC34, IC15 to IC35, IC2 to IC22, IC3 to IC23, IC4 to IC24, IC5 to IC25, IC6 to IC26, IC7 to IC27, IC8 to IC28, IC9 to IC29, OK1 to OK3, Q1 to Q23, Q2 to Q24, Q3 to Q25, Q4 to Q26, Q5 to Q27, Q6 to Q28, Q7 to Q29, Q8 to Q30, R1 to R122, R10 to R131, R11 to R132, R12 to R133, R13 to R134, R14 to R135, R15 to R136, R16 to R137, R17 to R138, R18 to R139, R19 to R140, R2 to R123, R20 to R141, R21 to R142, R22 to R143, R23 to R144, R24 to R145, R25 to R146, R26 to R147, R27 to R148, R28 to R149, R29 to R150, R3 to R124, R30 to R151, R31 to R152, R32 to R153, R33 to R154, R34 to R155, R35 to R156, R36 to R157, R37 to R158, R38 to R159, R4 to R125, R5 to R126, R6 to R127, R7 to R128, R8 to R129, R9 to R130, SH1 to SH3, TP1 to TP3, TP2 to TP4, X1 to X12, X2 to X13, X3 to X14, X4 to X15, X5 to X16, X6 to X17, X7 to X18, X8 to X19, X9 to X20, ZD1 to ZD8, ZD2 to ZD9, ZD3 to ZD10, ZD4 to ZD11, ZD5 to ZD12
Connections:
- removed net N$10: JP2-0R.2, LCD1.VCC
- removed net N$16: JP4-0R.2, LCD1.T_DIN
- removed net N$18: JP3-0R.2, LCD1.T_CLK
- removed net N$2: JP5-0R.2, LCD1.T_DO
- removed net N$33: D8.C, R151.2
- removed net N$35: D8.A, FB8.2
- new net N$102: JP4-0R.2, LCD1.VCC
- new net N$104: JP7-0R.2, LCD1.T_DO
- new net N$105: JP5-0R.2, LCD1.T_CLK
- new net N$106: JP6-0R.2, LCD1.T_DIN
- new net N$148: D29.C, R151.2
- new net N$149: D29.A, FB8.2
- net !PWD_RST: now also JP3.1; no longer JP1.1
- net +3V3: now also JP4-0R.3; no longer JP2-0R.3
- net +5V: now also JP4-0R.1; no longer JP2-0R.1
- net ENC_A: now also MCU-ADCH.ADC8; no longer MCU-ADCH.ADC14
- net ENC_B: now also MCU-ADCH.ADC9; no longer MCU-ADCH.ADC15
- net GND: now also JP3.2; no longer JP1.2
- net MISO: now also JP7-0R.1; no longer JP5-0R.1
- net MOSI: now also JP6-0R.1; no longer JP4-0R.1
- net SCLK: now also JP5-0R.1; no longer JP3-0R.1
- net TOUCH_DIN: now also JP6-0R.3; no longer JP4-0R.3
- net TOUCH_DOUT: now also JP7-0R.3; no longer JP5-0R.3
- net TOUCH_SCLK: now also JP5-0R.3; no longer JP3-0R.3
Other:
- note added: "10-pin IDC connector X16"
- note added: "10-pin connector X20"
- note added: "26-pin SPI and power out socket (X13, X14)"
- note added: "4-pin connector X19"
- note added: "6-pin push-in connector X17"
- note added: "8-pin connector X18"
- note added: "8-pin push-in connector X18"
- note removed: "10-pin IDC connector X5"
- note removed: "10-pin connector X9"
- note removed: "26-pin SPI and power out socket (X2, X4)"
- note removed: "4-pin connector X8"
- note removed: "6-pin push-in connector X3"
- note removed: "8-pin connector X7"
- note removed: "8-pin push-in connector X1"

Commit message: PCB fiducials, outlines, milling bridges
Parts:
- added U$15, U$16: FIDUCIAL_2, EEZ_Lib1:FIDUCIAL_2
Other:
- note added: "Note 8.1: Solder X1 and X3 on the PCB's opposite side"
- note added: "See Note 8.1"
- note added: "Solder LCD1 socket on the PCB's opposite side"
- note removed: "Note 1.1: Solder X1 and X3 on the PCB's opposite side"
- note removed: "See Note 1.1"
- note removed: "Solder LCD1 on the PCB's opposite side"
Changed lines of the file:
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@@
 <layer number="112" name="tSilk" color="7" fill="1" visible="no" active="no"/>
 <layer number="113" name="ReferenceLS" color="7" fill="1" visible="yes" active="yes"/>
+<layer number="114" name="EEZ" color="7" fill="1" visible="yes" active="yes"/>
 <layer number="116" name="Patch_BOT" color="7" fill="1" visible="no" active="no"/>
 <layer number="118" name="Rect_Pads" color="7" fill="1" visible="no" active="no"/>
@@
 <part name="LED_SP" library="EEZ_Lib1" deviceset="LED" device="0805" value="HSMH-C170"/>
 <part name="SW2" library="EEZ_Lib1" deviceset="TACT_SW" device="" value="1301.9316"/>
+<part name="U$15" library="EEZ_Lib1" deviceset="FIDUCIAL" device="_2"/>
+<part name="U$16" library="EEZ_Lib1" deviceset="FIDUCIAL" device="_2"/>
 </parts>
 <sheets>
@@
 <text x="189.23" y="82.55" size="1.4224" layer="104">Require SPI_MODE0</text>
 <text x="2.54" y="2.54" size="1.778" layer="94">Licensed under the TAPR Open Hardware License (www.tapr.org/OHL)</text>
-<text x="104.14" y="2.54" size="1.4224" layer="103">Note 1.1: Solder X1 and X3 on the PCB's opposite side</text>
-<text x="78.74" y="147.32" size="1.4224" layer="103">See Note 1.1</text>
-<text x="76.2" y="66.04" size="1.4224" layer="103">See Note 1.1</text>
+<text x="104.14" y="2.54" size="1.4224" layer="103">Note 8.1: Solder X1 and X3 on the PCB's opposite side</text>
+<text x="78.74" y="147.32" size="1.4224" layer="103">See Note 8.1</text>
+<text x="76.2" y="66.04" size="1.4224" layer="103">See Note 8.1</text>
 <circle x="109.22" y="36.83" radius="0.635" width="0.1524" layer="101"/>
 <circle x="106.68" y="36.83" radius="0.635" width="0.1524" layer="101"/>
@@
 <attribute name="PART" x="146.05" y="114.3" size="1.778" layer="95"/>
 </instance>
+<instance part="U$15" gate="FD" x="157.48" y="12.7"/>
+<instance part="U$16" gate="FD" x="157.48" y="5.08"/>
 </instances>
 <busses>
@@
 <text x="5.08" y="116.84" size="1.778" layer="97">Ethernet</text>
 <text x="206.375" y="153.67" size="1.778" layer="103">Temp in</text>
-<text x="167.64" y="40.64" size="1.4224" layer="103">Solder LCD1 on the PCB's opposite side</text>
+<text x="167.64" y="40.64" size="1.4224" layer="103">Solder LCD1 socket on the PCB's opposite side</text>
 <text x="87.63" y="133.35" size="1.4224" layer="104">Require SPI_MODE0</text>
 <text x="26.67" y="133.35" size="1.4224" layer="104">Require SPI_MODE0</text>
