File: Arduino shield/Eagle files/EEZ PSU Arduino shield+BP r3B4.brd (EAGLE design)
At the start: 207 x 74 mm, 185 parts, among them IC20 TLC5925IDBQR, IC21 Si8641EC-B-IS1, IC22 SI8651EC-B-IS1, IC23 SI8651EC-B-IS1, IC24 LD1117ADT33TR, IC25 Si8641EC-B-IS1, IC26 PCA21125T/Q900/1,1, IC27 AT25256B-SSHL-B, IC28 W5500, IC29 BC857BS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

Commit message: AUX PS r5B9
Other:
- board text added: "(0.75")"
- board text added: "M3 studs (4 pcs for display support)"
