File: Arduino shield/Eagle files/EEZ PSU Arduino shield+BP r3B4.sch (EAGLE design)
At the start: 181 parts, among them IC20 TLC5925IDBQR, IC21 Si8641EC-B-IS1, IC22 SI8651EC-B-IS1, IC23 SI8651EC-B-IS1, IC24 LD1117ADT33TR, IC25 Si8641EC-B-IS1, IC26 PCA21125T/Q900/1,1, IC27 AT25256B-SSHL-B, IC28 W5500, IC29 BC857BS, IC30 TLC555, IC31 SN74LVC2G08DCTR, IC32 TPS3705-33D, IC33 SN74LV1T34DBVR, IC34 SN74LVC2G02DCTR, J1 BS-244DSM-R, J2 BS-244DSM-G, J3 BS-244DSM-B, J4 BS-244DSM-R, J5 BS-244DSM-B, Q23 IRLML2246TRPBF, Q24 IRLML2246TRPBF, Q25 IRLML2246TRPBF, Q26 IRLML2246TRPBF, Q27 2N7002, Q28 IRLML2246TRPBF, Q29 2N7002, Q30 2N7002, SW1 A101SYCQ04, SW2 1301.9316, X12 MC000006, X13 TSW-113-07-F-D, X14 MC000005, X15 TSW-113-07-F-D, X16 09185067324, X17 22-23-2021, X18 826629-8, X19 22-23-2041, X20 SSW-105-02-S-D, Y1 32,768kHz, Y2 25MHz

Commit message: X18 type changed
Parts:
- X18: value 826629-8 -> MC34753
Changed lines of the file:
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@@
 <part name="OK3" library="EEZ_Lib1" deviceset="HCPL-181" device=""/>
 <part name="R159" library="rcl" deviceset="R-EU_" device="R0805" value="1K8"/>
-<part name="X18" library="con-samtec" deviceset="SSW-108-02-S-S" device="" value="826629-8">
+<part name="X18" library="con-samtec" deviceset="SSW-108-02-S-S" device="" value="MC34753">
 <attribute name="MPN" value="SSW-108-02-S-S"/>
 <attribute name="OC_NEWARK" value="11P9448"/>
