File: Aux power/Eagle files/EEZ AUX PS r4B41.sch (EAGLE design)
At the start: 66 parts, among them IC1 LM25575, IC2 UA78M12DCY, IC3 TPD4E002DRLR, IC4 TPD2E001DZDR, Q1 BTA26-600, Q2 BTA26-600, Q3 IRLL014N, X1 282836-5, X2 09185067324, X3 22-23-2031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

Commit message: Arduino Shield r1B14, AUX PS r4B41
Parts:
- removed C16: 100n, rcl:C-EUC0805
- removed IC3: TPD4E002DRLR, EEZ_Lib1:TPD4E002DRLR
- removed IC4: TPD2E001DZDR, EEZ_Lib1:TPD2E001DZDR
- removed L4: 470u, EEZ_Lib1:DE0704
- removed R19: 0R, rcl:R-EU_R0805
- removed X5: LMJ2138812S0LOT6C, EEZ_Lib1:RJ45-VERT
- removed X6: 826629-8, con-samtec:SSW-108-02-S-S
- removed X7: 826629-5, con-samtec:SSW-105-02-S-S
- removed X8: 2411-01, con-kycon:KUSBVX-BS1N
- added JP1: (no value), jumper:JP1E
- L3: value 60R@100MHz -> 470u; device MyLib6:FERRITE_BEAD0603 -> EEZ_Lib1:DE0704
Connections:
- removed net +3V3: L3.2, X6-8.1
- removed net ETH_ACTLED: X5.YELLOW_A, X6-2.1
- removed net ETH_IN+: IC3.IO4, X5.RD-, X6-4.1
- removed net ETH_IN-: IC3.IO3, X5.RD+, X6-5.1
- removed net ETH_LINKLED: X5.GREEN-A, X6-1.1
- removed net ETH_OUT+: IC3.IO2, X5.TD-, X6-6.1
- removed net ETH_OUT-: IC3.IO1, X5.TD+, X6-7.1
- removed net N$11: C16.2, IC4.VCC, X7-1.1, X8.1
- removed net N$125: L3.1, X5.CT
- removed net N$14: R19.2, X7-5.1
- removed net N$18: IC4.IO1, X7-2.1, X8.2
- removed net N$22: IC4.IO2, X7-3.1, X8.3
- removed net N$23: C16.1, IC4.GND, X7-4.1, X8.4
- new net N$10: JP1.1, R18.1
- net AC_EARTH: no longer R19.1, X5.SH, X8.S1, X8.S2
- net FAN_OUT: now also L3.2; no longer L4.2
- net FAN_SENSE: now also JP1.2; no longer R18.1
- net GND: no longer IC3.GND, X5.GREEN-C, X5.YELLOW-C
- net N$21: now also L3.1; no longer L4.1
Other:
- note added: "Note 2.1: Remove jumper if 5 V logic output is required"
- note added: "See note 2.1"
- note removed: "+3.3V (Input) 8"
- note removed: "12VDC fan control"
- note removed: "5-pin connector X7"
- note removed: "8-pin connector X6"
- note removed: "Data+ 3"
- note removed: "Data- 2"
- note removed: "Ethernet and USB PCB connectors"
- note removed: "Ethernet and USB connectors with optional surge protection"
- note removed: "Gnd 4"
- note removed: "LED Act (Input) 2"
- note removed: "LED Link (Input) 1"
- note removed: "Note 2.1: Mount X5 and X8 on the opposite (top) side of the PCB. Use 14 mm (e.g. Bossard B3X14/BN3320) for enclosure with 3 mm rear panel"
- note removed: "RX+ (Output) 4"
- note removed: "RX- (Output) 5"
- note removed: "Shield 3"
- note removed: "Shield 5"
- note removed: "TX+ (Input) 6"
- note removed: "TX- (Input) 7"
- note removed: "Vcc 1"
- moved on the sheet: C14, C15, D2, IC2, L3, Q3, R14, R15, R16, R17, R18, X2-3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
