File: Aux power/Eagle files/EEZ AUX PS r4B43.brd (EAGLE design)
At the start: 68 x 100 mm, 62 parts, among them IC1 LM25575, IC2 MC7812, Q1 BTA26-600, Q2 BTA26-600, Q3 IRLL014N, X1 282836-5, X2 09185067324, X3 22-23-2031, X4 22-23-2031

Commit message: AUX PS r4B3, various BOM corrections
Parts:
- C13: value 180p -> n.c.
- JP1: value (none) -> 826926-2
- TR1: value TEZ6/D230/15V -> TEZ6/D230/12V
Connections:
- removed net N$25: Q1.A2, R1.2, R2.1
- new net N$11: Q1.A2, R1.2, R2.1, R5.2
- net AC_IN1: no longer R3.2, R5.2
- net N$8: now also R3.2
Routing:
- net N$11: track 0.00 -> 61.3 mm
- net N$25: track 39.5 -> 0.00 mm
- net AC_IN1: track 173.6 -> 143.2 mm
- net N$8: track 82.5 -> 102.8 mm, vias 0 -> 1
- net N$4: track 32.8 -> 34.5 mm
Other:
- board text added: "EEZ AUX PS (05/2016) r4B43"
- board text added: "r4B43"
- board text removed: "EEZ AUX PS (05/2016) r4B42"
- board text removed: "r4B42"
