File: Mechanical/EEZ PSU enclosure (Economica 320x200x115, Arduino shield r1b14).brd (EAGLE design)
At the start: 350 x 600 mm, 0 parts

Commit message: Rubber feet added in Arduino shield BOM
Other:
- board size 350 x 600 mm -> 710 x 425 mm
- board text added: "Holes for screw fastened rubber feet e.g. TME: RI-SOF-15129"
