File: Panelized/Eagle files/PCB panel M1 (2016-05-26).brd (EAGLE design)
At the start: 246 x 207 mm, 726 parts, among them IC1 LM25575, IC10 SN74LV125APW, IC11 SI8620EC-B-IS, IC12 SI8620EC-B-IS, IC13 Si8660EC-B-IS1, IC14 PCA21125, IC15 AT25256B, IC16 ENC28J60-I/SS, IC17 BC857BS, IC18 NE555D, IC19 BC857BS, IC2 TLC5925, IC20 NE555D, IC21 DAC8552, IC22 ADS1120, IC23 MCP23S08-E/SO, IC24 LP339D, IC25 OP27GSZ, IC26 TL072D, IC27 TL072D, IC28 REF5025, IC29 DAC8552, IC3 SN74LVCC3245ADBRSSOP, IC30 ADS1120, IC31 MCP23S08-E/SO, IC32 LP339D, IC33 OP27GSZ, IC34 TL072D, IC35 TL072D, IC36 REF5025, IC37 LP2951SO8, IC38 LM337LZ, IC39 Si8610BC-B-IS, IC4 SN74LVCC3245ADBRSSOP, IC40 LP2951SO8, IC41 TLC555, IC42 LM5574, IC43 LP2951SO8, IC44 LM337LZ, IC45 Si8610BC-B-IS, IC46 LP2951SO8, IC47 TLC555, IC48 LM5574, IC49 SN74LVCC3245ADBRSSOP, IC5 SN74LVCC3245ADBRSSOP, IC50 SN74LV1T34, IC51 UA78M12DCY, IC6 LD1117ADT33TR, IC7 SN74LVCC3245ADBRSSOP, IC8 SN74LVCC3245ADBRSSOP, IC9 Si8660EC-B-IS1, J1 BS-244DSM-R, J2 BS-244DSM-B, J3 BS-244DSM-R, J4 BS-244DSM-G, J5 BS-244DSM-B, P1 500K, P2 500K, Q1 BTA26-600, Q10 2N7002, Q11 2N7002, Q12 2N7002, Q13 2N7002, Q14 IRFP250N, Q15 BCP56-16.115, Q16 MMBT5551, Q17 BC846C, Q18 BCP56-16.115, Q19 MMBT5401, Q2 BTA26-600, Q20 MMBT5401, Q21 MMBT5551, Q22 BC857C, Q23 2N7002, Q24 2N7002, Q25 2N7002, Q26 BSS84P, Q27 IRF9640, Q28 IRFP250N, Q29 BCP56-16.115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

Commit message: AUX PS r4B3, various BOM corrections
Parts:
- C1: value 180p -> n.c.
- C11: value 820p -> 1n
- IC51: value UA78M12DCY -> MC7812; device EEZ_Lib1:SOT230P700X180-4N -> EEZ_Lib1:TO252
- JP7: value (none) -> 826926-2
- TR3: value TEZ6/D230/15V -> TEZ6/D230/12V
- VAR1, VAR2: value *** -> S20K250
- moved IC51 1.53 mm to (-0.68, 100.2), turned to 90 degrees
Connections:
- removed net N$257 (its old number): Q1.A2, R1.2, R2.1
- new net N$258: Q1.A2, R1.2, R2.1, R5.2
- net AC_IN1: no longer R3.2, R5.2
- net GND: now also IC51.3; no longer IC51.2, IC51.4
- net N$17: now also R3.2
- net N$30: now also IC51.2; no longer IC51.3
Routing:
- net N$258: track 0.00 -> 61.3 mm
- net N$257 (its old number): track 39.5 -> 0.00 mm
- net AC_IN1: track 173.6 -> 143.2 mm
- net N$17: track 82.5 -> 102.8 mm, vias 0 -> 1
- net N$20: track 32.8 -> 34.5 mm
- net N$30: track 110.0 -> 110.7 mm
Other:
- board text added: "(05/2016)"
- board text added: "EEZ AUX PS (05/2016) r4B43"
- board text added: "r4B43"
- board text removed: "(04/2016)"
- board text removed: "EEZ AUX PS (04/2016) r4B41"
- board text removed: "r4B41"
