File: Power board/Eagle files/EEZ PSU power board r5B8.sch (EAGLE design)
At the start: 266 parts, among them IC1 LTC3864, IC10 REF5025, IC11 DAC8552, IC12 ADG465SOT-23, IC13 TS5A9411DCKT, IC14 ADS1120, IC15 LP339D, IC2 MC79L05, IC3 MC78L05, IC4 LM5574, IC5 LP2951SO8, IC6 TL072D, IC7 TL072D, IC8 OP27GSZ, IC9 MCP23S08-E/SO, Q1 SUD19P06-60, Q10 MMBT5401, Q11 MMBT5401, Q12 MMBT5551, Q13 MMBT5551, Q14 BSS84P, Q15 2N7002, Q16 MMBT5551, Q17 MMBT5401, Q18 MMBT5551, Q19 MMBT5551, Q2 MMBT5401, Q3 2N7002, Q4 IRFP250N, Q5 BC857C, Q6 BC846C, Q7 BCP56-16.115, Q8 IRFR5410, Q9 BCP56-16.115, X1 282836-3, X2 282836-2, X3 SSW-113-02-T-D-RA

Commit message: Power board R28, R29
Parts:
- R28: value 0R1/3W -> R080/3W; device EEZ_Lib1:R_EUCOMBO -> rcl:R-EU_R2512
- R29: device EEZ_Lib1:R_EUCOMBO -> rcl:R-EU_R2512
- TR1: value MSD1260-824 -> SRF0703-821M
Changed lines of the file:
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@@
 <setting verticaltext="up"/>
 </settings>
-<grid distance="0.1" unitdist="inch" unit="inch" style="lines" multiple="1" display="no" altdistance="0.01" altunitdist="inch" altunit="inch"/>
+<grid distance="0.025" unitdist="inch" unit="inch" style="lines" multiple="1" display="no" altdistance="0.01" altunitdist="inch" altunit="inch"/>
 <layers>
 <layer number="1" name="Top" color="4" fill="1" visible="no" active="no"/>
@@
 <part name="SUPPLY30" library="supply2" deviceset="GND" device="" value="PGND"/>
 <part name="X2" library="EEZ_Lib1" deviceset="TBLOCK5.0_2A" device="" value="282836-2"/>
-<part name="R28" library="EEZ_Lib1" deviceset="R_EU" device="COMBO" value="0R1/3W"/>
-<part name="R29" library="EEZ_Lib1" deviceset="R_EU" device="COMBO" value="2R2/2W"/>
 <part name="C5" library="EEZ_Lib1" deviceset="ECAP" device="7.5G_18MM" value="2m2"/>
 <part name="R3" library="rcl" deviceset="R-EU_" device="R0805" value="0R"/>
@@
 <part name="SW" library="EEZ_Lib1" deviceset="PCB_TEST_TAB" device="SMD" value="S1751-46R"/>
 <part name="GND" library="EEZ_Lib1" deviceset="PCB_TEST_TAB" device="SMD" value="S1751-46R"/>
-<part name="TR1" library="EEZ_Lib1" deviceset="BOURNS_SRF0703INV" device="" value="MSD1260-824"/>
+<part name="TR1" library="EEZ_Lib1" deviceset="BOURNS_SRF0703INV" device="" value="SRF0703-821M"/>
 <part name="R83" library="rcl" deviceset="R-EU_" device="R0805" value="330R"/>
 <part name="Q19" library="transistor" deviceset="*-NPN-" device="SOT23-BEC" technology="MMBT5551LT1" value="MMBT5551"/>
@@
 <part name="L1" library="EEZ_Lib1" deviceset="RN114" device="" value="RN114-4/02"/>
 <part name="C18" library="EEZ_Lib1" deviceset="ECAP" device="F" value="EEEFK1J470P"/>
+<part name="R28" library="rcl" deviceset="R-EU_" device="R2512" value="R080/3W"/>
+<part name="R29" library="rcl" deviceset="R-EU_" device="R2512" value="2R2/2W"/>
 </parts>
 <sheets>
@@
 <attribute name="NAME" x="471.17" y="67.691" size="1.778" layer="95"/>
 </instance>
-<instance part="R28" gate="G$1" x="345.44" y="76.2" smashed="yes">
-<attribute name="NAME" x="341.63" y="77.6986" size="1.778" layer="95"/>
-<attribute name="VALUE" x="341.63" y="72.898" size="1.778" layer="96"/>
-</instance>
-<instance part="R29" gate="G$1" x="386.08" y="71.12" smashed="yes" rot="R90">
-<attribute name="NAME" x="387.35" y="72.6186" size="1.778" layer="95"/>
-<attribute name="VALUE" x="387.35" y="70.358" size="1.778" layer="96"/>
-</instance>
 <instance part="ZD3" gate="G$1" x="449.58" y="66.04" smashed="yes" rot="R270">
 <attribute name="NAME" x="448.31" y="65.405" size="1.778" layer="95" rot="R180"/>
@@
 <attribute name="VALUE" x="350.52" y="-84.455" size="1.6764" layer="96"/>
 </instance>
+<instance part="R28" gate="G$1" x="345.44" y="76.2" smashed="yes">
+<attribute name="NAME" x="342.9" y="73.2536" size="1.778" layer="95"/>
+<attribute name="VALUE" x="342.9" y="70.993" size="1.778" layer="96"/>
+</instance>
+<instance part="R29" gate="G$1" x="386.08" y="71.12" smashed="yes" rot="R90">
+<attribute name="NAME" x="387.35" y="73.4314" size="1.778" layer="95" rot="MR180"/>
+<attribute name="VALUE" x="387.35" y="69.723" size="1.778" layer="96"/>
+</instance>
 </instances>
 <busses>
@@
 <wire x1="464.82" y1="76.2" x2="462.28" y2="76.2" width="0.1524" layer="91"/>
 <junction x="462.28" y="76.2"/>
-<pinref part="R28" gate="G$1" pin="2"/>
-<pinref part="R29" gate="G$1" pin="2"/>
-<junction x="386.08" y="76.2"/>
 <pinref part="ZD3" gate="G$1" pin="1"/>
 <wire x1="449.58" y1="68.58" x2="449.58" y2="76.2" width="0.1524" layer="91"/>
@@
 <wire x1="464.82" y1="55.88" x2="462.28" y2="55.88" width="0.1524" layer="91"/>
 <junction x="462.28" y="55.88"/>
+<pinref part="R28" gate="G$1" pin="2"/>
+<pinref part="R29" gate="G$1" pin="2"/>
+<junction x="386.08" y="76.2"/>
 </segment>
 </net>

Commit message: Rt value corrections for AUX PS and Power board
Parts:
- R22: value 18K -> 20K
Changed lines of the file:
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@@
 <setting verticaltext="up"/>
 </settings>
-<grid distance="0.025" unitdist="inch" unit="inch" style="lines" multiple="1" display="no" altdistance="0.01" altunitdist="inch" altunit="inch"/>
+<grid distance="0.1" unitdist="inch" unit="inch" style="lines" multiple="1" display="no" altdistance="0.01" altunitdist="inch" altunit="inch"/>
 <layers>
 <layer number="1" name="Top" color="4" fill="1" visible="no" active="no"/>
@@
 <part name="LED1" library="led" deviceset="LED" device="CHIPLED_0805" value="HSMY-C170"/>
 <part name="C39" library="rcl" deviceset="C-EU" device="C0805" value="3n3"/>
-<part name="R22" library="rcl" deviceset="R-EU_" device="R0805" value="18K"/>
+<part name="R22" library="rcl" deviceset="R-EU_" device="R0805" value="20K"/>
 <part name="R23" library="rcl" deviceset="R-EU_" device="R0805" value="51K"/>
 <part name="C40" library="rcl" deviceset="C-EU" device="C0805" value="1n"/>
