File: Consolidated/EEZ PSU consolidated r5B8.sch (EAGLE design)
At the start: 519 parts, among them IC1 LTC3864, IC10 REF5025, IC11 DAC8552, IC12 ADG465SOT-23, IC13 TS5A9411DCKT, IC14 ADS1120, IC15 LP339D, IC16 LM25575, IC17 MC7812, IC18 TPD4E002DRLR, IC19 TPD2E001DZDR, IC2 MC79L05, IC20 ADUM3160BRWZ, IC21 TLC5925IDBQR, IC22 Si8641EC-B-IS1, IC23 SI8651EC-B-IS1, IC24 SI8651EC-B-IS1, IC25 LD1117ADT33TR, IC26 Si8641EC-B-IS1, IC27 PCA21125, IC28 AT25256B, IC29 W5500, IC3 MC78L05, IC30 BC857BS, IC31 TLC555, IC32 SN74LVC2G08DCTR, IC33 TPS3705-33D, IC34 SN74LV1T34DBVR, IC35 SN74LVC2G02DCTR, IC4 LM5574, IC5 LP2951SO8, IC6 TL072D, IC7 TL072D, IC8 OP27GSZ, IC9 MCP23S08-E/SO, J1 BS-244DSM-R, J2 BS-244DSM-G, J3 BS-244DSM-B, J4 BS-244DSM-R, J5 BS-244DSM-B, Q1 SUD19P06-60, Q10 MMBT5401, Q11 MMBT5401, Q12 MMBT5551, Q13 MMBT5551, Q14 BSS84P, Q15 2N7002, Q16 MMBT5551, Q17 MMBT5401, Q18 MMBT5551, Q19 MMBT5551, Q2 MMBT5401, Q20 BTA26-600, Q21 BTA26-600, Q22 IRLL014N, Q23 IRLML2246TRPBF, Q24 IRLML2246TRPBF, Q25 IRLML2246TRPBF, Q26 IRLML2246TRPBF, Q27 2N7002, Q28 IRLML2246TRPBF, Q29 2N7002, Q3 2N7002, Q30 2N7002, Q4 IRFP250N, Q5 BC857C, Q6 BC846C, Q7 BCP56-16.115, Q8 IRFR5410, Q9 BCP56-16.115, SW1 A101SYCQ04, SW2 1301.9316, X1 282836-3, X10 826629-5, X11 2411-01, X12 MC000006, X13 TSW-113-07-F-D, X14 MC000005, X15 TSW-113-07-F-D, X16 09185067324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

Commit message: PCB fiducials, outlines, milling bridges
Parts:
- added U$11, U$12, U$13, U$14, U$15, U$16: FIDUCIAL_2, EEZ_Lib1:FIDUCIAL_2
- TR2: device EEZ_Lib1:PCB_TRAFO6VA_TEZ+VPP -> EEZ_Lib1:PCB_TRAFO6VA_TEZ+VPP+MYRRA
Other:
- note added: "Digikey: 237-1085-ND"
- note added: "Farnell: 2469211"
- note added: "Mouser: 553-VPP24-210"
- note added: "Myrra 47202"
- note added: "Newark: 93F8764"
- note added: "Note 7.1: Mount X4 and X8 on the opposite (top) side of the PCB. Use 14 mm (e.g. Bossard B3X14/BN3320) for enclosure with 3 mm rear panel"
- note added: "Note 8.1: Solder X1 and X3 on the PCB's opposite side"
- note added: "See Note 8.1"
- note added: "Solder LCD1 socket on the PCB's opposite side"
- note added: "TR2"
- note added: "VPP24-210"
- note added: "or AC/DC module"
- note removed: "Digikey: 237-1086-ND"
- note removed: "Mouser: 553-VPP28-180"
- note removed: "Newark: 37B9209"
- note removed: "Note 1.1: Solder X1 and X3 on the PCB's opposite side"
- note removed: "Note 2.1: Mount X4 and X8 on the opposite (top) side of the PCB. Use 14 mm (e.g. Bossard B3X14/BN3320) for enclosure with 3 mm rear panel"
- note removed: "Solder LCD1 on the PCB's opposite side"
- note removed: "TR1"
- note removed: "VPP28-180"
Changed lines of the file:
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@@
 <layer number="112" name="tSilk" color="7" fill="1" visible="no" active="no"/>
 <layer number="113" name="ReferenceLS" color="7" fill="1" visible="yes" active="yes"/>
+<layer number="114" name="EEZ" color="7" fill="1" visible="yes" active="yes"/>
 <layer number="116" name="Patch_BOT" color="7" fill="1" visible="no" active="no"/>
 <layer number="118" name="Rect_Pads" color="7" fill="1" visible="no" active="no"/>
@@
 <part name="R119" library="rcl" deviceset="R-EU_" device="R0805" value="10K"/>
 <part name="SUPPLY51" library="supply2" deviceset="GND" device=""/>
-<part name="TR2" library="EEZ_Lib1" deviceset="PCB_TRAFO6VA_TEZ+VPP" device="" value="TEZ6/D230/15V"/>
+<part name="TR2" library="EEZ_Lib1" deviceset="PCB_TRAFO6VA_TEZ+VPP" device="+MYRRA" value="TEZ6/D230/15V"/>
 <part name="VAR1" library="EEZ_Lib1" deviceset="VARISTOR" device="" value="S20K250"/>
 <part name="VAR2" library="EEZ_Lib1" deviceset="VARISTOR" device="" value="S20K250"/>
@@
 <part name="D21" library="diode" deviceset="DIODE-" device="SOD323-W" value="BAS316"/>
 <part name="C97" library="MyLib6" deviceset="ECAP" device="PANASONIC_C" value="10u"/>
+<part name="U$11" library="EEZ_Lib1" deviceset="FIDUCIAL" device="_2"/>
+<part name="U$12" library="EEZ_Lib1" deviceset="FIDUCIAL" device="_2"/>
+<part name="U$13" library="EEZ_Lib1" deviceset="FIDUCIAL" device="_2"/>
+<part name="U$14" library="EEZ_Lib1" deviceset="FIDUCIAL" device="_2"/>
+<part name="U$15" library="EEZ_Lib1" deviceset="FIDUCIAL" device="_2"/>
+<part name="U$16" library="EEZ_Lib1" deviceset="FIDUCIAL" device="_2"/>
 </parts>
 <sheets>
@@
 <instance part="L1" gate="-2" x="58.42" y="162.56"/>
 <instance part="L1" gate="-1" x="58.42" y="170.18"/>
+<instance part="U$11" gate="FD" x="157.48" y="5.08"/>
+<instance part="U$12" gate="FD" x="149.86" y="5.08"/>
 </instances>
 <busses>
@@
 <text x="6.985" y="176.53" size="1.778" layer="97" rot="MR180">AC input protection and soft-start/stand-by</text>
 <text x="10.16" y="157.48" size="1.778" layer="103">AC input (230V)</text>
-<text x="9.525" y="34.925" size="1.6764" layer="103">SAR1</text>
-<text x="9.525" y="24.765" size="1.6764" layer="103">VAR1, VAR2</text>
-<text x="9.525" y="22.225" size="1.6764" layer="103">ZD1, ZD2</text>
+<text x="6.985" y="34.925" size="1.6764" layer="103">SAR1</text>
+<text x="6.985" y="19.685" size="1.6764" layer="103">VAR1, VAR2</text>
+<text x="6.985" y="17.145" size="1.6764" layer="103">ZD1, ZD2</text>
 <text x="44.45" y="38.1" size="1.6764" layer="103">Code</text>
-<text x="26.67" y="38.1" size="1.6764" layer="103">Value</text>
-<text x="26.67" y="34.925" size="1.6764" layer="103">2027-23-BLF</text>
+<text x="24.13" y="38.1" size="1.6764" layer="103">Value</text>
+<text x="24.13" y="34.925" size="1.6764" layer="103">2027-23-BLF</text>
 <text x="44.45" y="34.925" size="1.6764" layer="103">Farnell: 1780455, TME: CG2-230L</text>
-<text x="26.67" y="24.765" size="1.6764" layer="103">S20K140</text>
-<text x="26.67" y="32.385" size="1.6764" layer="103">VPP28-180</text>
-<text x="44.45" y="27.305" size="1.6764" layer="103">Newark: 37B9209</text>
-<text x="44.45" y="24.765" size="1.6764" layer="103">Farnell: 1004387, TME: SIOV-S20K140</text>
-<wire x1="7.62" y1="40.64" x2="25.4" y2="40.64" width="0.1524" layer="103"/>
-<wire x1="25.4" y1="40.64" x2="43.18" y2="40.64" width="0.1524" layer="103"/>
+<text x="24.13" y="19.685" size="1.6764" layer="103">S20K140</text>
+<text x="24.13" y="32.385" size="1.6764" layer="103">VPP24-210</text>
+<text x="44.45" y="19.685" size="1.6764" layer="103">Farnell: 1004387, TME: SIOV-S20K140</text>
+<wire x1="5.08" y1="40.64" x2="22.86" y2="40.64" width="0.1524" layer="103"/>
+<wire x1="22.86" y1="40.64" x2="43.18" y2="40.64" width="0.1524" layer="103"/>
 <wire x1="43.18" y1="40.64" x2="87.63" y2="40.64" width="0.1524" layer="103"/>
 <wire x1="87.63" y1="40.64" x2="87.63" y2="37.465" width="0.1524" layer="103"/>
-<wire x1="87.63" y1="37.465" x2="87.63" y2="21.59" width="0.1524" layer="103"/>
-<wire x1="87.63" y1="21.59" x2="43.18" y2="21.59" width="0.1524" layer="103"/>
-<wire x1="43.18" y1="21.59" x2="25.4" y2="21.59" width="0.1524" layer="103"/>
-<wire x1="25.4" y1="21.59" x2="7.62" y2="21.59" width="0.1524" layer="103"/>
-<wire x1="7.62" y1="21.59" x2="7.62" y2="37.465" width="0.1524" layer="103"/>
-<wire x1="7.62" y1="37.465" x2="7.62" y2="40.64" width="0.1524" layer="103"/>
-<wire x1="25.4" y1="21.59" x2="25.4" y2="40.64" width="0.1524" layer="103"/>
-<wire x1="43.18" y1="21.59" x2="43.18" y2="40.64" width="0.1524" layer="103"/>
-<wire x1="7.62" y1="37.465" x2="87.63" y2="37.465" width="0.1524" layer="103"/>
-<text x="9.525" y="38.1" size="1.6764" layer="103">Name</text>
-<text x="6.985" y="41.91" size="1.6764" layer="103">115VAC option:</text>
-<text x="9.525" y="32.385" size="1.6764" layer="103">TR1</text>
-<text x="26.67" y="22.225" size="1.6764" layer="103">1.5KE200CA</text>
-<text x="44.45" y="22.225" size="1.6764" layer="103">Farnell: 1837117, TME: 1.5KE200CA</text>
-<text x="44.45" y="32.385" size="1.6764" layer="103">Digikey: 237-1086-ND</text>
-<text x="44.45" y="29.845" size="1.6764" layer="103">Mouser: 553-VPP28-180</text>
+<wire x1="87.63" y1="37.465" x2="87.63" y2="16.51" width="0.1524" layer="103"/>
+<wire x1="87.63" y1="16.51" x2="43.18" y2="16.51" width="0.1524" layer="103"/>
+<wire x1="43.18" y1="16.51" x2="22.86" y2="16.51" width="0.1524" layer="103"/>
+<wire x1="22.86" y1="16.51" x2="5.08" y2="16.51" width="0.1524" layer="103"/>
+<wire x1="5.08" y1="16.51" x2="5.08" y2="37.465" width="0.1524" layer="103"/>
+<wire x1="5.08" y1="37.465" x2="5.08" y2="40.64" width="0.1524" layer="103"/>
+<wire x1="22.86" y1="16.51" x2="22.86" y2="40.64" width="0.1524" layer="103"/>
+<wire x1="43.18" y1="16.51" x2="43.18" y2="40.64" width="0.1524" layer="103"/>
+<wire x1="5.08" y1="37.465" x2="87.63" y2="37.465" width="0.1524" layer="103"/>
+<text x="6.985" y="38.1" size="1.6764" layer="103">Name</text>
+<text x="4.445" y="41.91" size="1.6764" layer="103">115VAC option:</text>
+<text x="6.985" y="32.385" size="1.6764" layer="103">TR2</text>
+<text x="24.13" y="17.145" size="1.6764" layer="103">1.5KE200CA</text>
+<text x="44.45" y="17.145" size="1.6764" layer="103">Farnell: 1837117, TME: 1.5KE200CA</text>
 <circle x="232.41" y="67.31" radius="0.635" width="0.1524" layer="101"/>
 <circle x="232.41" y="69.85" radius="0.635" width="0.1524" layer="101"/>
@@
 <text x="2.54" y="152.4" size="1.4224" layer="103">or Schurter KM00.1105.11 IEC intlet</text>
 <text x="2.54" y="149.86" size="1.4224" layer="103">with Schurter 4301.1403 fuse drawer</text>
+<text x="44.45" y="22.225" size="1.6764" layer="103">Farnell: 2469211</text>
+<text x="44.45" y="32.385" size="1.6764" layer="103">Digikey: 237-1085-ND</text>
+<text x="44.45" y="29.845" size="1.6764" layer="103">Mouser: 553-VPP24-210</text>
+<text x="24.13" y="24.765" size="1.6764" layer="103">or AC/DC module</text>
+<text x="44.45" y="27.305" size="1.6764" layer="103">Newark: 93F8764</text>
+<text x="24.13" y="22.225" size="1.6764" layer="103">Myrra 47202</text>
 </plain>
 <instances>
@@
 <attribute name="NAME" x="199.39" y="143.891" size="1.778" layer="95"/>
 </instance>
+<instance part="U$13" gate="FD" x="149.86" y="5.08"/>
+<instance part="U$14" gate="FD" x="157.48" y="5.08"/>
 </instances>
 <busses>
@@
 <wire x1="177.8" y1="38.1" x2="177.8" y2="81.28" width="0.1524" layer="97" style="shortdash"/>
 <wire x1="177.8" y1="81.28" x2="157.48" y2="81.28" width="0.1524" layer="97" style="shortdash"/>
-<text x="6.985" y="13.97" size="1.27" layer="103">Note 2.1: Mount X4 and X8 on the opposite (top) side of the PCB. Use 14 mm (e.g. Bossard B3X14/BN3320) for enclosure with 3 mm rear panel</text>
+<text x="6.985" y="13.97" size="1.27" layer="103">Note 7.1: Mount X4 and X8 on the opposite (top) side of the PCB. Use 14 mm (e.g. Bossard B3X14/BN3320) for enclosure with 3 mm rear panel</text>
 <text x="164.465" y="29.845" size="2.54" layer="94" font="vector">Ethernet and USB PCB connectors</text>
 <text x="164.465" y="26.035" size="2.54" layer="94" font="vector">12VDC fan driver (max. 300 mA)</text>
@@
 <text x="189.23" y="82.55" size="1.4224" layer="104">Require SPI_MODE0</text>
 <text x="2.54" y="2.54" size="1.778" layer="94">Licensed under the TAPR Open Hardware License (www.tapr.org/OHL)</text>
-<text x="104.14" y="2.54" size="1.4224" layer="103">Note 1.1: Solder X1 and X3 on the PCB's opposite side</text>
-<text x="78.74" y="147.32" size="1.4224" layer="103">See Note 1.1</text>
-<text x="76.2" y="66.04" size="1.4224" layer="103">See Note 1.1</text>
+<text x="104.14" y="2.54" size="1.4224" layer="103">Note 8.1: Solder X1 and X3 on the PCB's opposite side</text>
+<text x="78.74" y="147.32" size="1.4224" layer="103">See Note 8.1</text>
+<text x="76.2" y="66.04" size="1.4224" layer="103">See Note 8.1</text>
 <circle x="109.22" y="36.83" radius="0.635" width="0.1524" layer="101"/>
 <circle x="106.68" y="36.83" radius="0.635" width="0.1524" layer="101"/>
@@
 <attribute name="PART" x="146.05" y="114.3" size="1.778" layer="95"/>
 </instance>
+<instance part="U$15" gate="FD" x="157.48" y="12.7"/>
+<instance part="U$16" gate="FD" x="157.48" y="5.08"/>
 </instances>
 <busses>
@@
 <text x="5.08" y="116.84" size="1.778" layer="97">Ethernet</text>
 <text x="206.375" y="153.67" size="1.778" layer="103">Temp in</text>
-<text x="167.64" y="40.64" size="1.4224" layer="103">Solder LCD1 on the PCB's opposite side</text>
+<text x="167.64" y="40.64" size="1.4224" layer="103">Solder LCD1 socket on the PCB's opposite side</text>
 <text x="87.63" y="133.35" size="1.4224" layer="104">Require SPI_MODE0</text>
 <text x="26.67" y="133.35" size="1.4224" layer="104">Require SPI_MODE0</text>
