File: Consolidated/Eagle files/EEZ PSU r5B9 panel.brd (EAGLE design)
At the start: 309 x 150 mm, 822 parts, among them IC1 LTC3864EMSE#PBF, IC10 REF5025AIDG4, IC11 DAC8552IDGKTG4, IC12 ADG465SOT-23, IC13 TS5A9411DCKT, IC14 ADS1120IPWR, IC15 LP339D, IC16 LM25575MH/NOPB, IC17 TPD4E002DRLR, IC18 TPD2E001DZDR, IC19 ADUM3160BRWZ, IC2 MC79L05, IC20 TLC5925IDBQR, IC21 Si8641EC-B-IS1, IC22 SI8651EC-B-IS1, IC23 SI8651EC-B-IS1, IC24 LD1117ADT33TR, IC25 Si8641EC-B-IS1, IC26 PCA21125T/Q900/1,1, IC27 AT25256B-SSHL-B, IC28 W5500, IC29 BC857BS, IC3 MC78L05, IC30 TLC555, IC31 SN74LVC2G08DCTR, IC32 TPS3705-33D, IC33 SN74LV1T34DBVR, IC34 SN74LVC2G02DCTR, IC35 DAC8552IDGKTG4, IC36 ADS1120IPWR, IC37 MCP23S08-E/SO, IC38 OP27GSZ, IC39 TL072D, IC4 LM5574MTX/NOPB, IC40 TL072D, IC41 REF5025AIDG4, IC42 LTC3864EMSE#PBF, IC43 LM5574MTX/NOPB, IC44 MC79L05, IC45 MC78L05, IC46 TS5A9411DCKT, IC47 ADG465SOT-23, IC48 LP339D, IC49 LP2951SO8, IC5 LP2951SO8, IC6 TL072D, IC7 TL072D, IC8 OP27GSZ, IC9 MCP23S08-E/SO, J1 BS-244DSM-R, J2 BS-244DSM-G, J3 BS-244DSM-B, J4 BS-244DSM-R, J5 BS-244DSM-B, Q1 SUD19P06-60, Q10 MMBT5401, Q11 MMBT5401, Q12 MMBT5551, Q13 MMBT5551, Q14 BSS84P, Q15 2N7002, Q16 MMBT5551, Q17 MMBT5401, Q18 MMBT5551, Q19 MMBT5551, Q2 MMBT5401, Q20 BTA26-600, Q21 BTA26-600, Q22 IRLL014N, Q23 IRLML2246TRPBF, Q24 IRLML2246TRPBF, Q25 IRLML2246TRPBF, Q26 IRLML2246TRPBF, Q27 2N7002, Q28 IRLML2246TRPBF, Q29 2N7002, Q3 2N7002, Q30 2N7002, Q31 IRFP250N, Q32 BCP56-16.115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

Commit message: BOM corrections, Q1 gate trace improved
Routing:
- net N$30: track 4.32 -> 0.59 mm
- net N$235: track 4.32 -> 0.59 mm
- added copper zone on layer 1, net N$235
- added copper zone on layer 1, net N$30
Other:
- board text removed: "C157"
- board text removed: "C158"
- board text removed: "C159"
- board text removed: "C160"
- board text removed: "C161"
- board text removed: "C162"
- board text removed: "C163"
- board text removed: "C164"
- board text removed: "C165"
- board text removed: "C166"
- board text removed: "C167"
- board text removed: "C168"
- board text removed: "C169"
- board text removed: "C170"
- board text removed: "C171"
- board text removed: "C172"
- board text removed: "C173"
- board text removed: "C174"
- board text removed: "C175"
- board text removed: "C176"
- board text removed: "C177"
- board text removed: "C178"
- board text removed: "C179"
- board text removed: "C180"
- board text removed: "C181"
- board text removed: "C182"
- board text removed: "C183"
- board text removed: "C184"
- board text removed: "C185"
- board text removed: "C186"
- board text removed: "C187"
- board text removed: "C188"
- board text removed: "C189"
- board text removed: "C190"
- board text removed: "C191"
- board text removed: "C192"
- board text removed: "C193"
- board text removed: "C194"
- board text removed: "C195"
- board text removed: "C196"
- board text removed: "C197"
- board text removed: "C198"
- board text removed: "C199"
- board text removed: "C200"
- board text removed: "C201"
- board text removed: "C202"
- board text removed: "C203"
- board text removed: "C204"
- board text removed: "C205"
- board text removed: "C206"
- board text removed: "C207"
- board text removed: "C208"
- board text removed: "C209"
- board text removed: "C210"
- board text removed: "C211"
- board text removed: "C212"
- board text removed: "C213"
- board text removed: "C214"
- board text removed: "C215"
- board text removed: "C216"
- board text removed: "C217"
- board text removed: "C218"
- board text removed: "C219"
- board text removed: "C220"
- board text removed: "C221"
- board text removed: "C222"
- board text removed: "C223"
- board text removed: "C224"
- board text removed: "C225"
- board text removed: "C226"
- board text removed: "C227"
- board text removed: "C228"
- board text removed: "C229"
- board text removed: "C230"
- board text removed: "C231"
- board text removed: "C232"
- board text removed: "C233"
- board text removed: "C234"
- board text removed: "C235"
- board text removed: "C236"
- board text removed: "C237"
- board text removed: "C238"
- board text removed: "C239"
- board text removed: "C240"
- board text removed: "D30"
- board text removed: "D31"
- board text removed: "D32"
- board text removed: "D33"
- board text removed: "D34"
- board text removed: "D35"
- board text removed: "D36"
- board text removed: "D37"
- board text removed: "D38"
- board text removed: "D39"
- board text removed: "D40"
- board text removed: "D41"
- board text removed: "D42"
- board text removed: "D43"
- board text removed: "D44"
- board text removed: "D45"
- board text removed: "D46"
- board text removed: "D47"
- board text removed: "FB10"
- board text removed: "FB8"
- board text removed: "FB9"
- board text removed: "GND1"
- board text removed: "IC35"
- board text removed: "IC36"
- board text removed: "IC37"
- board text removed: "IC38"
- board text removed: "IC39"
- board text removed: "IC40"
- board text removed: "IC41"
- board text removed: "IC42"
- board text removed: "IC43"
- board text removed: "IC44"
- board text removed: "IC45"
- board text removed: "IC46"
- board text removed: "IC47"
- board text removed: "IC48"
- board text removed: "IC49"
- board text removed: "JP10"
- board text removed: "JP9"
- board text removed: "L11"
- board text removed: "L12"
- board text removed: "L13"
- board text removed: "L14"
- board text removed: "L15"
- board text removed: "L16"
- board text removed: "L17"
- board text removed: "LED2"
- board text removed: "NTC2"
- board text removed: "Q31"
- board text removed: "Q32"
- board text removed: "Q33"
- board text removed: "Q34"
- board text removed: "Q35"
- board text removed: "Q36"
- board text removed: "Q37"
- board text removed: "Q38"
- board text removed: "Q39"
- board text removed: "Q40"
- board text removed: "Q41"
- board text removed: "Q42"
- board text removed: "Q43"
- board text removed: "Q44"
- board text removed: "Q45"
- board text removed: "Q46"
- board text removed: "Q47"
- board text removed: "Q48"
- board text removed: "Q49"
- board text removed: "R173"
- board text removed: "R174"
- board text removed: "R175"
- board text removed: "R176"
- board text removed: "R177"
- board text removed: "R178"
- board text removed: "R179"
- board text removed: "R180"
- board text removed: "R181"
- board text removed: "R182"
- board text removed: "R183"
- board text removed: "R184"
- board text removed: "R185"
- board text removed: "R186"
- board text removed: "R187"
- board text removed: "R188"
- board text removed: "R189"
- board text removed: "R190"
- board text removed: "R191"
- board text removed: "R192"
- board text removed: "R193"
- board text removed: "R194"
- board text removed: "R195"
- board text removed: "R196"
- board text removed: "R197"
- board text removed: "R198"
- board text removed: "R199"
- board text removed: "R200"
- board text removed: "R201"
- board text removed: "R202"
- board text removed: "R203"
- board text removed: "R204"
- board text removed: "R205"
- board text removed: "R206"
- board text removed: "R207"
- board text removed: "R208"
- board text removed: "R209"
- board text removed: "R210"
- board text removed: "R211"
- board text removed: "R212"
- board text removed: "R213"
- board text removed: "R214"
- board text removed: "R215"
- board text removed: "R216"
- board text removed: "R217"
- board text removed: "R218"
- board text removed: "R219"
- board text removed: "R220"
- board text removed: "R221"
- board text removed: "R222"
- board text removed: "R223"
- board text removed: "R224"
- board text removed: "R225"
- board text removed: "R226"
- board text removed: "R227"
- board text removed: "R228"
- board text removed: "R229"
- board text removed: "R230"
- board text removed: "R231"
- board text removed: "R232"
- board text removed: "R233"
- board text removed: "R234"
- board text removed: "R235"
- board text removed: "R236"
- board text removed: "R237"
- board text removed: "R238"
- board text removed: "R239"
- board text removed: "R240"
- board text removed: "R241"
- board text removed: "R242"
- board text removed: "R243"
- board text removed: "R244"
- board text removed: "R245"
- board text removed: "R246"
- board text removed: "R247"
- board text removed: "R248"
- board text removed: "R249"
- board text removed: "R250"
- board text removed: "R251"
- board text removed: "R252"
- board text removed: "R253"
- board text removed: "R254"
- board text removed: "R255"
- board text removed: "R256"
- board text removed: "R257"
- board text removed: "R258"
- board text removed: "R259"
- board text removed: "R260"
- board text removed: "R261"
- board text removed: "R262"
- board text removed: "R263"
- board text removed: "R264"
- board text removed: "R265"
- board text removed: "R266"
- board text removed: "R267"
- board text removed: "R268"
- board text removed: "R269"
- board text removed: "R270"
- board text removed: "R271"
- board text removed: "R272"
- board text removed: "R273"
- board text removed: "R274"
- board text removed: "R275"
- board text removed: "R276"
- board text removed: "R277"
- board text removed: "R278"
- board text removed: "SW3"
- board text removed: "TP4"
- board text removed: "TR3"
- board text removed: "X21"
- board text removed: "X22"
- board text removed: "X23"
- board text removed: "ZD13"
- board text removed: "ZD14"
- board text removed: "ZD15"
- board text removed: "ZD16"
- board text removed: "ZD17"

Commit message: Small corrections on top silkscreen
Parts:
- C212, C39: value 2u2 -> n.c.
Routing:
- net N$30: track 0.59 -> 0.00 mm
- net N$235: track 0.59 -> 0.00 mm
- net D+: vias 2 -> 1
Other:
- board text removed: "Remote programming 1"
