File: Consolidated/Eagle files/EEZ PSU consolidated r5B11.brd (EAGLE design)
At the start: 309 x 150 mm, 557 parts, among them IC1 LTC3864EMSE#PBF, IC10 REF5025AIDG4, IC11 DAC8552IDGKTG4, IC12 ADG465SOT-23, IC13 TS5A9411DCKT, IC14 ADS1120IPWR, IC15 LP339D, IC16 LM25575MH/NOPB, IC17 TPD4E002DRLR, IC18 TPD2E001DZDR, IC19 ADUM3160BRWZ, IC2 MC79L05, IC20 TLC5925IDBQR, IC21 Si8641EC-B-IS1, IC22 SI8651EC-B-IS1, IC23 SI8651EC-B-IS1, IC24 LD1117ADT33TR, IC25 Si8641EC-B-IS1, IC26 PCA21125T/Q900/1,1, IC27 AT25256B-SSHL-B, IC28 W5500, IC29 BC857BS, IC3 MC78L05, IC30 TLC555, IC31 SN74LVC08APWR, IC32 TPS3705-33D, IC33 SN74LV1T34DBVR, IC34 SN74LVC2G02DCTR, IC4 LM5574MTX/NOPB, IC5 LP2951SO8, IC6 TL072D, IC7 TL072D, IC8 OP27GSZ, IC9 MCP23S08-E/SO, J1 BS-244DSM-R, J2 BS-244DSM-G, J3 BS-244DSM-B, J4 BS-244DSM-R, J5 BS-244DSM-B, J6 1-726388-2, Q1 IRFR5305, Q10 MMBT5401, Q11 MMBT5401, Q12 MMBT5551, Q13 MMBT5551, Q14 BSS84P, Q15 2N7002, Q16 MMBT5551, Q17 MMBT5401, Q18 MMBT5551, Q19 MMBT5551, Q2 MMBT5401, Q20 BTA26-600, Q21 BTA26-600, Q22 IRLL014N, Q23 IRLML2246TRPBF, Q24 IRLML2246TRPBF, Q25 IRLML2246TRPBF, Q26 IRLML2246TRPBF, Q27 2N7002, Q28 IRLML2246TRPBF, Q29 2N7002, Q3 2N7002, Q30 2N7002, Q4 IRFP250N, Q5 BC857C, Q7 BCP56-16.115, Q8 IRFR5305, Q9 BCP56-16.115, SW1 A101SYCQ04, SW2 1301.9316, X1 39303035, X10 826629-5, X11 2411-01, X12 MC000006, X13 TSW-113-07-F-D, X14 MC000005, X15 TSW-113-07-F-D, X16 09185067324, X17 22-23-2021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

Commit message: optimized values for CC resistors
Parts:
- C95: value 3n9 -> 3n3
- R32: value 2K2 -> 1K
- R64, R72: value 2K55 0.1% -> 2K 0.1%
- R67, R71: value 102R 0.1% -> 82R 0.1%
- R70: value 5K1 -> 10K
- X14: value MC000005 -> MC000006
- Y1: value 32,768kHz -> 32.768kHz

Commit message: #16, #17, #18
Parts:
- added C153, C157: 50SVPF18M, Panasonic-EEEFK_EEEFP:CAPAE830X650N
- added C161: 4n7, rcl:C1210
- C106, C111: value EEEFK1J220P -> EEEFK1H470P
- moved C112 49.5 mm to (154.6, 44.8), flipped to the bottom, turned to 270 degrees
- moved C110 43.6 mm to (151.4, 47.7), flipped to the bottom
- moved C108 32.3 mm to (191.5, 21.4), flipped to the bottom, turned to 0 degrees
- moved F1 18.5 mm to (115.3, 29.8), flipped to the top
- moved OK4 15.1 mm to (117.5, 21.5), flipped to the top
- moved ZD3 14.1 mm to (118.4, 29.2), flipped to the top, turned to 90 degrees
- moved C105 14.0 mm to (191.5, 18.2), flipped to the bottom, turned to 180 degrees
- moved R30 12.0 mm to (123.3, 18.5)
- moved ZD11 5.97 mm to (132.4, 31.6)
- moved R136A 2.02 mm to (180.0, 7.49), flipped to the bottom
- moved C104A 1.97 mm to (182.5, 7.49), flipped to the bottom
- moved C109A 1.34 mm to (144.8, 11.4)
- moved R140A 1.34 mm to (142.2, 11.4)
- moved C125 0.76 mm to (290.9, 66.5)
Connections:
- net N$68 renamed AUX_SYNC
- net +3V3: now also C125.2, SP1.+B
- net +5V: no longer C125.2, SP1.+B
- net AC_EARTH: now also C161.1
- net AUX2_USET_IN: now also X14.8, X14.8.1; no longer X14.6, X14.6.1
- net CH2_GND: now also X14.7, X14.7.1; no longer X14.5, X14.5.1
- net EARTH: now also X14.3, X14.3.1; no longer X14.1, X14.1.1
- net GND: now also C161.2
- net N$188: now also X14.2, X14.2.1; no longer X14.8, X14.8.1
- net N$189: now also X14.1, X14.1.1; no longer X14.7, X14.7.1
- net OUT1+: now also C153.1; no longer C105.1
- net OUT1-: now also C153.2
- net OUT2+: now also C157.1
- net OUT2-: now also C157.2; no longer C112.2
- net PWR_IN1+: now also C105.1
- net PWR_IN2-: now also C112.2
- net SENSE2+: now also X14.5, X14.5.1; no longer X14.3, X14.3.1
- net SENSE2-: now also X14.4, X14.4.1; no longer X14.2, X14.2.1
Routing:
- net EARTH: track 238.2 -> 293.7 mm, vias 1 -> 4
- net +3V3: track 672.0 -> 715.6 mm
- net MISO: track 299.9 -> 264.0 mm, vias 13 -> 12
- net DOUT: track 134.7 -> 148.0 mm
- net N$189: track 9.38 -> 3.10 mm
- net OUT1+: track 18.5 -> 24.3 mm
- net GND: track 509.2 -> 514.7 mm, vias 298 -> 300
- net AUX2_USET_IN: track 16.1 -> 10.7 mm
- net SENSE2-: track 4.13 -> 9.15 mm
- net +5V: track 898.5 -> 893.9 mm
- net NTC2: track 205.2 -> 200.7 mm
- net N$182: track 3.09 -> 7.36 mm, vias 1 -> 0
- net PWR_IN1+: track 26.6 -> 30.6 mm, vias 0 -> 1
- net OUT1-: track 43.5 -> 47.1 mm, vias 0 -> 1
- net !CH2_RESET: track 86.4 -> 89.4 mm
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Other:
- board text added: "(01/2017)"
- board text added: "C153"
- board text added: "C157"
- board text added: "C161"
- board text added: "EEZ AUX PS r5B11"
- board text added: "EEZ AUX PS r5B11 (01/2017)"
- board text added: "EEZ Arduino shield (01/2017 r4B2)"
- board text added: "r4B2 (01/2017)"
- board text removed: "(10/2016)"
- board text removed: "EEZ AUX PS r5B10"
- board text removed: "EEZ AUX PS r5B10 (10/2016)"
- board text removed: "EEZ Arduino shield (12/2016 r4B1)"
- board text removed: "JP3"
- board text removed: "X14"
- board text removed: "r4B1 (12/2016)"
