File: Consolidated/Eagle files/EEZ PSU r5B11 panel.brd (EAGLE design)
At the start: 309 x 150 mm, 838 parts, among them IC1 LTC3864EMSE#PBF, IC10 REF5025AIDG4, IC11 DAC8552IDGKTG4, IC12 ADG465SOT-23, IC13 TS5A9411DCKT, IC14 ADS1120IPWR, IC15 LP339D, IC16 LM25575MH/NOPB, IC17 TPD4E002DRLR, IC18 TPD2E001DZDR, IC19 ADUM3160BRWZ, IC2 MC79L05, IC20 TLC5925IDBQR, IC21 Si8641EC-B-IS1, IC22 SI8651EC-B-IS1, IC23 SI8651EC-B-IS1, IC24 LD1117ADT33TR, IC25 Si8641EC-B-IS1, IC26 PCA21125T/Q900/1,1, IC27 AT25256B-SSHL-B, IC28 W5500, IC29 BC857BS, IC3 MC78L05, IC30 TLC555, IC31 SN74LVC08APWR, IC32 TPS3705-33D, IC33 SN74LV1T34DBVR, IC34 SN74LVC2G02DCTR, IC35 DAC8552IDGKTG4, IC36 ADS1120IPWR, IC37 MCP23S08-E/SO, IC38 OP27GSZ, IC39 TL072D, IC4 LM5574MTX/NOPB, IC40 TL072D, IC41 REF5025AIDG4, IC42 LTC3864EMSE#PBF, IC43 LM5574MTX/NOPB, IC44 MC79L05, IC45 MC78L05, IC46 TS5A9411DCKT, IC47 ADG465SOT-23, IC48 LP339D, IC49 LP2951SO8, IC5 LP2951SO8, IC6 TL072D, IC7 TL072D, IC8 OP27GSZ, IC9 MCP23S08-E/SO, J1 BS-244DSM-R, J2 BS-244DSM-G, J3 BS-244DSM-B, J4 BS-244DSM-R, J5 BS-244DSM-B, J6 1-726388-2, Q1 IRFR5305, Q10 MMBT5401, Q11 MMBT5401, Q12 MMBT5551, Q13 MMBT5551, Q14 BSS84P, Q15 2N7002, Q16 MMBT5551, Q17 MMBT5401, Q18 MMBT5551, Q19 MMBT5551, Q2 MMBT5401, Q20 BTA26-600, Q21 BTA26-600, Q22 IRLL014N, Q23 IRLML2246TRPBF, Q24 IRLML2246TRPBF, Q25 IRLML2246TRPBF, Q26 IRLML2246TRPBF, Q27 2N7002, Q28 IRLML2246TRPBF, Q29 2N7002, Q3 2N7002, Q30 2N7002, Q31 BCP56-16.115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

Commit message: #16, #17, #18
Parts:
- added C254: n.c, rcl:C1206
- added C255: 100n, rcl:C0603
- added C256: n.c., rcl:C0805
- C106, C111: value EEEFK1J220P -> EEEFK1H470P
- C153: value 100n -> 50SVPF18M; device rcl:C0603 -> Panasonic-EEEFK_EEEFP:CAPAE830X650N
- C157: value 1n -> 50SVPF18M; device rcl:C0805 -> Panasonic-EEEFK_EEEFP:CAPAE830X650N
- C161: value 100n -> 4n7; device rcl:C0603 -> rcl:C1210
- C162: value 120p -> 100n; device rcl:C0805 -> rcl:C0603
- C163: value 10u -> 1n; device rcl:C1210 -> rcl:C0805
- C165, C204: value 100n -> 120p; device rcl:C0603 -> rcl:C0805
- C166: value 100n -> 10u; device rcl:C0603 -> rcl:C1210
- C170, C172: value 47p -> 100n; device rcl:C0805 -> rcl:C0603
- C171, C177, C178: value 2n2 -> 100n; device rcl:C0805 -> rcl:C0603
- C173: value 2n2 -> 47p
- C174, C180: value 100n -> 2n2; device rcl:C0603 -> rcl:C0805
- C175: value 100n -> 47p; device rcl:C0603 -> rcl:C0805
- C176: value 1n -> 2n2
- C179, C216: value 10n -> 1n
- C181: value 1u -> 2n2
- C183, C188, C189: value 1u -> 100n; device rcl:C0805 -> rcl:C0603
- C184: value 10n -> 1u
- C185: value 100n -> 10n; device rcl:C0603 -> rcl:C0805
- C186: value 100n -> 1u; device rcl:C0603 -> rcl:C0805
- C187: value 1u -> 10n
- C190: value 1u/100V -> 1u; device rcl:C1206 -> rcl:C0805
- C191: value 4u7 -> 1u; device rcl:C1210 -> rcl:C0805
- C192: value 10u -> 1u; device rcl:C1210 -> rcl:C0805
- C193, C220: value 330p -> 1u/100V; device rcl:C0805 -> rcl:C1206
- C194: value 10u -> 4u7
- C195: value 4u7 -> 10u
- C196: value 4n7 -> 330p
- C197: value 120p -> 10u; device rcl:C0805 -> rcl:C1210
- C198: value 1u/100V -> 4u7; device rcl:C1206 -> rcl:C1210
- C199: value 470n -> 4n7
- C205: value n.c. -> 1u/100V; device rcl:C0805 -> rcl:C1206
- C206: value n.c. -> 470n
- C207: value 2u2 -> 100n; device rcl:C0805 -> rcl:C0603
- C208, C209: value 47u -> n.c.; device EEZ_Lib1:CAPAE660X610N -> rcl:C0805
- C211: value 470n -> 47u; device rcl:C0805 -> EEZ_Lib1:CAPAE660X610N
- C212: value 3n3 -> 47u; device rcl:C0805 -> EEZ_Lib1:CAPAE660X610N
- C213: value 1n -> 2u2
- C214: value 22n -> 470n
- C215: value 100n -> 3n3; device rcl:C0603 -> rcl:C0805
- C217: value 1u/100V -> 22n; device rcl:C1206 -> rcl:C0805
- C218: value n.c. -> 100n; device rcl:C0805 -> rcl:C0603
- C219: value 2u2 -> 10n
- C221: value 2m2 -> n.c.; device EEZ_Lib1:ECAP7.5/18 -> rcl:C0805
- C222: value 470n -> 2u2
- C223: value 100n -> 330p; device rcl:C0603 -> rcl:C0805
- C224: value 100n -> 2m2; device rcl:C0603 -> EEZ_Lib1:ECAP7.5/18
- C225: value 100n -> 470n; device rcl:C0603 -> rcl:C0805
- C226: value 10u -> 100n; device EEZ_Lib1:EC1206 -> rcl:C0603
- C227: value 4u7 -> 100n; device EEZ_Lib1:EC1206 -> rcl:C0603
- C228: value 2m2 -> 100n; device EEZ_Lib1:ECAP7.5/18 -> rcl:C0603
- C229: value EEEFK1J470P -> 10u; device Panasonic-EEEFK_EEEFP:CAPAE830X1050N -> EEZ_Lib1:EC1206
- C230: value 470p -> 4u7; device rcl:C0805 -> EEZ_Lib1:EC1206
- C231: value 4u7 -> 2m2; device rcl:C1210 -> EEZ_Lib1:ECAP7.5/18
- C232: value 10n -> EEEFK1J470P; device rcl:C0805 -> Panasonic-EEEFK_EEEFP:CAPAE830X1050N
- C233: value 10n -> 470p
- C234: value 2n2 -> 4u7; device rcl:C0805 -> rcl:C1210
- C235, C236: value 4n7 -> 10n; device rcl:C1206 -> rcl:C0805
- C237: value 4n7 -> 2n2; device rcl:C1206 -> rcl:C0805
- C238: value 100n -> 4n7; device rcl:C0603 -> rcl:C1206
- C239, C240: value 3n3 -> 4n7; device rcl:C0805 -> rcl:C1206
- C241: value 3n3 -> 100n; device rcl:C0805 -> rcl:C0603
- C243: value EEEFK1J101P -> 3n3; device EEZ_Lib1:PANASONIC_F -> rcl:C0805
- C244: value 1u -> 3n3
- C245: value n.c. -> 3n3
- C246: value 1u/100V -> EEEFK1J101P; device rcl:C1206 -> EEZ_Lib1:PANASONIC_F
- C247: value 1n -> 1u; device rcl:C1206 -> rcl:C0805
- C248: value 1n -> n.c.; device rcl:C1206 -> rcl:C0805
- C249: value 1n -> 1u/100V
- C251: value n.c -> 1n
- C252: value 100n -> 1n; device rcl:C0603 -> rcl:C1206
- C253: value n.c. -> 1n; device rcl:C0805 -> rcl:C1206
- C95: value 3n9 -> 3n3
- R197, R32: value 2K2 -> 1K
- R221, R224, R64, R72: value 2K55 0.1% -> 2K 0.1%
- R222, R223, R67, R71: value 102R 0.1% -> 82R 0.1%
- R280, R70: value 5K1 -> 10K
- X14: value MC000005 -> MC000006
- Y1: value 32,768kHz -> 32.768kHz
- moved C161 153.2 mm to (65.7, 56.1), turned to 270 degrees
- moved C235 133.9 mm to (156.2, 86.7)
- moved C237 125.6 mm to (165.4, 89.1)
- moved C236 124.6 mm to (168.6, 116.7), turned to 180 degrees
- moved C153 115.6 mm to (174.2, 4.57)
- moved C252 113.0 mm to (277.1, 142.1), turned to 90 degrees
- moved C253 108.8 mm to (277.1, 130.6), turned to 90 degrees
- moved C240 106.7 mm to (290.7, 97.7), turned to 180 degrees
- moved C157 103.0 mm to (136.1, 4.57), turned to 180 degrees
- moved C238 101.7 mm to (289.1, 102.2)
- moved C239 99.3 mm to (292.3, 102.2), turned to 270 degrees
- moved C234 86.6 mm to (251.0, 102.1), turned to 270 degrees
- moved C191 82.2 mm to (188.1, 146.2), turned to 0 degrees
- moved C232 81.9 mm to (238.1, 84.7), turned to 270 degrees
- moved C243 78.2 mm to (190.0, 132.7), turned to 90 degrees
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Connections:
- net N$68 renamed AUX_SYNC
- removed net N$195 (its old number): C167.2, C187.2, IC36.12, R182.2
- removed net N$203 (its old number): C176.2, R192.1
- removed net N$206 (its old number): C178.2, R194.1
- removed net N$212 (its old number): C179.1, R198.1
- removed net N$228 (its old number): C189.1, IC41.5
- removed net N$232 (its old number): C230.2, D40.A, Q41.B, R231.1, R233.2
- removed net N$236 (its old number): C199.1, IC42.9
- removed net N$242 (its old number): C207.1, D42.A, L13.1
- removed net N$246 (its old number): C214.2, IC43.16
- removed net N$251 (its old number): C216.1, IC43.10
- removed net N$255 (its old number): C224.1, D48.C, FB9.P$1, IC45.1
- removed net N$257 (its old number): C253.2, IC47.1, R247.1
- removed net N$262 (its old number): C234.2, Q45.C, R260.1, R262.2
- removed net N$265 (its old number): C234.1, Q46.B, R260.2, R261.2
- removed net N$267 (its old number): C227.+, FB10.P$1, IC49.1, R248.1, R250.1
- removed net N$272 (its old number): C242.1, IC36.6, R269.2
- removed net N$274 (its old number): C157.1, R273.1
- removed net N$279 (its old number): C252.1, IC40.5, R279.1, R280.2
- new net N$193: C165.1, D31.C, IC39.2, R181.2, R194.2
- new net N$198: C176.1, R217.2, R219.1
- new net N$204: C180.2, R193.1
- new net N$211: C182.1, R198.1
- new net N$227: C192.1, IC41.5
- new net N$229: C165.2, R227.1
- new net N$233: C204.1, IC42.6, R236.2
- new net N$238: C207.2, IC42.4
- new net N$243: C216.2, R241.2
- new net N$248: C218.2, IC43.1
- new net N$252: C223.2, R246.2
- new net N$256: C256.2, IC47.1, R247.1
- new net N$260: C235.2, Q45.B, R255.1, R256.2, R275.2
- new net N$263: C236.1, Q44.B, R258.2, R259.1
- new net N$266: C230.+, FB10.P$1, IC49.1, R248.1, R250.1
- new net N$268: C242.2, IC36.10, R266.2
- new net N$273: C163.1, R273.1
- new net N$277: C254.2, R278.1
- net +3V3: now also C125.2, SP1.+B
- net +5V: no longer C125.2, SP1.+B
- net +5V1: now also C169.1, C171.2, C191.2; no longer C166.1, C168.2, C188.2
- net +VNR1: now also C213.1, C225.1, C226.1; no longer C210.1, C222.1, C223.1
- net +VREF1: now also C168.2, C229.+, C241.2; no longer C165.2, C226.+, C238.2
- net -9V1: now also C214.2; no longer C208.2
- net AC_EARTH: now also C161.1
- net AC_IN3: now also C250.1, C251.2, C254.1; no longer C247.1, C248.2, C251.1
- net AC_IN4: now also C252.1, C253.2; no longer C249.1, C250.2
- net AUX2_USET_IN: now also X14.8, X14.8.1; no longer X14.6, X14.6.1
- net CH2_GND: now also X14.7, X14.7.1; no longer X14.5, X14.5.1
- net DC+1: now also C240.2; no longer C237.2
- net DC-1: now also C240.1; no longer C237.1
- net DC_BIAS1: now also C193.1; no longer C190.1
- net DC_OUT1: now also C194.1, C205.1, C206.2, C224.+, C231.+, C234.1, C238.2, C251.1, C253.1; no longer C191.1, C195.1, C199.2, C221.+, C228.+, C231.1, C235.2, C248.1, C250.1
- net DC_PREG3: now also C220.1, C249.1; no longer C217.1, C246.1
- net EARTH: now also X14.3, X14.3.1; no longer X14.1, X14.1.1
- net EARTH1: now also C238.1, C239.2; no longer C235.1, C236.2
- net GND: now also C161.2
- net GND1: now also C162.1, C169.2, C170.1, C171.1, C172.1, C177.1, C178.2, C182.2, C183.2, C189.1, C190.1, C191.1, C193.2, C197.2, C205.2, C212.2, C213.2, C214.1, C218.1, C220.2, C221.2, C224.-, C225.2, C226.2, C227.2, C228.1, C229.-, C230.-, C231.-, C234.2, C242.1, C243.1, C244.1, C245.2, C250.2, C255.2, C256.1; no longer C153.1, C161.1, C163.2, C165.1, C169.1, C174.1, C175.2, C179.2, C180.2, C181.1, C182.1, C183.1, C189.2, C190.2, C191.2, C207.2, C208.1, C209.2, C212.1, C216.2, C217.2, C218.2, C221.-, C223.2, C224.2, C225.1, C226.-, C227.-, C228.-, C231.2, C236.1, C238.1, C240.1, C242.2, C243.2, C247.2, C253.1
- net I_SERVO1: now also C163.2; no longer C157.2
- net L_OUT12: now also C195.1, C197.1, C246.1; no longer C192.1, C194.1, C243.1
- net N$188: now also X14.2, X14.2.1; no longer X14.8, X14.8.1
- net N$189: now also X14.1, X14.1.1; no longer X14.7, X14.7.1
- net N$194: now also C170.2, C190.2, IC36.12, R182.2; no longer C162.1, D31.C, IC39.2, R181.2, R194.2
- net N$199: now also C174.1, R216.2, R218.1; no longer C173.1, R217.2, R219.1
- net N$200: now also C173.2, R189.1; no longer C171.1, R216.2, R218.1
- net N$201: now also C175.2, R190.1; no longer C170.2, R189.1
- net N$202: now also C179.2, R192.1; no longer C172.2, R190.1
- net N$205: now also C181.2, R194.1; no longer C177.2, R193.1
- net N$230: now also C196.2, R230.2; no longer C162.2, R227.1
- net N$231: now also C233.2, D40.A, Q41.B, R231.1, R233.2; no longer C193.2, R230.2
- net N$234: now also C199.1, R236.1; no longer C197.1, IC42.6, R236.2
- net N$235: now also C206.1, IC42.9; no longer C196.1, R236.1
- net N$239: now also C233.1, Q41.C, Q43.3, R252.1; no longer C204.2, IC42.4
- net N$240: now also C208.2, C247.1, L11.1, L12.2, R237.1, R254.2; no longer C230.1, Q41.C, Q43.3, R252.1
- net N$241: now also C210.1, D42.A, L13.1; no longer C205.2, C244.1, L11.1, L12.2, R237.1, R254.2
- net N$244: now also C216.1, IC43.6, R242.2, R243.1; no longer C213.2, R241.2
- net N$245: now also C217.2, IC43.16; no longer C213.1, IC43.6, R242.2, R243.1
- net N$249: now also IC43.8; no longer IC43.1
- net N$250: now also C219.1, IC43.10; no longer C212.2, IC43.8
- net N$253: now also C228.2, D47.A, FB8.P$1, IC44.1; no longer C220.2, R246.2
- net N$254: now also C227.1, D48.C, FB9.P$1, IC45.1; no longer C225.2, D47.A, FB8.P$1, IC44.1
- net N$261: now also C237.2, Q45.C, R260.1, R262.2; no longer C232.2, Q45.B, R255.1, R256.2, R275.2
- net N$264: now also C237.1, Q46.B, R260.2, R261.2; no longer C233.1, Q44.B, R258.2, R259.1
- net N$269: now also C243.2, IC36.7, R267.2; no longer C239.2, IC36.10, R266.2
- net N$270: now also C244.2, IC36.11, R268.2; no longer C240.2, IC36.7, R267.2
- net N$271: now also C245.1, IC36.6, R269.2; no longer C241.2, IC36.11, R268.2
- net N$278: now also C255.1, IC40.5, R279.1, R280.2; no longer C251.2, R278.1
- net OUT+1: now also C174.2, C179.1, C181.1, C235.1; no longer C171.2, C176.1, C178.1, C232.1
- net OUT-1: now also C176.2, C180.1, C236.2; no longer C173.2, C177.1, C233.2
- net OUT1+: now also C153.1; no longer C105.1
- net OUT1-: now also C153.2
- net OUT2+: now also C157.1
- net OUT2-: now also C157.2; no longer C112.2
- net POUT-1: now also C208.1, C209.2, C232.2, C247.2, C248.2; no longer C205.1, C206.2, C229.2, C244.2, C245.2
- net PREG_OUT1: now also C209.1, C232.1, C248.1; no longer C206.1, C229.1, C245.1
- net PWR_IN1+: now also C105.1
- net PWR_IN2-: now also C112.2
- net SENSE+1: now also C173.1; no longer C170.1
- net SENSE-1: now also C175.1; no longer C172.1
- net SENSE2+: now also X14.5, X14.5.1; no longer X14.3, X14.3.1
- net SENSE2-: now also X14.4, X14.4.1; no longer X14.2, X14.2.1
- net SGND1: now also C199.2, C204.2, C207.1; no longer C196.2, C197.2, C204.1
- net SW3: now also C196.1; no longer C193.1
- net SW4: now also C217.1, C223.1; no longer C214.1, C220.1
- net V+1: now also C162.2, C166.1, C167.2, C172.2, C178.1, C187.2, C188.2; no longer C153.2, C163.1, C164.2, C169.2, C175.1, C181.2, C185.2
- net V-1: now also C164.2, C177.2, C183.1, C185.2, C189.2; no longer C161.2, C174.2, C180.1, C182.2, C183.2
- net VOUT+1: now also C212.1, C221.1, C222.1; no longer C209.1, C218.1, C219.1
Routing:
- net EARTH: track 238.2 -> 293.7 mm, vias 1 -> 4
- net N$262 (its old number): track 43.7 -> 0.00 mm, vias 2 -> 0
- net +3V3: track 672.0 -> 715.6 mm
- net MISO: track 299.9 -> 264.0 mm, vias 13 -> 12
- net N$261: track 8.39 -> 43.7 mm, vias 0 -> 2
- net N$193: track 0.00 -> 22.0 mm
- net N$267 (its old number): track 16.8 -> 0.00 mm
- net N$266: track 0.00 -> 16.8 mm
- net N$241: track 20.8 -> 7.11 mm
- net DOUT: track 134.7 -> 148.0 mm
- net N$232 (its old number): track 12.6 -> 0.00 mm
- net N$268: track 0.00 -> 12.1 mm, vias 0 -> 2
- net N$194: track 22.0 -> 10.8 mm
- net N$195 (its old number): track 10.8 -> 0.00 mm
- net N$244: track 1.97 -> 12.7 mm
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Other:
- board text added: "(01/2017)"
- board text added: "Alu thermal bridge (5mm thick)"
- board text added: "C153"
- board text added: "C157"
- board text added: "C161"
- board text added: "EEZ AUX PS r5B11"
- board text added: "EEZ AUX PS r5B11 (01/2017)"
- board text added: "EEZ Arduino shield (01/2017 r4B2)"
- board text added: "r4B2 (01/2017)"
- board text removed: "(10/2016)"
- board text removed: "EEZ AUX PS r5B10"
- board text removed: "EEZ AUX PS r5B10 (10/2016)"
- board text removed: "EEZ Arduino shield (12/2016 r4B1)"
- board text removed: "JP3"
- board text removed: "X14"
- board text removed: "r4B1 (12/2016)"
