File: Consolidated/Eagle files/EEZ PSU consolidated r5B12.brd (EAGLE design)
At the start: 337 x 150 mm, 552 parts, among them IC1 LTC3864EMSE#PBF, IC10 DAC8552IDGKTG4, IC11 ADG465SOT-23, IC12 TS5A9411DCKT, IC13 ADS1120IPWR, IC14 LP339D, IC15 TPD4E002DRLR, IC16 TPD2E001DZDR, IC17 ADUM3160BRWZ, IC18 TLC5925IDBQR, IC19 Si8641EC-B-IS1, IC2 LP2951SO8, IC20 SI8651EC-B-IS1, IC21 SI8651EC-B-IS1, IC22 LD1117ADT33TR, IC23 Si8641EC-B-IS1, IC24 PCA21125T/Q900/1,1, IC25 AT25256B-SSHL-B, IC26 W5500, IC27 BC857BS, IC28 TLC555, IC29 SN74LVC08APWR, IC3 TL783CKTTR, IC30 SN74LV1T34DBVR, IC31 TPS3705-33D, IC32 SN74LVC2G02DCTR, IC33 74LVC1G125GW.125, IC34 TPA6205A1DGN, IC4 LTC3260EMSE#PBF, IC5 TL072D, IC6 TL072D, IC7 OP27GSZ, IC8 MCP23S17-E/SS, IC9 REF5025AIDG4, J1 BS-244DSM-R, J2 1-726388-2, J3 BS-244DSM-G, J4 BS-244DSM-B, J5 BS-244DSM-R, J6 BS-244DSM-B, Q1 IRFR5305, Q10 MMBT5401, Q11 MMBT5551, Q12 MMBT5551, Q13 IRLL2705PBF, Q14 IRFR48ZPBF, Q15 IRLML2246TRPBF, Q16 2N7002, Q17 MMBT5551, Q18 MMBT5401, Q19 MMBT5551, Q2 MMBT5401, Q20 MMBT5551, Q21 BTA26-600, Q22 BTA26-600, Q23 IRLL2705PBF, Q24 MMBT5551, Q25 2N7002, Q26 IRLML2246TRPBF, Q27 IRLML2246TRPBF, Q28 IRLML2246TRPBF, Q29 IRLML2246TRPBF, Q3 2N7002, Q30 2N7002, Q31 IRLML2246TRPBF, Q32 2N7002, Q33 2N7002, Q4 IRFP250N, Q5 BC857C, Q6 BCP56-16.115, Q7 IRFR5305, Q8 BCP56-16.115, Q9 MMBT5401, SW1 A101SYCQ04, SW2 PEC11R-4015F-S0024, SW3 1301.9316, X1 39-30-1039, X10 826629-5, X11 2411-01, X12 MC000006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

Commit message: #28
Connections:
- removed net N$125: FB4.P$1, X7.2
- new net N$24: FB4.P$1, X7.10, X7.12, X7.2
- net AUX_ETH_ACTLED: now also X7.9; no longer X7.10
- net AUX_ETH_LINKLED: now also X7.11; no longer X7.12
- net GND: no longer X7.11, X7.9
Routing:
- net N$24: track 0.00 -> 27.2 mm
- net N$125: track 2.65 -> 0.00 mm
- net AUX_ETH_ACTLED: track 23.9 -> 25.7 mm
- net AUX_ETH_LINKLED: track 24.3 -> 22.6 mm

Commit message: Update encoder models
Parts:
- SW2: value PEC11R-4015F-S0024 -> EC12E20-24P24C-SW
Changed lines of the file:
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@@
 <layer number="23" name="tOrigins" color="15" fill="1" visible="no" active="yes"/>
 <layer number="24" name="bOrigins" color="15" fill="1" visible="no" active="yes"/>
-<layer number="25" name="tNames" color="7" fill="1" visible="no" active="yes"/>
+<layer number="25" name="tNames" color="7" fill="1" visible="yes" active="yes"/>
 <layer number="26" name="bNames" color="13" fill="1" visible="no" active="yes"/>
 <layer number="27" name="tValues" color="10" fill="1" visible="no" active="yes"/>
@@
 <text x="147.447" y="124.3965" size="1.016" layer="125" ratio="10" rot="R90">C148</text>
 <text x="325.882" y="59.8805" size="1.016" layer="125" ratio="10" rot="R90">C149</text>
-<text x="319.532" y="45.212" size="1.016" layer="125" ratio="10" rot="R90">C150</text>
+<text x="319.532" y="44.7675" size="1.016" layer="125" ratio="10" rot="R90">C150</text>
 <text x="326.009" y="35.1155" size="1.016" layer="125" ratio="10" rot="R270">C151</text>
-<text x="328.295" y="39.8145" size="0.8128" layer="125" ratio="10" rot="R90">C152</text>
+<text x="328.3585" y="39.497" size="0.8128" layer="125" ratio="10" rot="R90">C152</text>
 <text x="325.628" y="45.72" size="0.8128" layer="125" ratio="10" rot="R180">C153</text>
 <text x="321.1195" y="37.084" size="1.016" layer="125" ratio="10" rot="R90">C154</text>
-<text x="323.215" y="50.3555" size="0.8128" layer="125" ratio="10">C155</text>
+<text x="322.453" y="50.3555" size="0.8128" layer="125" ratio="10">C155</text>
 <text x="141.605" y="99.3775" size="1.27" layer="125" ratio="10">D1</text>
 <text x="114.002996875" y="112.411003125" size="1.016" layer="125" ratio="10" rot="R180">D2</text>
 <text x="80.0735" y="78.5495" size="1.016" layer="125" ratio="10" rot="R180">D3</text>
-<text x="79.629" y="92.5195" size="1.016" layer="125" ratio="10" rot="R270">D4</text>
+<text x="76.708" y="92.3925" size="1.016" layer="125" ratio="10" rot="R270">D4</text>
 <text x="54.864" y="98.2345" size="1.016" layer="125" ratio="10" rot="R270">D5</text>
 <text x="80.0735" y="80.391" size="1.016" layer="125" ratio="10" rot="R180">D6</text>
@@
 <text x="149.0289875" y="51.50200625" size="1.016" layer="125" ratio="10">D15</text>
 <text x="118.3012875" y="53.1026875" size="1.016" layer="125" ratio="10">D16</text>
-<text x="313.98570625" y="2.0074875" size="1.27" layer="125" ratio="10">D17</text>
+<text x="313.41420625" y="3.7219875" size="1.27" layer="125" ratio="10">D17</text>
 <text x="286.985203125" y="51.732003125" size="1.27" layer="125" ratio="10" rot="R90">D18</text>
 <text x="189.23" y="61.4045" size="1.27" layer="125" ratio="10">D19</text>
@@
 <text x="81.407" y="98.3615" size="1.016" layer="125" ratio="10">Q9</text>
 <text x="85.344" y="98.3615" size="1.016" layer="125" ratio="10">Q10</text>
-<text x="84.7725" y="94.234" size="1.016" layer="125" ratio="10" rot="R180">Q11</text>
+<text x="85.471" y="94.361" size="1.016" layer="125" ratio="10" rot="R180">Q11</text>
 <text x="103.759" y="112.7125" size="1.016" layer="125" ratio="10">Q12</text>
 <text x="27.432" y="88.5952" size="1.27" layer="125" ratio="10" rot="R180">Q13</text>
@@
 <text x="48.7426" y="118.4656" size="1.016" layer="125" ratio="10" rot="R180">R32</text>
 <text x="107.2515" y="80.01" size="1.016" layer="125" ratio="10">R33</text>
-<text x="82.7151" y="88.6206" size="0.9906" layer="125" ratio="10" rot="R180">R34</text>
+<text x="82.0166" y="87.6554" size="0.9906" layer="125" ratio="10" rot="R90">R34</text>
 <text x="84.0486" y="106.7816" size="1.016" layer="125" ratio="10" rot="R180">R35</text>
 <text x="88.3031" y="106.7816" size="1.016" layer="125" ratio="10" rot="R180">R36</text>
@@
 <text x="82.6389" y="87.5919" size="0.9906" layer="125" ratio="10">R46</text>
 <text x="62.4586" y="129.1336" size="1.016" layer="125" ratio="10" rot="R180">R47</text>
-<text x="89.9541" y="89.2556" size="0.889" layer="125" ratio="10" rot="R180">R48</text>
+<text x="88.2269" y="88.4174" size="0.889" layer="125" ratio="10">R48</text>
 <text x="63.9445" y="128.143" size="1.016" layer="125" ratio="10">R49</text>
 <text x="82.7024" y="95.8469" size="0.9906" layer="125" ratio="10">R50</text>
@@
 <text x="322.453" y="40.8305" size="1.016" layer="125" ratio="10" rot="R270">R170</text>
 <text x="323.469" y="41.402" size="0.8128" layer="125" ratio="10" rot="R90">R171</text>
-<text x="319.532" y="48.7045" size="1.016" layer="125" ratio="10" rot="R90">R172</text>
+<text x="319.532" y="48.8315" size="1.016" layer="125" ratio="10" rot="R90">R172</text>
 <text x="325.374" y="50.9905" size="0.8128" layer="125" ratio="10">R173</text>
 <text x="321.7545" y="45.847" size="0.8128" layer="125" ratio="10" rot="R270">R174</text>
@@
 </element>
 <element name="D4" library="diode" package="SOD323-W" value="BAS316" x="78.6765" y="91.2495" smashed="yes" rot="R270">
-<attribute name="NAME" x="79.629" y="92.5195" size="1.016" layer="25" ratio="10" rot="R270"/>
+<attribute name="NAME" x="76.708" y="92.3925" size="1.016" layer="25" ratio="10" rot="R270"/>
 <attribute name="VALUE" x="78.0415" y="94.869" size="1.016" layer="27" ratio="10" rot="R270"/>
 </element>
@@
 </element>
 <element name="R34" library="rcl" package="R0805" value="16K" x="81.5975" y="85.5345" smashed="yes" rot="R270">
-<attribute name="NAME" x="82.7151" y="88.6206" size="0.9906" layer="25" ratio="10" rot="R180"/>
+<attribute name="NAME" x="82.0166" y="87.6554" size="0.9906" layer="25" ratio="10" rot="R90"/>
 <attribute name="VALUE" x="81.0641" y="87.0331" size="1.016" layer="27" ratio="10" rot="R270"/>
 </element>
@@
 </element>
 <element name="R48" library="rcl" package="R0805" value="51K" x="89.3445" y="87.3125" smashed="yes">
-<attribute name="NAME" x="89.9541" y="89.2556" size="0.889" layer="25" ratio="10" rot="R180"/>
+<attribute name="NAME" x="88.2269" y="88.4174" size="0.889" layer="25" ratio="10"/>
 <attribute name="VALUE" x="88.2269" y="86.8426" size="1.016" layer="27" ratio="10"/>
 </element>
@@
 </element>
 <element name="Q11" library="transistor" package="SOT23-BEC" value="MMBT5551" x="82.7405" y="91.5035" smashed="yes" rot="R90">
-<attribute name="NAME" x="84.7725" y="94.234" size="1.016" layer="25" ratio="10" rot="R180"/>
+<attribute name="NAME" x="85.471" y="94.361" size="1.016" layer="25" ratio="10" rot="R180"/>
 <attribute name="VALUE" x="87.249" y="92.075" size="1.016" layer="27" ratio="10" rot="R180"/>
 </element>
@@
 </element>
 <element name="D17" library="MyLib6" package="DO214AA" value="SMBJ5.0A-TR" x="318.7212" y="5.2705" smashed="yes" rot="R90">
-<attribute name="NAME" x="313.9857" y="2.0075" size="1.27" layer="25" ratio="10"/>
+<attribute name="NAME" x="313.4142" y="3.722" size="1.27" layer="25" ratio="10"/>
 <attribute name="VALUE" x="319.0142" y="0.789" size="1.016" layer="27" ratio="10" rot="R90"/>
 </element>
@@
 <attribute name="VALUE" x="102.0445" y="119.6975" size="1.27" layer="27" ratio="10"/>
 </element>
-<element name="SW2" library="EEZ_Lib1" package="EC12E_SW" value="PEC11R-4015F-S0024" x="216" y="62" smashed="yes" rot="MR270">
+<element name="SW2" library="EEZ_Lib1" package="EC12E_SW" value="EC12E20-24P24C-SW" x="216" y="62" smashed="yes" rot="MR270">
 <attribute name="NAME" x="219.218" y="55.2905" size="1.27" layer="26" rot="MR180"/>
 <attribute name="VALUE" x="206.455" y="62.5915" size="1.27" layer="28" rot="MR180"/>
@@
 </element>
 <element name="R172" library="rcl" package="R0805" value="10K" x="320.6115" y="50.3555" smashed="yes" rot="R270">
-<attribute name="NAME" x="319.532" y="48.7045" size="1.016" layer="25" ratio="10" rot="R90"/>
+<attribute name="NAME" x="319.532" y="48.8315" size="1.016" layer="25" ratio="10" rot="R90"/>
 <attribute name="VALUE" x="321.1195" y="49.0855" size="1.016" layer="27" ratio="10" rot="R90"/>
 </element>
 <element name="C155" library="rcl" package="C0805" value="220n" x="324.5485" y="48.26" smashed="yes" rot="R90">
-<attribute name="NAME" x="323.215" y="50.3555" size="0.8128" layer="25" ratio="10"/>
+<attribute name="NAME" x="322.453" y="50.3555" size="0.8128" layer="25" ratio="10"/>
 <attribute name="VALUE" x="324.9295" y="46.609" size="1.016" layer="27" ratio="10" rot="R90"/>
 </element>
 <element name="C150" library="rcl" package="C0805" value="470n" x="320.6115" y="46.4185" smashed="yes" rot="R270">
-<attribute name="NAME" x="319.532" y="45.212" size="1.016" layer="25" ratio="10" rot="R90"/>
+<attribute name="NAME" x="319.532" y="44.7675" size="1.016" layer="25" ratio="10" rot="R90"/>
 <attribute name="VALUE" x="321.056" y="44.577" size="1.016" layer="27" ratio="10" rot="R90"/>
 </element>
@@
 </element>
 <element name="C152" library="rcl" package="C0805" value="4n7" x="326.517" y="40.9575" smashed="yes" rot="R270">
-<attribute name="NAME" x="328.295" y="39.8145" size="0.8128" layer="25" ratio="10" rot="R90"/>
+<attribute name="NAME" x="328.3585" y="39.497" size="0.8128" layer="25" ratio="10" rot="R90"/>
 <attribute name="VALUE" x="326.0725" y="42.3545" size="1.016" layer="27" ratio="10" rot="R270"/>
 </element>

Commit message: #30 (optional microSD card)
Parts:
- added J7: 693072010801, EEZ_Lib1:693072010801
- moved X17 12.8 mm to (271.2, 16.1)
- moved R160 0.32 mm to (284.4, 32.1)
- moved Y1 0.27 mm to (278.3, 50.4)
- moved D10 0.06 mm to (29.9, 106.9)
Connections:
- new net EXTSD_CS: J7.2, MCU.A12
- net +3V3: now also J7.4
- net GND: now also J7.6, J7.Z1, J7.Z2
- net MISO: now also J7.7
- net MOSI: now also J7.3
- net SCLK: now also J7.5
Routing:
- net EXTSD_CS: track 0.00 -> 30.0 mm
- net MOSI: track 305.9 -> 325.9 mm
- net SCLK: track 289.8 -> 308.0 mm
- net MISO: track 289.5 -> 305.7 mm
- net TEMP_ANALOG: track 37.7 -> 29.5 mm
- net +3V3: track 731.8 -> 736.1 mm
- net NTC1: track 117.4 -> 115.6 mm
- net I_SERVO: track 36.8 -> 35.6 mm
- net LCD_DB7: track 88.6 -> 87.5 mm
- net LCD_DB15: track 100.5 -> 99.4 mm
- net LCD_DB6: track 85.3 -> 84.3 mm
- net BATT_NTC: track 119.1 -> 120.0 mm
- net LCD_RS: track 98.4 -> 99.0 mm
- net NTC2: vias 4 -> 5
Other:
- board text added: "J7"
- board text removed: "X21"

Commit message: Q24-> mosfet, swap outputs of Q32, Q33
Parts:
- Q24: value MMBT5551 -> 2N7002; device transistor:SOT23-BEC -> EEZ_Lib1:SOT103P240X110-3N
- R160: value 47K -> n.c.
- R21: value 16K -> 220R
- moved Q24 0.06 mm to (87.2, 40.1), turned to 180 degrees
Connections:
- net 0V: now also Q24.2; no longer Q24.E
- net N$208: now also Q24.3; no longer Q24.C
- net N$66: now also Q24.1; no longer Q24.B
- net PWR_DIRECT: now also Q33.3; no longer Q32.3
- net PWR_SSTART: now also Q32.3; no longer Q33.3
Routing:
- net PWR_SSTART: track 23.5 -> 22.7 mm
Other:
- board text added: "(03/2017)"
- board text added: "3.5" rotated!"
- board text added: "EEZ AUX PS r5B12 (03/2017)"
- board text added: "EEZ Arduino shield (03/2017 r5B12)"
- board text added: "r5B12 (03/2017)"
- board text removed: "(02/2017)"
- board text removed: "EEZ AUX PS r5B12 (02/2017)"
- board text removed: "EEZ Arduino shield (02/2017 r5B12)"
- board text removed: "r5B12 (02/2017)"

Commit message: IC7-> LTC2050HV
Parts:
- IC7: value OP27GSZ -> LTC2050HVCS8#PBF
Changed lines of the file:
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@@
 <layer number="49" name="Reference" color="7" fill="1" visible="no" active="yes"/>
 <layer number="50" name="dxf" color="7" fill="1" visible="no" active="no"/>
-<layer number="51" name="tDocu" color="14" fill="1" visible="no" active="yes"/>
+<layer number="51" name="tDocu" color="14" fill="1" visible="yes" active="yes"/>
 <layer number="52" name="bDocu" color="7" fill="1" visible="no" active="yes"/>
 <layer number="53" name="tGND_GNDA" color="7" fill="9" visible="no" active="no"/>
@@
 </element>
 <element name="SH1" library="EEZ_Lib1" package="SHORT_NOHOLE" value="Pgnd to Pout- short" x="116.84" y="82.931" smashed="yes" rot="R180"/>
-<element name="IC7" library="EEZ_Lib1" package="SOIC127P600X173-8N" value="OP27GSZ" x="45.0215" y="100.6475" smashed="yes" rot="R180">
+<element name="IC7" library="EEZ_Lib1" package="SOIC127P600X173-8N" value="LTC2050HVCS8#PBF" x="45.0215" y="100.6475" smashed="yes" rot="R180">
 <attribute name="NAME" x="47.1551" y="96.3295" size="1.27" layer="25" ratio="10" rot="SR0"/>
 <attribute name="VALUE" x="41.7036" y="100.249" size="1.016" layer="27" ratio="10" rot="SR0"/>

Commit message: #31
Parts:
- added R176: 1M, rcl:R0805
- moved X17 1.89 mm to (273.1, 16.1)
- moved C105 0.54 mm to (278.1, 17.0), turned to 270 degrees
Connections:
- net N$111: now also R176.2
- net N$112: now also R176.1
Routing:
- net NTC2: track 214.2 -> 219.7 mm
- net N$112: track 13.0 -> 18.4 mm
- net N$111: track 12.3 -> 17.6 mm
- net +3V3: track 736.1 -> 732.7 mm
- net TEMP_ANALOG: track 29.5 -> 27.8 mm
- net +5V: track 967.4 -> 968.6 mm
- net GND: vias 422 -> 421
Other:
- board text added: "(03/2017 r5B12)"
- board text added: "EEZ PSU power board (03/2017 r5B12)"
- board text added: "R176"
- board text removed: "(02/2017 r5B12)"
- board text removed: "EEZ PSU power board (02/2017 r5B12)"

Commit message: X1 rotated
Parts:
- added X21: ZL262-5SG, con-samtec:SSW-105-02-S-S
- C89, C94: value EEEFK1H470P -> UWT1H220MCL
- L1: device EEZ_Lib1:RN114 -> EEZ_Lib1:RN112
- R6: value 0R -> 1R
- X1: value 39-30-1039 -> (none)
- moved C27 17.6 mm to (117.3, 129.2)
- moved R21 16.7 mm to (116.9, 135.3), turned to 90 degrees
- moved R24 16.0 mm to (119.1, 138.8), turned to 180 degrees
- moved IC3 8.98 mm to (129.7, 134.3), turned to 270 degrees
- moved X1 7.25 mm to (163.1, 81.6), turned to 180 degrees
- moved C1 1.81 mm to (161.7, 96.5)
- moved ZD1 1.71 mm to (153.6, 106.0)
- moved L1 1.23 mm to (161.2, 103.4)
Connections:
- net AC_EARTH: now also X3.1; no longer X3.5
- net AC_IN_L: now also X3.5; no longer X3.1
- net DC+: now also X1.3; no longer X1.1
- net DC_OUT: now also X21.5
- net EARTH: now also X1.1; no longer X1.3
- net FB: now also X21.4
- net OUT+: now also X21.3
- net PREG_OUT: now also X21.2
- net V-: now also X21.1
Routing:
- net DC_OUT: track 120.4 -> 140.0 mm, vias 53 -> 54
- net PREG_OUT: track 4.77 -> 21.6 mm, vias 0 -> 2
- net FB: track 16.6 -> 32.7 mm
- net +VNR: track 81.9 -> 66.4 mm, vias 19 -> 20
- net OUT+: track 235.2 -> 243.7 mm
- net V-: track 137.9 -> 144.8 mm, vias 11 -> 12
- net DC-: track 5.43 -> 2.35 mm
- net +5V: track 968.6 -> 970.0 mm
- net EARTH: track 315.7 -> 314.5 mm
- net N$7: track 5.48 -> 6.07 mm
- net DC+: track 4.19 -> 4.74 mm
Other:
- board text added: "1 -5V"
- board text added: "2 Pout"
- board text added: "3 Out+"
- board text added: "4 FB"
- board text added: "5 +Vin"
- board text added: "DC in+ 3"
- board text added: "Earth 1"
- board text added: "X21"
- board text removed: "DC in+ 1"
- board text removed: "Earth 3"

Commit message: X20 rotated
Parts:
- moved X20 18.9 mm to (229.9, 46.4), turned to 270 degrees
- moved J7 0.06 mm to (275.8, 4.45)
Routing:
- net AUDIO_OUT: track 113.2 -> 131.9 mm
- net LCDSD_CS: track 101.5 -> 116.5 mm
- net !LCD_INT: track 16.4 -> 29.2 mm
- net MOSI: track 325.9 -> 313.8 mm
- net MISO: track 305.7 -> 294.9 mm, vias 13 -> 12
- net LCD_CS: track 127.5 -> 117.1 mm
- net !LCD_PD: track 15.3 -> 25.1 mm
- net SYNC1: track 36.1 -> 45.4 mm
- net +3V3: track 732.7 -> 740.0 mm
- net SCLK: track 308.0 -> 302.3 mm, vias 10 -> 8
- net GND: track 447.2 -> 449.1 mm, vias 421 -> 416
- net !ADC1_SELECT: track 87.1 -> 86.5 mm
