File: Consolidated/Eagle files/EEZ PSU r5B12 panel.brd (EAGLE design)
At the start: 337 x 150 mm, 812 parts, among them IC1 LTC3864EMSE#PBF, IC10 DAC8552IDGKTG4, IC11 ADG465SOT-23, IC12 TS5A9411DCKT, IC13 ADS1120IPWR, IC14 LP339D, IC15 TPD4E002DRLR, IC16 TPD2E001DZDR, IC17 ADUM3160BRWZ, IC18 TLC5925IDBQR, IC19 Si8641EC-B-IS1, IC2 LP2951SO8, IC20 SI8651EC-B-IS1, IC21 SI8651EC-B-IS1, IC22 LD1117ADT33TR, IC23 Si8641EC-B-IS1, IC24 PCA21125T/Q900/1,1, IC25 AT25256B-SSHL-B, IC26 W5500, IC27 BC857BS, IC28 TLC555, IC29 SN74LVC08APWR, IC3 TL783CKTTR, IC30 SN74LV1T34DBVR, IC31 TPS3705-33D, IC32 SN74LVC2G02DCTR, IC33 74LVC1G125GW.125, IC34 TPA6205A1DGN, IC35 DAC8552IDGKTG4, IC36 ADS1120IPWR, IC37 OP27GSZ, IC38 TL072D, IC39 TL072D, IC4 LTC3260EMSE#PBF, IC40 REF5025AIDG4, IC41 LTC3864EMSE#PBF, IC42 TS5A9411DCKT, IC43 ADG465SOT-23, IC44 LP339D, IC45 LTC3260EMSE#PBF, IC46 LP2951SO8, IC47 MCP23S17-E/SS, IC48 TL783CKTTR, IC5 TL072D, IC6 TL072D, IC7 OP27GSZ, IC8 MCP23S17-E/SS, IC9 REF5025AIDG4, J1 BS-244DSM-R, J2 1-726388-2, J3 BS-244DSM-G, J4 BS-244DSM-B, J5 BS-244DSM-R, J6 BS-244DSM-B, Q1 IRFR5305, Q10 MMBT5401, Q11 MMBT5551, Q12 MMBT5551, Q13 IRLL2705PBF, Q14 IRFR48ZPBF, Q15 IRLML2246TRPBF, Q16 2N7002, Q17 MMBT5551, Q18 MMBT5401, Q19 MMBT5551, Q2 MMBT5401, Q20 MMBT5551, Q21 BTA26-600, Q22 BTA26-600, Q23 IRLL2705PBF, Q24 MMBT5551, Q25 2N7002, Q26 IRLML2246TRPBF, Q27 IRLML2246TRPBF, Q28 IRLML2246TRPBF, Q29 IRLML2246TRPBF, Q3 2N7002, Q30 2N7002, Q31 IRLML2246TRPBF, Q32 2N7002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

Commit message: #28
Connections:
- new net +5V2: C80.1, C81.1, D12.C, IC17.16, K_DOUT.A1, OK1.1, OK2.1, OK3.4, TR1.4, X5.10, X5.8
- new net GND7: C80.2, C81.2, C84.2, IC15.2, IC17.15, IC17.9, Q25.2, R118.2, R122.2, R123.1, TR1.3, X10.4, X5.1, X5.2, X5.9
- net +5V: no longer C80.1, C81.1, D12.C, IC17.16, K_DOUT.A1, OK1.1, OK2.1, OK3.4, TR1.4, X5.10, X5.8
- net AUX_ETH_ACTLED: now also X7.9; no longer X7.10
- net AUX_ETH_LINKLED: now also X7.11; no longer X7.12
- net GND: no longer C80.2, C81.2, C84.2, IC15.2, IC17.15, IC17.9, Q25.2, R118.2, R122.2, R123.1, TR1.3, X10.4, X5.1, X5.2, X5.9, X7.11, X7.9
- net N$125: now also X7.10, X7.12
Routing:
- net +5V: track 967.4 -> 836.7 mm, vias 23 -> 20
- net +5V2: track 0.00 -> 130.7 mm, vias 0 -> 3
- net N$125: track 2.65 -> 27.2 mm
- net GND: track 448.0 -> 434.2 mm, vias 422 -> 414
- net GND7: track 0.00 -> 13.3 mm, vias 0 -> 8
- net AUX_ETH_ACTLED: track 23.9 -> 25.7 mm
- net AUX_ETH_LINKLED: track 24.3 -> 22.6 mm
- added copper zone on layer 16, net GND7

Commit message: #30 (optional microSD card)
Parts:
- added J7: 693072010801, EEZ_Lib1:693072010801
- SW2: value PEC11R-4015F-S0024 -> EC12E20-24P24C-SW
- moved X17 12.8 mm to (279.2, 16.1)
- moved R160 0.32 mm to (292.4, 32.1)
- moved Y1 0.27 mm to (286.3, 50.4)
- moved D10 0.06 mm to (22.9, 106.9)
- moved D26 0.06 mm to (189.9, 106.9)
Connections:
- removed net +5V2: C80.1, C81.1, D12.C, IC17.16, K_DOUT.A1, OK1.1, OK2.1, OK3.4, TR1.4, X5.10, X5.8
- removed net GND7: C80.2, C81.2, C84.2, IC15.2, IC17.15, IC17.9, Q25.2, R118.2, R122.2, R123.1, TR1.3, X10.4, X5.1, X5.2, X5.9
- new net EXTSD_CS: J7.2, MCU.A12
- net +3V3: now also J7.4
- net +5V: now also C80.1, C81.1, D12.C, IC17.16, K_DOUT.A1, OK1.1, OK2.1, OK3.4, TR1.4, X5.10, X5.8
- net GND: now also C80.2, C81.2, C84.2, IC15.2, IC17.15, IC17.9, J7.6, J7.Z1, J7.Z2, Q25.2, R118.2, R122.2, R123.1, TR1.3, X10.4, X5.1, X5.2, X5.9
- net MISO: now also J7.7
- net MOSI: now also J7.3
- net SCLK: now also J7.5
Routing:
- net +5V: track 836.7 -> 967.4 mm, vias 20 -> 23
- net +5V2: track 130.7 -> 0.00 mm, vias 3 -> 0
- net EXTSD_CS: track 0.00 -> 30.0 mm
- net MOSI: track 305.9 -> 325.9 mm
- net SCLK: track 289.8 -> 308.0 mm
- net MISO: track 289.5 -> 305.7 mm
- net GND7: track 13.3 -> 0.00 mm, vias 8 -> 0
- net GND: track 434.2 -> 447.5 mm, vias 414 -> 422
- net TEMP_ANALOG: track 37.7 -> 29.5 mm
- net +3V3: track 731.8 -> 736.1 mm
- net NTC1: track 117.4 -> 115.6 mm
- net I_SERVO1: track 36.8 -> 35.6 mm
- net I_SERVO: track 36.8 -> 35.6 mm
- net LCD_DB7: track 88.6 -> 87.5 mm
- net LCD_DB15: track 100.5 -> 99.4 mm
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- removed copper zone on layer 16, net GND7
Other:
- board text added: "J7"
- board text removed: "X21"

Commit message: Q24-> mosfet, swap outputs of Q32, Q33
Parts:
- Q24: value MMBT5551 -> 2N7002; device transistor:SOT23-BEC -> EEZ_Lib1:SOT103P240X110-3N
- R160: value 47K -> n.c.
- R21, R277: value 16K -> 220R
- moved Q24 0.06 mm to (95.2, 40.1), turned to 180 degrees
Connections:
- net 0V: now also Q24.2; no longer Q24.E
- net N$208: now also Q24.3; no longer Q24.C
- net N$66: now also Q24.1; no longer Q24.B
- net PWR_DIRECT: now also Q33.3; no longer Q32.3
- net PWR_SSTART: now also Q32.3; no longer Q33.3
Routing:
- net PWR_SSTART: track 23.5 -> 22.7 mm
Other:
- board text added: "(03/2017)"
- board text added: "EEZ AUX PS r5B12 (03/2017)"
- board text added: "EEZ Arduino shield (03/2017 r5B12)"
- board text added: "r5B12 (03/2017)"
- board text removed: "(02/2017)"
- board text removed: "EEZ AUX PS r5B12 (02/2017)"
- board text removed: "EEZ Arduino shield (02/2017 r5B12)"
- board text removed: "r5B12 (02/2017)"

Commit message: #31
Parts:
- added R280: 0R2, rcl:R1210
- IC37, IC7: value OP27GSZ -> LTC2050HVCS8#PBF
- R176: value 2K2 -> 1M
- R180: value 10K -> 2K2
- R182: value 10R -> 10K; device rcl:R1206 -> rcl:R0805
- R183: value 10K -> 10R; device rcl:R0805 -> rcl:R1206
- R184: value 2K2 -> 10K
- R185: value 5K6 -> 2K2
- R187: value 5K1 -> 5K6
- R189, R276: value 10K -> 5K1
- R193, R210, R277: value 220R -> 10K
- R195: value 470R -> 220R
- R196: value 100R -> 470R
- R197: value 1K -> 100R
- R198: value 470R -> 1K
- R199: value 16K -> 470R
- R200: value 750R -> 16K
- R201: value 2K2 -> 750R
- R203: value 220R -> 2K2
- R204: value 1K -> 220R
- R205: value 47K -> 1K
- R206, R252: value 10K -> 47K
- R208, R232: value 100K -> 10K
- R209, R231, R242: value 10K -> 100K
- R212, R278: value 1K8 -> 220R
- R213: value 51K -> 1K8
- R214: value 100K -> 51K
- R215: value 7K5 0.1% -> 100K
- R216: value 100K 0.1% -> 7K5 0.1%
- R218: value 24K 0.1% -> 100K 0.1%
- R220: value 7K5 0.1% -> 24K 0.1%
- R221: value 2K 0.1% -> 7K5 0.1%
- R222: value 82R 0.1% -> 2K 0.1%
- R224: value 2K 0.1% -> 82R 0.1%
- R225: value 10K -> 2K 0.1%
- R226, R269: value 0R -> 10K
- R227: value 330K -> 0R
- R228: value 4K7 -> 330K
- R229: value 10R -> 4K7; device rcl:R1206 -> rcl:R0805
- R230: value 100K -> 10R; device rcl:R0805 -> rcl:R1206
- R233: value 47K -> 100K
- R234: value R010/2W -> 47K; device rcl:R2512 -> rcl:R0805
- R235: value 10K -> R010/2W; device rcl:R0805 -> rcl:R2512
- R236: value 100R -> 10K
- R237: value 12K -> 100R; device rcl:R1206 -> rcl:R0805
- R238: value 330K -> 12K; device rcl:R0805 -> rcl:R1206
- R239: value 100K -> 330K
- R240: value 1K -> 100K
- R241: value 100K -> 1K
- R243: value n.c. -> 10K
- R244: value 100R -> n.c.
- R245: value 330R -> 100R
- R246, R249: value 750R -> 330R
- R247: value 1K -> 750R
- R248: value 330R -> 1K
- R250: value 47K -> 750R
- R254: value 47K -> 10K
- R255: value 220R -> 47K
- R259: value 2R2/2W -> 220R; device rcl:R2512 -> rcl:R0805
- R260: value 330K -> 2R2/2W; device rcl:R0805 -> rcl:R2512
- R261: value 1K -> 330K
- R262: value 2K2 -> 1K
- R264: value 10R -> 2K2; device rcl:R1206 -> rcl:R0805
- R265: value n.c. -> 10R; device rcl:R0805 -> rcl:R1206
- R266: device rcl:R1206 -> rcl:R0805
- R267: value 220R -> n.c.; device rcl:R0805 -> rcl:R1206
- R268: value 10K -> 220R
- R270: value n.c. -> 0R
- R271: value 0R020 -> n.c.; device EEZ_Lib1:R_2512-4WIRE -> rcl:R0805
- R272: value 47K -> 0R020; device rcl:R0805 -> EEZ_Lib1:R_2512-4WIRE
- R274: value 16K -> 47K
- R275: value 5K1 -> 16K
- R279: value 0R2 -> 1K8; device rcl:R1210 -> rcl:R0805
- moved R271 127.7 mm to (330.1, 107.7), turned to 270 degrees
- moved R176 117.5 mm to (275.6, 12.0), turned to 90 degrees
- moved R267 116.1 mm to (308.7, 133.6), flipped to the bottom, turned to 180 degrees
- moved R274 101.1 mm to (198.3, 87.2), turned to 270 degrees
- moved R279 98.1 mm to (291.8, 129.0), turned to 0 degrees
- moved R269 90.9 mm to (198.7, 116.3), turned to 180 degrees
- moved R245 87.5 mm to (279.6, 91.9), turned to 90 degrees
- moved R264 85.6 mm to (183.9, 91.4), turned to 0 degrees
- moved R261 81.4 mm to (264.2, 125.8), turned to 0 degrees
- moved R241 70.3 mm to (193.8, 122.9)
- moved R240 68.4 mm to (262.0, 127.8), turned to 0 degrees
- moved R262 66.5 mm to (184.1, 111.1)
- moved R263 61.9 mm to (245.5, 85.5), turned to 90 degrees
- moved R260 61.1 mm to (217.7, 86.1), turned to 270 degrees
- moved R238 58.9 mm to (320.7, 125.7), turned to 0 degrees
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Connections:
- net !DP_DRIVE1: now also R205.1, R210.1; no longer R204.1, R209.1
- net !SET_DP1: now also R215.2; no longer R214.2
- net +5V1: now also R189.2, R215.1, R254.2; no longer R187.2, R214.1, R253.2
- net +VNR1: now also R278.1; no longer R277.1
- net +VREF1: now also R269.1; no longer R268.1
- net -12V1: now also R205.2; no longer R203.2
- net -5VOUT1: now also R261.2; no longer R260.2
- net AC_IN4: now also R267.2; no longer R266.2
- net AUX_USET_IN1: now also R241.2; no longer R240.2
- net CC_ACTIVE1: now also R187.2, R189.1; no longer R186.2, R188.1
- net CURR_500MA1: now also R274.2; no longer R273.2
- net CURR_5A1: now also R273.2; no longer R272.2
- net CV_ACTIVE1: now also R186.2, R188.1; no longer R185.2, R187.1
- net DC_BIAS1: now also R212.2, R265.2; no longer R210.2, R264.2
- net DC_OUT1: now also R235.1, R238.1, R265.1, R271.2; no longer R234.1, R237.1, R264.1, R270.2
- net DP_LED1: now also R210.2; no longer R209.2
- net EARTH1: now also R266.2; no longer R265.2
- net FB1: now also R228.2, R229.1, R244.2; no longer R227.2, R228.1, R243.2
- net GCOM1: now also R216.1, R222.1; no longer R215.1, R221.1
- net GND1: now also R185.1, R201.1, R209.1, R214.1, R226.2, R230.1, R238.2, R240.1, R242.2, R252.1, R255.1, R263.1, R268.2, R274.1, R276.2, R279.2; no longer R184.1, R200.1, R208.1, R213.1, R225.2, R229.1, R237.2, R239.1, R241.2, R251.1, R254.1, R262.1, R267.2, R272.1, R275.2, R278.2
- net HEATSINK1: now also R266.1; no longer R265.1
- net ISENSE+1: now also R223.2; no longer R221.2
- net ISENSE-1: now also R224.2, R225.1; no longer R223.2, R224.1
- net I_MON1: now also R177.1, R225.2, R257.1; no longer R176.1, R224.2, R256.1
- net I_SERVO1: now also R208.1; no longer R207.1
- net I_SET1: now also R178.1, R259.1; no longer R177.1, R258.1
- net LOOP_CTRL1: now also R196.1; no longer R195.1
- net L_OUT12: now also R228.1, R233.1, R245.1; no longer R227.1, R231.1, R244.1
- net N$111: now also R176.2
- net N$112: now also R176.1
- net N$125: now also R182.2, R195.2; no longer R181.2, R194.2
- net N$154: now also R183.2; no longer R182.2
- net N$168: now also R186.1; no longer R185.1
- net N$179: now also R190.2, R216.2, R217.1; no longer R189.2, R215.2, R216.1
- net N$180: now also R191.2, R218.1, R221.2; no longer R190.2, R217.1, R220.2
- net N$191: now also R218.2, R220.1; no longer R217.2, R219.1
- net N$192: now also R217.2, R219.1; no longer R216.2, R218.1
- net N$196: now also R190.1; no longer R189.1
- net N$202: now also R191.1; no longer R190.1
- net N$203: now also R193.1; no longer R192.1
- net N$204: now also R177.2, R193.2; no longer R176.2, R191.2
- net N$205: now also R194.1; no longer R193.1
- net N$206: now also R195.1; no longer R194.1
- net N$209: now also R198.1; no longer R197.1
- net N$211: now also R197.1, R199.2; no longer R196.1, R198.2
- net N$213: now also R199.1; no longer R198.1
- net N$215: now also R203.1, R260.1; no longer R201.1, R259.1
- net N$216: now also R203.2; no longer R202.2
- net N$217: now also R196.2; no longer R195.2
- net N$218: now also R187.1; no longer R186.1
- net N$219: now also R207.2; no longer R206.2
- net N$220: now also R208.2; no longer R207.2
- net N$221: now also R185.2, R206.1; no longer R184.2, R205.1
- net N$222: now also R184.2, R226.1; no longer R183.2, R225.1
- net N$223: now also R211.1; no longer R210.1
- net N$224: now also R212.1; no longer R211.1
- net N$225: now also R213.2; no longer R212.2
- net N$226: now also R200.1, R201.2, R263.2; no longer R199.1, R200.2, R262.2
- net N$227: now also R204.1; no longer R203.1
- net N$228: now also R202.2; no longer R201.2
- net N$231: now also R227.1; no longer R226.1
- net N$232: now also R230.2; no longer R229.2
- net N$233: now also R231.1, R233.2; no longer R230.1, R232.2
- net N$234: now also R232.2; no longer R231.2
- net N$235: now also R236.2; no longer R235.2
- net N$236: now also R236.1; no longer R235.1
- net N$238: now also R270.1; no longer R269.1
- net N$239: now also R234.1; no longer R233.1
- net N$241: now also R244.1; no longer R243.1
- net N$242: now also R237.1, R245.2; no longer R236.1, R244.2
- net N$243: now also R239.1; no longer R238.1
- net N$245: now also R241.1; no longer R240.1
- net N$246: now also R243.1; no longer R242.1
- net N$247: now also R246.1, R247.2, R264.2; no longer R245.1, R246.2, R263.2
- net N$248: now also R251.1, R253.2; no longer R250.1, R252.2
- net N$249: now also R248.1; no longer R247.1
- net N$250: now also R249.2, R250.1; no longer R248.2, R249.1
- net N$251: now also R252.2; no longer R250.2
- net N$252: now also R253.1, R255.2; no longer R252.1, R254.2
- net N$253: now also R256.2; no longer R255.2
- net N$254: now also R257.2; no longer R256.2
- net N$255: now also R258.2; no longer R257.2
- net N$256: now also R259.2; no longer R258.2
- net N$257: now also R192.1, R262.2; no longer R191.1, R261.2
- net N$258: now also R262.1; no longer R261.1
- net N$259: now also R248.2, R264.1; no longer R247.2, R263.1
- net N$260: now also R267.1; no longer R266.1
- net N$261: now also R268.1, R269.2; no longer R267.1, R268.2
- net N$262: now also R270.2; no longer R269.2
- net N$263: now also R239.2, R242.1; no longer R238.2, R241.1
- net N$266: now also R240.2, R261.1; no longer R239.2, R260.1
- net N$269: now also R271.1; no longer R270.1
- net N$270: now also R272.2; no longer R271.2
- net N$271: now also R275.2, R276.1; no longer R274.2, R275.1
- net N$272: now also R275.1, R277.1; no longer R274.1, R276.1
- net N$274: now also R224.1, R272.1S; no longer R223.1, R271.1S
- net N$275: now also R223.1, R280.2; no longer R222.1, R279.2
- net N$276: now also R278.2, R279.1; no longer R277.2, R278.1
- net N$277: now also R272.2S, R280.1; no longer R271.2S, R279.1
- net N$59: now also R178.2; no longer R177.2
- net N$60: now also R181.2, R194.2; no longer R180.2, R193.2
- net OUT+1: now also R179.1, R198.2, R200.2, R231.2, R246.2, R260.2; no longer R178.1, R197.2, R199.2, R230.2, R245.2, R259.2
- net OUT-1: now also R180.2, R249.1; no longer R179.2, R248.1
- net POST_OE1: now also R213.1; no longer R212.1
- net POUT-1: now also R272.1; no longer R271.1
- net PREG_OUT1: now also R237.2; no longer R236.2
- net PRE_OE1: now also R209.2, R243.2; no longer R208.2, R242.2
- net PWRGOOD1: now also R277.2; no longer R276.2
- net SENSE+1: now also R179.2, R219.2, R247.1; no longer R178.2, R218.2, R246.1
- net SENSE-1: now also R180.1, R220.2, R250.2; no longer R179.1, R219.2, R249.2
- net SENSE1: now also R235.2; no longer R234.2
- net SENSE_ERR1: now also R254.1; no longer R253.1
- net SENSE_PROT1: now also R197.2, R214.2; no longer R196.2, R213.2
- net SGND1: now also R229.2, R234.2; no longer R228.2, R233.2
- net U_MON1: now also R182.1, R221.1, R256.1; no longer R181.1, R220.1, R255.1
- net U_SERVO1: now also R207.1, R227.2; no longer R206.1, R226.2
- net U_SET_OUT1: now also R181.1, R258.1; no longer R180.1, R257.1
- net V+1: now also R183.1, R206.2; no longer R182.1, R205.2
- net V-1: now also R184.1; no longer R183.1
Routing:
- net NTC2: track 214.2 -> 219.7 mm
- net N$112: track 13.0 -> 18.4 mm
- net N$111: track 12.3 -> 17.6 mm
- net +3V3: track 736.1 -> 732.7 mm
- net TEMP_ANALOG: track 29.5 -> 27.8 mm
- net +5V: track 967.4 -> 968.6 mm
- net GND: vias 422 -> 421
Other:
- board text added: "(03/2017 r5B12)"
- board text added: "EEZ PSU power board (03/2017 r5B12)"
- board text added: "R176"
- board text removed: "(02/2017 r5B12)"
- board text removed: "EEZ PSU power board (02/2017 r5B12)"

Commit message: X1 rotated
Parts:
- added X24: (no value), EEZ_Lib1:MINIFIT_39301039
- added X25: ZL262-5SG, con-samtec:SSW-105-02-S-S
- C89, C94: value EEEFK1H470P -> UWT1H220MCL
- L1, L9: device EEZ_Lib1:RN114 -> EEZ_Lib1:RN112
- R270, R6: value 0R -> 1R
- X1: value 39-30-1039 -> (none)
- X21: value SSW-113-02-T-D-RA -> ZL262-5SG; device EEZ_Lib1:SSW-113-02-T-D-RA -> con-samtec:SSW-105-02-S-S
- X22: value 282836-2 -> SSW-113-02-T-D-RA; device EEZ_Lib1:TBLOCK5.0_2 -> EEZ_Lib1:SSW-113-02-T-D-RA
- X23: value 39-30-1039 -> 282836-2; device EEZ_Lib1:MINIFIT_39301039 -> EEZ_Lib1:TBLOCK5.0_2
- moved X22 153.2 mm to (179.5, 97.8), flipped to the top, turned to 90 degrees
- moved X21 85.6 mm to (95.9, 116.1), turned to 0 degrees
- moved X23 52.8 mm to (326.4, 141.5), turned to 180 degrees
- moved C27 17.6 mm to (110.3, 129.2)
- moved C236 17.6 mm to (277.3, 129.2)
- moved R21 16.7 mm to (109.9, 135.3), turned to 90 degrees
- moved R278 16.7 mm to (276.9, 135.3), turned to 90 degrees
- moved R279 16.0 mm to (279.1, 138.8), turned to 180 degrees
- moved R24 16.0 mm to (112.1, 138.8), turned to 180 degrees
- moved IC48 8.98 mm to (289.7, 134.3), turned to 270 degrees
- moved IC3 8.98 mm to (122.7, 134.3), turned to 270 degrees
- moved X1 7.25 mm to (156.1, 81.6), turned to 180 degrees
- moved C1 1.81 mm to (154.7, 96.5)
- moved C214 1.81 mm to (321.7, 96.5)
- moved ZD19 1.71 mm to (313.6, 106.0)
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Connections:
- net !INT1: now also X22.8; no longer X21.8
- net !PS_RESET1: now also X22.5; no longer X21.5
- net +5V1: now also X22.2; no longer X21.2
- net AC_EARTH: now also X3.1; no longer X3.5
- net AC_IN3: now also X23.2; no longer X22.2
- net AC_IN4: now also X23.1; no longer X22.1
- net AC_IN_L: now also X3.5; no longer X3.1
- net AUX_USET_IN1: now also X22.11; no longer X21.11
- net CS_ADC1: now also X22.6; no longer X21.6
- net CS_DAC1: now also X22.4; no longer X21.4
- net CS_EXPANDER1: now also X22.3; no longer X21.3
- net DC+: now also X1.3; no longer X1.1
- net DC+1: now also X24.3; no longer X23.1
- net DC-1: now also X24.2; no longer X23.2
- net DC_OUT: now also X21.5
- net DC_OUT1: now also X25.5
- net EARTH: now also X1.1; no longer X1.3
- net EARTH1: now also X24.1; no longer X23.3
- net FB: now also X21.4
- net FB1: now also X25.4
- net GND1: now also X22.10, X22.12, X22.14; no longer X21.10, X21.12, X21.14
- net MCU_VCC1: now also X22.15; no longer X21.15
- net OUT+: now also X21.3
- net OUT+1: now also X22.23, X22.24, X22.25, X22.26, X25.3; no longer X21.23, X21.24, X21.25, X21.26
- net OUT-1: now also X22.17, X22.18, X22.19, X22.20; no longer X21.17, X21.18, X21.19, X21.20
- net PREG_OUT: now also X21.2
- net PREG_OUT1: now also X25.2
- net PS_MISO1: now also X22.9; no longer X21.9
- net PS_MOSI1: now also X22.1; no longer X21.1
- net PS_SCLK1: now also X22.7; no longer X21.7
- net SENSE+1: now also X22.22; no longer X21.22
- net SENSE-1: now also X22.21; no longer X21.21
- net SYNC3: now also X22.16; no longer X21.16
- net TEMP_NTC1: now also X22.13; no longer X21.13
- net V-: now also X21.1
- net V-1: now also X25.1
Routing:
- net DC_OUT1: track 120.4 -> 140.0 mm, vias 53 -> 54
- net DC_OUT: track 120.4 -> 140.0 mm, vias 53 -> 54
- net PREG_OUT: track 4.77 -> 21.6 mm, vias 0 -> 2
- net PREG_OUT1: track 4.77 -> 21.6 mm, vias 0 -> 2
- net FB: track 16.6 -> 32.7 mm
- net FB1: track 16.6 -> 32.7 mm
- net +VNR1: track 81.9 -> 66.4 mm, vias 19 -> 20
- net +VNR: track 81.9 -> 66.4 mm, vias 19 -> 20
- net OUT+: track 235.2 -> 243.7 mm
- net OUT+1: track 235.2 -> 243.7 mm
- net V-1: track 137.9 -> 144.8 mm, vias 11 -> 12
- net V-: track 137.9 -> 144.8 mm, vias 11 -> 12
- net DC-1: track 5.43 -> 2.35 mm
- net DC-: track 5.43 -> 2.35 mm
- net +5V: track 968.6 -> 970.0 mm
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Other:
- board text added: "1 -5V"
- board text added: "2 Pout"
- board text added: "3 Out+"
- board text added: "4 FB"
- board text added: "5 +Vin"
- board text added: "DC in+ 3"
- board text added: "Earth 1"
- board text added: "X21"
- board text removed: "DC in+ 1"
- board text removed: "Earth 3"

Commit message: X20 rotated
Parts:
- moved X20 18.9 mm to (237.9, 46.4), turned to 270 degrees
- moved J7 0.06 mm to (283.8, 4.45)
Routing:
- net AUDIO_OUT: track 113.2 -> 131.9 mm
- net LCDSD_CS: track 101.5 -> 116.5 mm
- net !LCD_INT: track 16.4 -> 29.2 mm
- net MOSI: track 325.9 -> 313.8 mm
- net MISO: track 305.7 -> 294.9 mm, vias 13 -> 12
- net LCD_CS: track 127.5 -> 117.1 mm
- net !LCD_PD: track 15.3 -> 25.1 mm
- net SYNC1: track 36.1 -> 45.4 mm
- net +3V3: track 732.7 -> 740.0 mm
- net SCLK: track 308.0 -> 302.3 mm, vias 10 -> 8
- net GND: track 447.2 -> 449.1 mm, vias 421 -> 416
- net !ADC1_SELECT: track 87.1 -> 86.5 mm
