File: Consolidated/Eagle files/EEZ PSU block diagram rev5.4.sch (EAGLE design)
At the start: 0 parts

Commit message: #38
Other:
- note added: "48 Vdc max. 3.2 A"
- note added: "5"
- note added: "Ch#1 40 V / 5 A"
- note added: "Ch#2 40 V / 5 A"
- note added: "Diagram revision: 5.4 (04/2017)"
- note removed: "+0...40 Vdc"
- note removed: "+48 Vdc"
- note removed: "4"
- note removed: "48-54 Vdc max. 3 A"
- note removed: "AC input (115/230 Vac)"
- note removed: "AC/DC module"
- note removed: "Ch#1 0-40 V or 0-80 V max. 5 A or 10 A"
- note removed: "Ch#2 0-40 V max. 5 A"
- note removed: "Diagram revision: 5.3 (02/2017)"
- note removed: "Post-regulator (linear)"
- note removed: "Power pre-regulator (SMPS)"

Commit message: block diagram updated
Other:
- note added: "3.2" TFT color display, 240x320 with touch screen"
- note added: "CC control loop (LTC2050HV, ½ TL072)"
- note added: "Reset SW"
- note removed: "!Reset! (optional)"
- note removed: "(LM25575)"
- note removed: "+5V SMPS"
- note removed: "240x320 TFT color display (SSD1289) + touch screen (XPT2046)"
- note removed: "Aux PCB"
- note removed: "CC control loop (½ TL072, OP27)"
- note removed: "Level shifter"
