File: Consolidated/Eagle files/EEZ PSU consolidated r5B13.brd (EAGLE design)
At the start: 337 x 150 mm, 555 parts, among them IC1 LTC3864EMSE#PBF, IC10 DAC8552IDGKTG4, IC11 ADG465SOT-23, IC12 TS5A9411DCKT, IC13 ADS1120IPWR, IC14 LP339D, IC15 TPD4E002DRL, IC16 TPD2E001DZDR, IC17 ADUM3160BRWZ, IC18 TLC5925IDBQR, IC19 Si8641EC-B-IS1, IC2 LP2951SO8, IC20 SI8651EC-B-IS1, IC21 SI8651EC-B-IS1, IC22 LD1117S33TR, IC23 Si8641EC-B-IS1, IC24 PCA21125T/Q900/1,1, IC25 AT25256B-SSHL-B, IC26 W5500, IC27 BC857BS, IC28 TLC555, IC29 SN74LVC08APWR, IC3 TL783CKTTR, IC30 SN74LV1T34DBVR, IC31 TPS3705-33D, IC32 SN74LVC2G02DCTR, IC33 74LVC1G125GW.125, IC34 TPA6205A1DGN, IC4 LTC3260EMSE#PBF, IC5 TL072D, IC6 TL072D, IC7 LTC2050HVCS8#PBF, IC8 MCP23S17-E/SS, IC9 REF5025AIDG4, J1 BS-244DSM-R, J2 1-726388-2, J3 BS-244DSM-G, J4 BS-244DSM-B, J5 BS-244DSM-R, J6 BS-244DSM-B, J7 693072010801, Q1 IRFR5305, Q10 MMBT5401, Q11 MMBT5551, Q12 MMBT5551, Q13 IRLL2705PBF, Q14 IRFR48ZPBF, Q15 IRLML2246TRPBF, Q16 2N7002, Q17 MMBT5551, Q18 MMBT5401, Q19 MMBT5551, Q2 MMBT5401, Q20 MMBT5551, Q21 BTA26-600, Q22 BTA26-600, Q23 IRLL2705PBF, Q24 2N7002, Q25 2N7002, Q26 IRLML2246TRPBF, Q27 IRLML2246TRPBF, Q28 IRLML2246TRPBF, Q29 IRLML2246TRPBF, Q3 2N7002, Q30 2N7002, Q31 IRLML2246TRPBF, Q32 2N7002, Q33 2N7002, Q4 IRFP250N, Q5 BC857C, Q6 BCP56-16.115, Q7 IRFR5305, Q8 BCP56-16.115, Q9 MMBT5401, SW1 A101SYCQ04, SW2 PEC12R-4225F-S0024, SW3 1301.9316, X1 39-30-1039, X10 826629-5, X11 2411-01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

Commit message: r5B13 Eagle files, gerbers
Parts:
- added JP10, JP9: 0R-JUMPA, jump-0r-smd:A0R-JMP
- added Q34: 2N7002, EEZ_Lib1:SOT103P240X110-3N
- added R179: 0R75?, rcl:R1206
- added R180: 47K, rcl:R0805
- added R65A, R65B: 0R030, EEZ_Lib1:R_2512-4WIRE
- added ZD16: PDZ5.6B, EEZ_Lib1:SOD323-W
- IC22: value LD1117S33TR -> LD1117ADT33TR
- R13, R20, R25: value 330K -> 316K
- R32, R59: value 2K2 -> n.c.
- R60, R70: value 1K91 -> 3K9 0.1%
- R62, R71: value 82R -> 82R 0.1%
- R63: value 0R16 -> 0R082
- R65: value 0R020 (1-3W) -> 0R030
- moved R92 43.1 mm to (22.5, 135.7), turned to 180 degrees
- moved R93 42.4 mm to (22.5, 133.7)
- moved Q20 40.9 mm to (26.7, 135.7), turned to 90 degrees
- moved C74 38.3 mm to (30.9, 135.7), turned to 90 degrees
- moved R101 36.8 mm to (32.8, 135.7), turned to 270 degrees
- moved R96 33.6 mm to (29.9, 132.7), turned to 180 degrees
- moved R94 11.4 mm to (35.8, 146.1), turned to 0 degrees
- moved R100 11.3 mm to (28.3, 145.9), turned to 90 degrees
- moved Q19 10.7 mm to (31.7, 145.9), turned to 270 degrees
- moved Q18 9.12 mm to (25.8, 101.2), turned to 90 degrees
- moved R95 7.69 mm to (25.8, 140.9), turned to 270 degrees
- moved C71 6.56 mm to (28.8, 140.0)
- moved R87 6.56 mm to (28.8, 141.9)
- moved Q17 6.42 mm to (35.1, 140.9)
- moved R86 6.41 mm to (31.8, 140.9)
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Connections:
- new net CURR_50MA: IC8.3, Q34.1, R180.2
- new net N$125: IC17.5, JP10.2
- new net N$54: IC17.13, JP9.2
- new net N$60: Q34.2, R179.1, R62.1
- net GND: now also JP9.3, R180.1, ZD16.A
- net N$169: now also R65A.2, R65B.2
- net N$200: now also R65A.1S, R65B.1S
- net N$201: now also R179.2; no longer R62.1
- net N$70: now also R65A.2S, R65B.2S
- net N$87: now also JP10.1; no longer IC17.5
- net N$91: now also JP9.1; no longer IC17.13
- net OUT-: now also Q34.3
- net POUT-: now also R65A.1, R65B.1
- net V+: now also ZD16.C
- net XUSB_GND: now also JP10.3
Routing:
- net CURR_50MA: track 0.00 -> 66.7 mm, vias 0 -> 2
- net N$25: track 16.2 -> 44.0 mm, vias 0 -> 2
- net OUT-: track 96.4 -> 119.1 mm, vias 8 -> 10
- net N$60: track 0.00 -> 18.0 mm
- net N$70: track 5.86 -> 21.9 mm
- net OUT+: track 235.2 -> 222.5 mm
- net N$200: track 14.8 -> 25.9 mm
- net DC_OUT: track 134.2 -> 123.7 mm, vias 54 -> 53
- net EARTH: track 314.8 -> 325.0 mm
- net SENSE_ERR: track 27.0 -> 18.7 mm
- net N$201: track 16.0 -> 8.31 mm
- net N$125: track 0.00 -> 6.95 mm
- net N$54: track 0.00 -> 6.10 mm
- net SENSE_PROT: track 82.2 -> 87.9 mm
- net N$91: track 7.12 -> 12.4 mm
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Other:
- board text added: "(09/2017 r5B13)"
- board text added: "(09/2017)"
- board text added: "EEZ AUX PS r5B13"
- board text added: "EEZ AUX PS r5B13 (09/2017)"
- board text added: "EEZ Arduino shield (09/2017 r5B12)"
- board text added: "EEZ PSU power board (09/2017 r5B13)"
- board text added: "IMPORTANT: JP9 and JP10"
- board text added: "JP10"
- board text added: "JP9"
- board text added: "Q34"
- board text added: "R179"
- board text added: "R180"
- board text added: "R65A"
- board text added: "R65B"
- board text added: "ZD16"
- board text added: "must be on the same position!"
- board text added: "r5B12 (09/2017)"
- board text removed: "(03/2017 r5B12)"
- board text removed: "(03/2017)"
- board text removed: "EEZ AUX PS r5B12a"
- board text removed: "EEZ AUX PS r5B12a (03/2017)"
- board text removed: "EEZ Arduino shield (03/2017 r5B12)"
- board text removed: "EEZ PSU power board (03/2017 r5B12)"
- board text removed: "r5B12 (03/2017)"
