File: Consolidated/Eagle files/EEZ PSU consolidated r5B13.sch (EAGLE design)
At the start: 543 parts, among them IC1 LTC3864EMSE#PBF, IC10 DAC8552IDGKTG4, IC11 ADG465SOT-23, IC12 TS5A9411DCKT, IC13 ADS1120IPWR, IC14 LP339D, IC15 TPD4E002DRL, IC16 TPD2E001DZDR, IC17 ADUM3160BRWZ, IC18 TLC5925IDBQR, IC19 Si8641EC-B-IS1, IC2 LP2951SO8, IC20 SI8651EC-B-IS1, IC21 SI8651EC-B-IS1, IC22 LD1117S33TR, IC23 Si8641EC-B-IS1, IC24 PCA21125T/Q900/1,1, IC25 AT25256B-SSHL-B, IC26 W5500, IC27 BC857BS, IC28 TLC555, IC29 SN74LVC08APWR, IC3 TL783CKTTR, IC30 SN74LV1T34DBVR, IC31 TPS3705-33D, IC32 SN74LVC2G02DCTR, IC33 74LVC1G125GW.125, IC34 TPA6205A1DGN, IC4 LTC3260EMSE#PBF, IC5 TL072D, IC6 TL072D, IC7 LTC2050HVCS8#PBF, IC8 MCP23S17-E/SS, IC9 REF5025AIDG4, J1 BS-244DSM-R, J2 1-726388-2, J3 BS-244DSM-G, J4 BS-244DSM-B, J5 BS-244DSM-R, J6 BS-244DSM-B, J7 693072010801, Q1 IRFR5305, Q10 MMBT5401, Q11 MMBT5551, Q12 MMBT5551, Q13 IRLL2705PBF, Q14 IRFR48ZPBF, Q15 IRLML2246TRPBF, Q16 2N7002, Q17 MMBT5551, Q18 MMBT5401, Q19 MMBT5551, Q2 MMBT5401, Q20 MMBT5551, Q21 BTA26-600, Q22 BTA26-600, Q23 IRLL2705PBF, Q24 2N7002, Q25 2N7002, Q26 IRLML2246TRPBF, Q27 IRLML2246TRPBF, Q28 IRLML2246TRPBF, Q29 IRLML2246TRPBF, Q3 2N7002, Q30 2N7002, Q31 IRLML2246TRPBF, Q32 2N7002, Q33 2N7002, Q4 IRFP250N, Q5 BC857C, Q6 BCP56-16.115, Q7 IRFR5305, Q8 BCP56-16.115, Q9 MMBT5401, SW1 A101SYCQ04, SW2 PEC12R-4225F-S0024, SW3 1301.9316, X1 39-30-1039, X10 826629-5, X11 2411-01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

Commit message: r5B13 Eagle files, gerbers
Parts:
- added JP10, JP9: 0R-JUMPA, jump-0r-smd:0R-JUMPA
- added Q34: 2N7002, EEZ_Lib1:2N7002
- added R179: 0R75?, rcl:R-EU_R1206
- added R180: 47K, rcl:R-EU_R0805
- added R65A, R65B: 0R030, EEZ_Lib1:R-EU_4WIRE2512
- added ZD16: PDZ5.6B, EEZ_Lib1:ZENER-DIODESOD323
- IC22: value LD1117S33TR -> LD1117ADT33TR
- R13, R20, R25: value 330K -> 316K
- R32, R59: value 2K2 -> n.c.
- R60, R70: value 1K91 -> 3K9 0.1%
- R62, R71: value 82R -> 82R 0.1%
- R63: value 0R16 -> 0R082
- R65: value 0R020 (1-3W) -> 0R030
Connections:
- new net CURR_50MA: IC8.GPB2, Q34.G, R180.2
- new net N$125: IC17.SPU, JP10-0R.2
- new net N$54: IC17.SPD, JP9-0R.2
- new net N$60: Q34.S, R179.1, R62.1
- net GND: now also JP9-0R.3, R180.1, ZD16.A
- net N$169: now also R65A.2, R65B.2
- net N$200: now also R65A.1S, R65B.1S
- net N$201: now also R179.2; no longer R62.1
- net N$70: now also R65A.2S, R65B.2S
- net N$87: now also JP10-0R.1; no longer IC17.SPU
- net N$91: now also JP9-0R.1; no longer IC17.SPD
- net OUT-: now also Q34.D
- net POUT-: now also R65A.1, R65B.1
- net V+: now also ZD16.C
- net XUSB_GND: now also JP10-0R.3
Other:
- note added: "10"
- note added: "11-15"
- note added: "3K9"
- note added: "4K7"
- note added: "6K2"
- note added: "CV/CC linear post-regulator, Output enable and "down-programmer""
- note added: "Current control loop (tripple range)"
- note added: "Current range 5 A"
- note added: "Current range 50 mA"
- note added: "Current range 500 mA"
- note added: "EEZ PSU consolidated r5B13 - Sheet: 3/12"
- note added: "Note 3.1: Q4 is mounted on the external heatsink"
- note added: "Note 3.2: Use power resistors with the lowest possible TCR (± 75 ppm/oC or better)"
- note removed: "10-15"
- note removed: "1K91"
- note removed: "2K7 (not tested)"
- note removed: "3K16 (not tested)"
- note removed: "CV/CC linear post-regulator"
- note removed: "Current control loop"
- note removed: "Current range HIGH"
- note removed: "Current range LOW"
- note removed: "Note 3.1: Q4 is mounted on the external heatsink (e.g. RAD-A4463/120)"
- note removed: "Note 3.2: Use power resistor with the lowest possible TCR (± 75 ppm/oC or better)"
- note removed: "Output enable and "down-programmer""
- moved on the sheet: C52, C53, C81, C82, C83, C84, C85, D10, D9, FB2, FB5, FB6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
