File: Consolidated/Eagle files/EEZ PSU r5B13 panel.brd (EAGLE design)
At the start: 337 x 150 mm, 815 parts, among them IC1 LTC3864EMSE#PBF, IC10 DAC8552IDGKTG4, IC11 ADG465SOT-23, IC12 TS5A9411DCKT, IC13 ADS1120IPWR, IC14 LP339D, IC15 TPD4E002DRL, IC16 TPD2E001DZDR, IC17 ADUM3160BRWZ, IC18 TLC5925IDBQR, IC19 Si8641EC-B-IS1, IC2 LP2951SO8, IC20 SI8651EC-B-IS1, IC21 SI8651EC-B-IS1, IC22 LD1117ADT33TR, IC23 Si8641EC-B-IS1, IC24 PCA21125T/Q900/1,1, IC25 AT25256B-SSHL-B, IC26 W5500, IC27 BC857BS, IC28 TLC555, IC29 SN74LVC08APWR, IC3 TL783CKTTR, IC30 SN74LV1T34DBVR, IC31 TPS3705-33D, IC32 SN74LVC2G02DCTR, IC33 74LVC1G125GW.125, IC34 TPA6205A1DGN, IC35 DAC8552IDGKTG4, IC36 ADS1120IPWR, IC37 LTC2050HVCS8#PBF, IC38 TL072D, IC39 TL072D, IC4 LTC3260EMSE#PBF, IC40 REF5025AIDG4, IC41 LTC3864EMSE#PBF, IC42 TS5A9411DCKT, IC43 ADG465SOT-23, IC44 LP339D, IC45 LTC3260EMSE#PBF, IC46 LP2951SO8, IC47 MCP23S17-E/SS, IC48 TL783CKTTR, IC5 TL072D, IC6 TL072D, IC7 LTC2050HVCS8#PBF, IC8 MCP23S17-E/SS, IC9 REF5025AIDG4, J1 BS-244DSM-R, J2 1-726388-2, J3 BS-244DSM-G, J4 BS-244DSM-B, J5 BS-244DSM-R, J6 BS-244DSM-B, J7 693072010801, Q1 IRFR5305, Q10 MMBT5401, Q11 MMBT5551, Q12 MMBT5551, Q13 IRLL2705PBF, Q14 IRFR48ZPBF, Q15 IRLML2246TRPBF, Q16 2N7002, Q17 MMBT5551, Q18 MMBT5401, Q19 MMBT5551, Q2 MMBT5401, Q20 MMBT5551, Q21 BTA26-600, Q22 BTA26-600, Q23 IRLL2705PBF, Q24 2N7002, Q25 2N7002, Q26 IRLML2246TRPBF, Q27 IRLML2246TRPBF, Q28 IRLML2246TRPBF, Q29 IRLML2246TRPBF, Q3 2N7002, Q30 2N7002, Q31 IRLML2246TRPBF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

Commit message: r5B13 Eagle files, gerbers
Parts:
- added JP12, JP13: 0R-JUMPA, jump-0r-smd:A0R-JMP
- added Q54: IRFR48ZPBF, EEZ_Lib1:TO229P990X239-3N
- added Q55: 2N7002, EEZ_Lib1:SOT103P240X110-3N
- added R282: 1K8, rcl:R0805
- added R283: 0R082, rcl:R1210
- added R284: 0R75?, rcl:R1206
- added R285: 47K, rcl:R0805
- added R65A, R65A1, R65B, R65B1: 0R030, EEZ_Lib1:R_2512-4WIRE
- added ZD20: SMAJ51A, EEZ_Lib1:DO214AA
- added ZD21: PDZ5.6B, EEZ_Lib1:SOD323-W
- Q34: value IRFP250N -> 2N7002; device EEZ_Lib1:TO247BH-CLR -> EEZ_Lib1:SOT103P240X110-3N
- Q35: value BCP56-16.115 -> IRFP250N; device EEZ_Lib1:SOT230P700X180-4N -> EEZ_Lib1:TO247BH-CLR
- Q36: value MMBT5551 -> BCP56-16.115; device transistor:SOT23-BEC -> EEZ_Lib1:SOT230P700X180-4N
- Q37: value BCP56-16.115 -> MMBT5551; device EEZ_Lib1:SOT230P700X180-4N -> transistor:SOT23-BEC
- Q38: value MMBT5401 -> BCP56-16.115; device transistor:SOT23-BEC -> EEZ_Lib1:SOT230P700X180-4N
- Q40, Q50: value MMBT5551 -> MMBT5401
- Q41: value BC857C -> MMBT5551
- Q42: value 2N7002 -> BC857C; device EEZ_Lib1:SOT103P240X110-3N -> transistor:SOT23-BEC
- Q43: value IRLML2246TRPBF -> 2N7002; device EEZ_Lib1:SOT95P237X112-3N -> EEZ_Lib1:SOT103P240X110-3N
- Q44: value IRFR5305 -> IRLML2246TRPBF; device EEZ_Lib1:TO229P990X239-3N -> EEZ_Lib1:SOT95P237X112-3N
- Q45: value MMBT5401 -> IRFR5305; device transistor:SOT23-BEC -> EEZ_Lib1:TO229P990X239-3N
- Q46: value IRFR5305 -> MMBT5401; device EEZ_Lib1:TO229P990X239-3N -> transistor:SOT23-BEC
- Q47: value 2N7002 -> IRFR5305; device EEZ_Lib1:SOT103P240X110-3N -> EEZ_Lib1:TO229P990X239-3N
- Q48: value MMBT5551 -> 2N7002; device transistor:SOT23-BEC -> EEZ_Lib1:SOT103P240X110-3N
- Q49: value MMBT5401 -> MMBT5551
- Q52: value IRLL2705PBF -> MMBT5551; device transistor-power:SOT223 -> transistor:SOT23-BEC
- Q53: value IRFR48ZPBF -> IRLL2705PBF; device EEZ_Lib1:TO229P990X239-3N -> transistor-power:SOT223
- R13, R20, R25: value 330K -> 316K
- R179: value 2K2 -> 0R75?; device rcl:R0805 -> rcl:R1206
- R180: value 2K2 -> 47K
- R182, R183: value 10K -> n.c.
- R184: value 10R -> 10K; device rcl:R1206 -> rcl:R0805
- R186: value 2K2 -> 10R; device rcl:R0805 -> rcl:R1206
- R187: value 5K6 -> 10K
- R188: value 5K6 -> 2K2
- R189, R190: value 5K1 -> 5K6
- R191, R192: value 10K -> 5K1
- R195, R196, R213, R257: value 220R -> 10K
- R197: value 470R -> 220R
- R198: value 100R -> 220R
- R199: value 1K -> 470R
- R200: value 470R -> 100R
- R201: value 16K -> 1K
- R202: value 750R -> 470R
- R203: value 2K2 -> 16K
- R204: value 2K2 -> 750R
- R205: value 220R -> 2K2
- R206: value 1K -> 2K2
- R207: value 47K -> 220R
- R208, R244: value 10K -> 1K
- R209, R237, R254, R255: value 10K -> 47K
- R210: value 100K -> 10K
- R212: value 220R -> 100K
- R214: value 1K8 -> 220R
- R215: value 51K -> 220R
- R216: value 100K -> 1K8
- R217: value 7K5 0.1% -> 51K
- R218: value 100K 0.1% -> 100K
- R219: value 100K 0.1% -> 7K5 0.1%
- R220, R221: value 24K 0.1% -> 100K 0.1%
- R222: value 7K5 0.1% -> 24K 0.1%
- R223: value 2K 0.1% -> 24K 0.1%
- R224: value 82R 0.1% -> 7K5 0.1%
- R225: value 82R 0.1% -> 3K9 0.1%
- R226: value 2K 0.1% -> 82R 0.1%
- R227: value 10K -> 82R 0.1%
- R228: value 0R -> 3K9 0.1%
- R229: value 330K -> 10K
- R230: value 4K7 -> 0R
- R231: value 10R -> 316K; device rcl:R1206 -> rcl:R0805
- R232: value 100K -> 4K7
- R233: value 10K -> 10R; device rcl:R0805 -> rcl:R1206
- R235, R256: value 47K -> 10K
- R236: value R010/2W -> 100K; device rcl:R2512 -> rcl:R0805
- R238: value 100R -> R010/2W; device rcl:R0805 -> rcl:R2512
- R239: value 12K -> 10K; device rcl:R1206 -> rcl:R0805
- R240: value 330K -> 100R
- R241: value 100K -> 12K; device rcl:R0805 -> rcl:R1206
- R242: value 1K -> 316K
- R245: value n.c. -> 100K
- R246: value 100R -> 10K
- R247: value 330R -> n.c.
- R248: value 750R -> 100R
- R249: value 1K -> 330R
- R250: value 330R -> 750R
- R251: value 750R -> 1K
- R252: value 47K -> 330R
- R253: value 47K -> 750R
- R258: value 220R -> 47K
- R261: value 2R2/2W -> 220R; device rcl:R2512 -> rcl:R0805
- R262: value 330K -> 220R
- R263: value 1K -> 2R2/2W; device rcl:R0805 -> rcl:R2512
- R264: value 2K2 -> 316K
- R265: value 2K2 -> 1K
- R266: value 10R -> 2K2; device rcl:R1206 -> rcl:R0805
- R267: value n.c. -> 2K2
- R268: value n.c. -> 10R
- R269: value 220R -> n.c.
- R270: value 10K -> n.c.; device rcl:R0805 -> rcl:R1206
- R271: value 1R -> 220R
- R272: value n.c. -> 10K
- R273: value 0R020 (1-3W) -> 1R; device EEZ_Lib1:R_2512-4WIRE -> rcl:R0805
- R274: value 47K -> n.c.
- R275: value 47K -> 0R030; device rcl:R0805 -> EEZ_Lib1:R_2512-4WIRE
- R276: value 16K -> 47K
- R277: value 5K1 -> 47K
- R278: value 10K -> 16K
- R279: value 220R -> 5K1
- R280: value 1K8 -> 10K
- R281: value 0R16 -> 220R; device rcl:R1210 -> rcl:R0805
- R32, R59: value 2K2 -> n.c.
- R60, R70: value 2K 0.1% -> 3K9 0.1%
- R63: value 0R16 -> 0R082
- R65: value 0R020 (1-3W) -> 0R030
- ZD16: value BZX384-C15 -> PDZ5.6B
- ZD17: value PDZ6.2B -> BZX384-C15
- ZD18: value n.c. -> PDZ6.2B; device EEZ_Lib1:DO214AA -> EEZ_Lib1:SOD323-W
- ZD19: value SMAJ51A -> n.c.
- moved JP9 270.6 mm to (27.1, 64.4)
- moved Q34 231.5 mm to (21.6, 94.6), turned to 180 degrees
- moved R180 186.5 mm to (25.8, 93.5)
- moved JP10 183.0 mm to (45.8, 63.3), turned to 270 degrees
- moved R179 178.9 mm to (31.2, 92.7), turned to 270 degrees
- moved ZD16 173.3 mm to (81.2, 145.9), turned to 180 degrees
- moved R267 138.2 mm to (182.5, 133.7)
- moved R272 131.6 mm to (198.7, 116.3), turned to 180 degrees
- moved R274 131.3 mm to (330.1, 107.7)
- moved R269 121.9 mm to (310.1, 80.4), turned to 0 degrees
- moved R270 111.3 mm to (308.7, 133.6), flipped to the bottom
- moved R277 105.9 mm to (196.2, 87.2), turned to 270 degrees
- moved R276 101.1 mm to (198.2, 87.2), turned to 270 degrees
- moved JP11 96.1 mm to (291.4, 122.6), turned to 180 degrees
- moved R271 95.9 mm to (193.7, 116.9), turned to 90 degrees
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Connections:
- net N$157 renamed EOUT_B
- net N$159 renamed EOUT_A
- removed net N$231 (its old number): IC39.6, IC39.7, JP11.1
- removed net N$239 (its old number): IC41.12, R271.1
- removed net N$242 (its old number): C208.1, Q45.C, Q47.3, R245.1
- removed net N$246 (its old number): C230.2, IC43.1, R242.1
- removed net N$267 (its old number): IC45.4, R241.2, R262.1
- removed net N$270 (its old number): LED1.A, R272.1
- removed net N$275: R225.1, R273.1S
- new net CURR_50MA: IC8.3, Q34.1, R180.2
- new net CURR_50MA1: IC47.3, Q55.1, R285.2
- new net N$157: IC17.5, JP10.2
- new net N$159: IC39.3, R181.2
- new net N$230: Q42.B, R205.2
- new net N$238: C193.1, R239.1
- new net N$241: IC41.2, R237.1
- new net N$245: C203.1, C231.+, FB9.P$1, IC45.12, R242.1
- new net N$265: IC45.15, R242.2, R245.1
- new net N$268: IC45.4, R243.2, R264.1
- new net N$274: C235.+, FB10.P$1, IC46.1, R278.1, R280.1
- new net N$279: R275.2S, R283.1, R65A1.2S, R65B1.2S
- new net N$280: Q55.2, R226.1, R284.1
- net !DP_DRIVE1: now also Q38.1, R208.1, R213.1; no longer Q37.1, R206.1, R211.1
- net !INT1: now also JP12.2; no longer JP10.2
- net !PS_DRDY1: now also JP12.3; no longer JP10.3
- net !SET_100%1: now also Q48.1; no longer Q47.1
- net !SET_DP1: now also Q44.1, R218.2; no longer Q43.1, R216.2
- net +5V1: now also Q37.B, Q44.2, R191.2, R192.2, R218.1, R257.2; no longer Q36.B, Q43.2, R189.2, R190.2, R216.1, R255.2
- net +VNR1: now also R281.1; no longer R279.1
- net +VREF1: now also R272.1; no longer R270.1
- net -12V1: now also R207.2, R208.2; no longer R205.2, R206.2
- net -5VOUT1: now also R264.2; no longer R262.2
- net AC_IN3: now also ZD19.C; no longer ZD18.C
- net AC_IN4: now also R270.2, ZD19.A; no longer R268.2, ZD18.A
- net AUX_USET_IN1: now also R244.2; no longer R242.2
- net CC_ACTIVE1: now also R190.2, R192.1; no longer R188.2, R190.1
- net CURR_500MA1: now also Q53.1, R277.2; no longer Q52.1, R275.2
- net CURR_5A1: now also Q54.1, R276.2; no longer Q53.1, R274.2
- net CV_ACTIVE1: now also R189.2, R191.1; no longer R187.2, R189.1
- net DC+: now also L1.3; no longer L1.2
- net DC+1: now also L9.3; no longer L9.2
- net DC_BIAS1: now also Q36.2, Q36.4, R214.2, R215.2, R268.2; no longer Q35.2, Q35.4, R212.2, R213.2, R266.2
- net DC_OUT: now also L1.4; no longer L1.3
- net DC_OUT1: now also L9.4, R238.1, R241.1, R268.1, R274.2, ZD20.C; no longer L9.3, R236.1, R239.1, R266.1, R272.2, ZD19.C
- net DP_LED1: now also Q44.3, R213.2; no longer Q43.3, R211.2
- net EARTH1: now also R269.2; no longer R267.2
- net ENC_A: now also C138.1, MCU.A9, R165.1; no longer C137.2, MCU.A8, R157.1
- net ENC_B: now also C137.2, MCU.A8, R157.1; no longer C138.1, MCU.A9, R165.1
- net FB1: now also Q48.2, R231.2, R232.1, R247.2; no longer Q47.2, R229.2, R230.1, R245.2
- net GCOM1: now also JP13.2, R219.1, R225.1; no longer JP11.2, R217.1, R223.1
- net GND: now also JP9.3, L1.2, R180.1, ZD16.A; no longer L1.4
- net GND1: now also JP13.3, L9.2, Q43.2, Q45.2, Q52.E, R188.1, R204.1, R212.1, R217.1, R229.2, R233.1, R241.2, R243.1, R245.2, R255.1, R258.1, R266.1, R271.2, R276.1, R277.1, R279.2, R282.2, R285.1, ZD20.A, ZD21.A; no longer JP11.3, L9.4, Q42.2, Q44.2, Q50.E, R186.1, R202.1, R210.1, R215.1, R227.2, R231.1, R239.2, R241.1, R243.2, R253.1, R256.1, R264.1, R269.2, R274.1, R275.1, R277.2, R280.2, ZD19.A
- net HEATSINK1: now also R269.1; no longer R267.1
- net INT_EXP1: now also JP12.1; no longer JP10.1
- net ISENSE+1: now also R225.2, R226.2; no longer R223.2, R224.2
- net ISENSE-1: now also R227.2, R228.1; no longer R225.2, R226.1
- net I_MON1: now also R228.2, R260.1; no longer R226.2, R258.1
- net I_SERVO1: now also R211.1; no longer R209.1
- net I_SET1: now also R181.1, R262.1; no longer R179.1, R260.1
- net LOOP_CTRL1: now also R199.1; no longer R197.1
- net L_OUT12: now also R231.1, R235.1, R236.1, R248.1; no longer R229.1, R233.1, R234.1, R246.1
- net MODE1: now also JP11.2; no longer JP9.2
- net N$125: now also Q34.2, R179.1, R62.1; no longer IC39.3, R179.2
- net N$154: now also IC17.13, JP9.2; no longer IC38.3, R182.2, R195.2
- net N$168: now also IC38.3, R184.2, R197.2; no longer C159.1, D27.C, IC38.2, R183.2, R196.2
- net N$169: now also R65A.2, R65B.2
- net N$179: now also C159.1, D27.C, IC38.2, R185.2, R198.2; no longer C164.2, C184.2, IC36.12, R184.2
- net N$180: now also C164.2, C184.2, IC36.12, R186.2; no longer IC44.1, IC44.2, R187.1
- net N$189: now also IC44.1, IC44.2, R189.1; no longer IC38.5, R191.2, R217.2, R218.1
- net N$191: now also IC38.5, R193.2, R219.2, R220.1; no longer IC38.6, R192.2, R219.1, R222.2
- net N$192: now also IC38.6, R194.2, R224.2; no longer C170.1, R219.2
- net N$196: now also C170.1, R221.2, R223.1; no longer C168.1, R218.2, R220.1
- net N$200: now also R65A.1S, R65B.1S
- net N$201: now also R179.2; no longer R62.1
- net N$202: now also C168.1, R220.2, R222.1; no longer C167.2, R191.1
- net N$203: now also C167.2, R193.1; no longer C169.2, R192.1
- net N$204: now also C169.2; no longer C173.2
- net N$205: now also C173.2, R196.1; no longer D26.C, IC39.2, R178.2, R193.2, R194.2
- net N$206: now also D26.C, IC39.2, R178.2, R195.2, R196.2; no longer C174.2, R195.1
- net N$209: now also C174.2, R197.1; no longer C175.2, R196.1
- net N$210: now also C175.2, R198.1; no longer D30.C, D32.A, Q34.G, R199.1
- net N$211: now also D30.C, D32.A, Q35.G, R201.1; no longer D30.A, Q35.3
- net N$212: now also D30.A, Q36.3; no longer D31.A, Q35.1, R198.1, R200.2
- net N$213: now also D31.A, Q36.1, R200.1, R202.2; no longer D31.C, ZD16.C
- net N$214: now also D31.C, ZD17.C; no longer C176.1, R200.1
- net N$215: now also C176.1, R202.1; no longer D32.C, ZD17.C
- net N$216: now also D32.C, ZD18.C; no longer Q44.3, R203.1, R204.1, R261.1
- net N$217: now also Q45.3, R205.1, R206.1, R263.1; no longer D33.A, Q41.C, Q44.1, R204.2
- net N$218: now also D33.A, Q42.C, Q45.1, R206.2; no longer Q40.E, R197.2
- net N$219: now also Q41.E, R199.2; no longer IC44.13, IC44.14, R188.1
- net N$220: now also IC44.13, IC44.14, R190.1; no longer IC44.5, IC44.6, R208.2
- net N$221: now also IC44.5, IC44.6, R210.2; no longer IC44.11, IC44.8, R209.2
- net N$222: now also IC44.11, IC44.8, R211.2; no longer IC44.7, IC44.9, R186.2, R207.1
- net N$223: now also IC44.7, IC44.9, R188.2, R209.1; no longer IC44.10, IC44.4, R185.2, R227.1
- net N$224: now also IC44.10, IC44.4, R187.2, R229.1; no longer Q39.E, R212.1
- net N$225: now also Q40.E, R214.1; no longer Q38.E, R213.1
- net N$226: now also Q39.E, R215.1; no longer Q36.E, R214.2
- net N$227: now also Q37.E, R216.2; no longer Q40.B, R201.1, R202.2, R264.2
- net N$228: now also Q41.B, R203.1, R204.2, R266.2; no longer Q37.3, R205.1
- net N$229: now also Q38.3, R207.1; no longer Q41.B, R203.2
- net N$232: now also IC39.6, IC39.7, JP13.1; no longer C159.2, R228.1
- net N$233: now also C159.2, R230.1; no longer C190.2, R231.2
- net N$234: now also C190.2, R233.2; no longer C208.2, D35.A, Q45.B, R232.1, R234.2
- net N$235: now also C208.2, D35.A, Q46.B, R234.1, R236.2; no longer D35.C, Q45.E, R233.2
- net N$236: now also D35.C, Q46.E, R235.2; no longer C194.1, IC41.6, R237.2
- net N$237: now also C194.1, IC41.6, R239.2; no longer C193.1, R237.1
- net N$240: now also IC41.12, R273.1; no longer IC41.2, R235.1
- net N$243: now also C208.1, Q46.C, Q48.3, R247.1; no longer C221.1, L6.1, L7.2, R238.1, R246.2
- net N$244: now also C221.1, L6.1, L7.2, R248.2; no longer C203.1, C231.+, FB9.P$1, IC45.12
- net N$247: now also C230.2, IC43.1; no longer IC41.8
- net N$248: now also IC41.8, R246.1; no longer C209.2, Q49.B, R247.1, R248.2, R265.2
- net N$249: now also C209.2, Q50.B, R249.1, R250.2, R267.2; no longer C211.2, Q49.C, R252.1, R254.2
- net N$250: now also C211.2, Q50.C, R254.1, R256.2; no longer Q48.C, R249.1
- net N$251: now also Q49.C; no longer C210.1, Q48.B, R250.2
- net N$252: now also C210.1, Q49.B, R253.1; no longer C211.1, Q50.B, R253.2
- net N$253: now also C211.1, R254.2, R255.2; no longer R254.1, R256.2
- net N$254: now also Q52.B, R256.1, R258.2; no longer C216.2, IC36.10, R257.2
- net N$255: now also C216.2, IC36.10, R259.2; no longer C217.2, IC36.7, R258.2
- net N$256: now also C217.2, IC36.7, R260.2; no longer C218.2, IC36.11, R259.2
- net N$257: now also C218.2, IC36.11, R261.2; no longer C219.1, IC36.6, R260.2
- net N$258: now also C219.1, IC36.6, R262.2; no longer R193.1, R263.2
- net N$259: now also R195.1, R265.2; no longer C157.1, R263.1
- net N$260: now also C157.1; no longer R249.2
- net N$261: now also R251.2, R267.1; no longer C228.2, R268.1
- net N$262: now also C228.2, R270.1; no longer C229.1, IC39.5, R269.1, R270.2
- net N$263: now also C229.1, IC39.5, R271.1, R272.2; no longer Q46.1, R271.2
- net N$264: now also Q47.1, R273.2; no longer IC45.15, R240.2, R243.1
- net N$271: now also LED1.A, R274.1; no longer Q53.3, R273.2
- net N$272: now also Q54.3, R275.2, R65A1.2, R65B1.2; no longer IC46.7, R276.2, R277.1
- net N$273: now also IC46.7, R278.2, R279.1; no longer C235.+, FB10.P$1, IC46.1, R276.1, R278.1
- net N$276: now also R227.1, R275.1S, R65A1.1S, R65B1.1S; no longer Q52.3, R224.1, R281.2
- net N$277: now also Q53.3, R283.2, R284.2; no longer IC48.1, R279.2, R280.1
- net N$278: now also IC48.1, R281.2, R282.1; no longer R273.2S, R281.1
- net N$70: now also R65A.2S, R65B.2S
- net N$87: now also JP10.1; no longer IC17.5
- net N$91: now also JP9.1; no longer IC17.13
- net OUT+1: now also Q35.S, Q42.E, Q50.E, R182.1, R203.2, R234.2, R249.2, R263.2, ZD17.A; no longer Q34.S, Q41.E, Q49.E, R180.1, R199.2, R232.2, R247.2, R261.2, ZD16.A
- net OUT-: now also Q34.3
- net OUT-1: now also Q49.E, Q53.4, Q54.2, Q55.3, R183.2, R252.1; no longer Q48.E, Q52.2, Q52.4, R181.2, R250.1
- net POST_OE1: now also Q43.3, R216.1; no longer Q42.3, R214.1
- net POUT-: now also R65A.1, R65B.1
- net POUT-1: now also R275.1, R65A1.1, R65B1.1; no longer R273.1
- net PREG_OUT1: now also Q35.D, R240.2; no longer Q34.D, R238.2
- net PRE_OE1: now also Q43.1, R212.2, R246.2; no longer Q42.1, R210.2, R244.2
- net PWRGOOD1: now also R280.2; no longer R278.2
- net Q7C1: now also Q37.C, Q39.C, Q40.B; no longer Q36.C, Q38.B, Q38.C
- net Q9C1: now also Q38.2, Q38.4, ZD18.A; no longer Q37.2, Q37.4, ZD17.A
- net SENSE+1: now also R182.2, R222.2, R250.1; no longer R180.2, R220.2, R248.1
- net SENSE-1: now also R183.1, R223.2, R253.2; no longer R181.1, R221.2, R251.2
- net SENSE1: now also Q47.3, R238.2; no longer Q46.3, R236.2
- net SENSE_ERR1: now also Q52.C, R257.1; no longer Q51.C, R255.1
- net SENSE_PROT1: now also Q41.C, Q51.C, R200.2, R217.2; no longer Q39.C, Q50.C, R198.2, R215.2
- net SGND1: now also JP11.1, R232.2, R237.2; no longer JP9.1, R230.2, R235.2
- net SW1: now also Q47.2; no longer Q46.2
- net SYNC3: now also JP11.3; no longer JP9.3
- net U_MON1: now also R185.1, R224.1, R259.1; no longer R183.1, R222.1, R257.1
- net U_SERVO1: now also R210.1, R230.2; no longer R208.1, R228.2
- net U_SET_OUT1: now also R184.1, R261.1; no longer R182.1, R259.1
- net V+: now also ZD16.C
- net V+1: now also R186.1, R209.2, ZD21.C; no longer R184.1, R207.2
- net V-1: now also R187.1; no longer R185.1
- net XUSB_GND: now also JP10.3
Routing:
- net CURR_50MA: track 0.00 -> 66.7 mm, vias 0 -> 2
- net CURR_50MA1: track 0.00 -> 66.7 mm, vias 0 -> 2
- net N$221: track 55.5 -> 8.19 mm, vias 4 -> 2
- net N$222: track 9.85 -> 55.5 mm, vias 0 -> 4
- net N$250: track 3.63 -> 46.4 mm, vias 0 -> 2
- net N$25: track 16.2 -> 44.0 mm, vias 0 -> 2
- net OUT-: track 96.4 -> 119.1 mm, vias 8 -> 10
- net OUT-1: track 96.4 -> 119.1 mm, vias 8 -> 10
- net N$210: track 25.3 -> 3.14 mm, vias 1 -> 0
- net N$279: track 0.00 -> 21.9 mm
- net N$205: track 23.7 -> 2.04 mm
- net N$211: track 4.70 -> 25.3 mm, vias 0 -> 1
- net N$206: track 3.12 -> 23.3 mm
- net N$159: track 0.00 -> 19.2 mm
- net N$280: track 0.00 -> 18.0 mm
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- added copper zone on layer 1, net N$240
- added copper zone on layer 1, net N$245
- added copper zone on layer 1, net N$272
- added copper zone on layer 1, net N$275
- removed copper zone on layer 1, net N$239 (its old number)
- removed copper zone on layer 1, net N$243
- removed copper zone on layer 1, net N$271
- removed copper zone on layer 1, net N$274
Other:
- board text added: "(09/2017 r5B13)"
- board text added: "(09/2017)"
- board text added: "EEZ AUX PS r5B13"
- board text added: "EEZ AUX PS r5B13 (09/2017)"
- board text added: "EEZ Arduino shield (09/2017 r5B12)"
- board text added: "EEZ PSU power board (09/2017 r5B13)"
- board text added: "IMPORTANT: JP9 and JP10"
- board text added: "JP10"
- board text added: "JP9"
- board text added: "Q34"
- board text added: "R179"
- board text added: "R180"
- board text added: "R65A"
- board text added: "R65B"
- board text added: "ZD16"
- board text added: "must be on the same position!"
- board text added: "r5B12 (09/2017)"
- board text removed: "(03/2017 r5B12)"
- board text removed: "(03/2017)"
- board text removed: "EEZ AUX PS r5B12a"
- board text removed: "EEZ AUX PS r5B12a (03/2017)"
- board text removed: "EEZ Arduino shield (03/2017 r5B12)"
- board text removed: "EEZ PSU power board (03/2017 r5B12)"
- board text removed: "r5B12 (03/2017)"
