File: Consolidated/Eagle files/EEZ PSU consolidated r5B13a.sch (EAGLE design)
At the start: 550 parts, among them IC1 LTC3864EMSE#PBF, IC10 DAC8552IDGKTG4, IC11 ADG465SOT-23, IC12 TS5A9411DCKT, IC13 ADS1120IPWR, IC14 LP339D, IC15 TPD4E002DRL, IC16 TPD2E001DZDR, IC17 ADUM3160BRWZ, IC18 TLC5925IDBQR, IC19 Si8641EC-B-IS1, IC2 LP2951SO8, IC20 SI8651EC-B-IS1, IC21 SI8651EC-B-IS1, IC22 LD1117ADT33TR, IC23 Si8641EC-B-IS1, IC24 PCA21125T/Q900/1,1, IC25 AT25256B-SSHL-B, IC26 W5500, IC27 BC857BS, IC28 TLC555, IC29 SN74LVC08APWR, IC3 TL783CKTTR, IC30 SN74LV1T34DBVR, IC31 TPS3705-33D, IC32 SN74LVC2G02DCTR, IC33 74LVC1G125GW.125, IC34 TPA6205A1DGN, IC4 LTC3260EMSE#PBF, IC5 TL072D, IC6 TL072D, IC7 LTC2050HVCS8#PBF, IC8 MCP23S17-E/SS, IC9 REF5025AIDG4, J1 BS-244DSM-R, J2 1-726388-2, J3 BS-244DSM-G, J4 BS-244DSM-B, J5 BS-244DSM-R, J6 BS-244DSM-B, J7 693072010801, Q1 IRFR5305, Q10 MMBT5401, Q11 MMBT5551, Q12 MMBT5551, Q13 IRLL2705PBF, Q14 IRFR48ZPBF, Q15 IRLML2246TRPBF, Q16 2N7002, Q17 MMBT5551, Q18 MMBT5401, Q19 MMBT5551, Q2 MMBT5401, Q20 MMBT5551, Q21 BTA26-600, Q22 BTA26-600, Q23 IRLL2705PBF, Q24 2N7002, Q25 2N7002, Q26 IRLML2246TRPBF, Q27 IRLML2246TRPBF, Q28 IRLML2246TRPBF, Q29 IRLML2246TRPBF, Q3 2N7002, Q30 2N7002, Q31 IRLML2246TRPBF, Q32 2N7002, Q33 2N7002, Q34 2N7002, Q4 IRFP250N, Q5 BC857C, Q6 BCP56-16.115, Q7 IRFR5305, Q8 BCP56-16.115, Q9 MMBT5401, SW1 A101SYCQ04, SW2 PEC12R-4225F-S0024, SW3 1301.9316, X1 39-30-1039, X10 826629-5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

Commit message: #64, #65
Parts:
- removed IC11: ADG465SOT-23, EEZ_Lib1:ADG465SOT-23
- removed LED: n.c., EEZ_Lib1:LEDHSMH-C170
- removed R1: n.c., rcl:R-EU_R0805
- removed R78: 1K, rcl:R-EU_R0805
- added R78A, R78B: 470R, rcl:R-EU_R0805
- added ZD18: SLVU2.8-TP, EEZ_Lib1:SLVU2.8
- C57: value 10u -> 4u7
- C62: value n.c. -> 10n
- D10, D13, D16, D2, D21, D3, D4, D5, D6, D7, D8, D9: device diode:DIODE-SOD323-W -> EEZ_Lib1:DIODESOD323R
- JP1, JP2, JP3, JP4: value 0R-JUMPA -> JP3-CUT; device jump-0r-smd:0R-JUMPA -> EEZ_Lib1:JP3-CUT
- R179: value 0R75? -> 0R75
- R65, R65B: device EEZ_Lib1:R-EU_4WIRE2512 -> rcl:R-EU_R2512
Connections:
- removed net N$78: LED.A, R1.1
- removed net N$9: IC11.VS, IC12.S1
- new net N$104: R78A.1, R78B.2
- net !INT: now also JP3.COM; no longer JP3-0R.2
- net !PS_DRDY: now also JP3.NC; no longer JP3-0R.3
- net +3V3: now also JP4.NO; no longer JP4-0R.3
- net +5V: now also JP4.NC; no longer JP4-0R.1
- net AUX_USET_IN: now also R78A.2; no longer R78.2
- net DC_OUT: no longer R1.2
- net GCOM: now also JP2.COM; no longer JP2-0R.2
- net GND: now also JP2.NO, ZD18.A; no longer JP2-0R.3, LED.C
- net INT_EXP: now also JP3.NO; no longer JP3-0R.1
- net MODE: now also JP1.COM; no longer JP1-0R.2
- net N$102: now also JP4.COM; no longer JP4-0R.2
- net N$12: now also IC12.S1, R78B.1, ZD18.C; no longer IC11.VD, R78.1
- net N$16: now also JP2.NC; no longer JP2-0R.1
- net N$200: no longer R65.1S, R65B.1S
- net N$70: no longer R65.2S, R65B.2S
- net SGND: now also JP1.NO; no longer JP1-0R.1
- net SYNC: now also JP1.NC; no longer JP1-0R.3
- net V+: no longer IC11.VDD
- net V-: no longer IC11.VSS
Other:
- note added: "+16.5 V"
- note added: "+16.75 V"
- note added: "-11.5 V"
- note added: "-9.7 V"
- note added: "DP values for Vout = +20 V"
- moved on the sheet: C62, X2-11
