File: Consolidated/KiCad/EEZ PSU consolidated r5B13a.kicad_pcb (KiCad board)
At the start: 2 copper layers, 337 x 150 mm, 534 parts, among them IC1 LTC3864EMSE#PBF, IC10 DAC8552IDGKTG4, IC12 TS5A9411DCKT, IC13 ADS1120IPWR, IC14 LP339D, IC15 TPD4E002DRL, IC16 TPD2E001DZDR, IC17 ADUM3160BRWZ, IC18 TLC5925IDBQR, IC19 Si8641EC-B-IS1, IC2 LP2951SO8, IC20 SI8651EC-B-IS1, IC21 SI8651EC-B-IS1, IC22 LD1117ADT33TR, IC23 Si8641EC-B-IS1, IC24 PCA21125T/Q900/1,1, IC25 AT25256B-SSHL-B, IC26 W5500, IC27 BC857BS, IC28 TLC555, IC29 SN74LVC08APWR, IC3 TL783CKTTR, IC30 SN74LV1T34DBVR, IC31 TPS3705-33D, IC32 SN74LVC2G02DCTR, IC33 74LVC1G125GW.125, IC34 TPA6205A1DGN, IC4 LTC3260EMSE#PBF, IC5 TL072D, IC6 TL072D, IC7 LTC2050HVCS8#PBF, IC8 MCP23S17-E/SS, IC9 REF5025AIDG4, J1 BS-244DSM-R, J2 1-726388-2, J3 BS-244DSM-G, J4 BS-244DSM-B, J5 BS-244DSM-R, J6 BS-244DSM-B, J7 693072010801, Q1 IRFR5305, Q10 MMBT5401, Q11 MMBT5551, Q12 MMBT5551, Q13 IRLL2705PBF, Q14 IRFR48ZPBF, Q15 IRLML2246TRPBF, Q16 2N7002, Q17 MMBT5551, Q18 MMBT5401, Q19 MMBT5551, Q2 MMBT5401, Q20 MMBT5551, Q21 BTA26-600, Q22 BTA26-600, Q23 IRLL2705PBF, Q24 2N7002, Q25 2N7002, Q26 IRLML2246TRPBF, Q27 IRLML2246TRPBF, Q28 IRLML2246TRPBF, Q29 IRLML2246TRPBF, Q3 2N7002, Q30 2N7002, Q31 IRLML2246TRPBF, Q32 2N7002, Q33 2N7002, Q34 2N7002, Q4 IRFP250N, Q5 BC857C, Q6 BCP56-16.115, Q7 IRFR5305, Q8 BCP56-16.115, Q9 MMBT5401, SW1 A101SYCQ04, SW2 PEC12R-4225F-S0024, SW3 1301.9316, X1 39-30-1039, X10 826629-5, X11 2411-01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

Commit message: Modified Kicad PCB Files
Parts:
- removed SH1: Pgnd to Pout- short, EEZ PSU consolidated r5B13a:SHORT_NOHOLE
- removed SH2: Sgnd to Pgnd short, EEZ PSU consolidated r5B13a:SHORT_NOHOLE
- added C156: 1u, EEZ PSU consolidated r5B13a:C0805, F.Cu at (132.0, 175.6)
- added C156: 1u, EEZ PSU consolidated r5B13a:C0805, F.Cu at (128.0, 175.6)
- added C156: 1u, EEZ PSU consolidated r5B13a:C0805, F.Cu at (166.9, 173.6)
- added C156: 1u, EEZ PSU consolidated r5B13a:C0805, F.Cu at (169.9, 172.6)
- added C156: 1u, EEZ PSU consolidated r5B13a:C0805, B.Cu at (311.6, 159.0)
- added HCPL-181: Relay_DPDT_Schrack-RT2-FormC_RM5mm, Relays_ThroughHole:Relay_DPDT_Schrack-RT2-FormC_RM5mm, F.Cu at (66.8, 145.4)
- added K_PAR: Relay_DPDT_Schrack-RT2-FormC_RM5mm, Relays_ThroughHole:Relay_DPDT_Schrack-RT2-FormC_RM5mm, F.Cu at (136.2, 133.6)
- added K_SER: Relay_DPDT_Schrack-RT2-FormC_RM5mm, Relays_ThroughHole:Relay_DPDT_Schrack-RT2-FormC_RM5mm, F.Cu at (160.7, 156.3)
- added R65: 0R030, EEZ PSU consolidated r5B13a:R2512, F.Cu at (35.3, 101.3)
- added R65A: 0R030, EEZ PSU consolidated r5B13a:R_2512-4WIRE, F.Cu at (35.3, 97.5)
- added R78A1: 470R, EEZ PSU consolidated r5B13a:C0805, F.Cu at (19.1, 56.8)
- added R78B1: 470R, EEZ PSU consolidated r5B13a:C0805, F.Cu at (23.0, 56.8)
- added REF**: Pin_Header_Straight_2x18_Pitch2.54mm, Pin_Headers:Pin_Header_Straight_2x18_Pitch2.54mm, F.Cu at (229.7, 108.6)
- added REF**: Pin_Header_Straight_1x08_Pitch2.54mm, Pin_Headers:Pin_Header_Straight_1x08_Pitch2.54mm, F.Cu at (257.7, 156.9)
- added REF**: Pin_Header_Straight_1x08_Pitch2.54mm, Pin_Headers:Pin_Header_Straight_1x08_Pitch2.54mm, F.Cu at (234.8, 156.9)
- added REF**: Pin_Header_Straight_1x08_Pitch2.54mm, Pin_Headers:Pin_Header_Straight_1x08_Pitch2.54mm, F.Cu at (284.6, 108.6)
- added REF**: Pin_Header_Straight_1x08_Pitch2.54mm, Pin_Headers:Pin_Header_Straight_1x08_Pitch2.54mm, F.Cu at (262.8, 108.6)
- added REF**: Pin_Header_Straight_1x08_Pitch2.54mm, Pin_Headers:Pin_Header_Straight_1x08_Pitch2.54mm, F.Cu at (239.9, 108.6)
- added REF**: Pin_Header_Straight_1x06_Pitch2.54mm, Pin_Headers:Pin_Header_Straight_1x06_Pitch2.54mm, F.Cu at (280.5, 156.9)
- added REF**: Pin_Header_Straight_2x03_Pitch2.54mm, Pin_Headers:Pin_Header_Straight_2x03_Pitch2.54mm, F.Cu at (260.2, 128.9)
- moved X15 0.13 mm to (129.3, 127.7)
Connections:
- C11 pad 2: POUT- -> GND
- C12 pad 2: POUT- -> GND
- C13 pad 2: POUT- -> GND
- R65 pad 1: POUT- -> GND
Routing:
- net GND: track 399.7 -> 528.1 mm, vias 390 -> 401
- net POUT-: track 93.9 -> 0.00 mm, vias 12 -> 0
- net OUT+: track 222.5 -> 256.4 mm
- net VSS: track 9.47 -> 0.00 mm
- net OUT-: track 119.8 -> 128.2 mm
- net 0V: track 64.3 -> 71.1 mm
- net (no net): track 0.00 -> 6.13 mm, vias 0 -> 1
- net Net-(C26-Pad2): track 0.00 -> 5.49 mm
- net /Isolators, Arduino/~CH1_DAC: track 35.1 -> 40.5 mm
- net Net-(C26-Pad1): track 1.02 -> 6.00 mm
- net /Reset, load temp, digital input/AUX1_USET_IN: track 34.1 -> 39.0 mm
- net Net-(K_S1-Pad3): track 30.4 -> 34.9 mm
- net Net-(IC14-Pad13): track 3.90 -> 7.82 mm
- net /Binding posts relays, LED driver/OUT2-: track 26.4 -> 22.6 mm
- net /Isolators, Arduino/CH1_SCLK: track 36.3 -> 40.1 mm
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- added copper zone on B.Cu, net EARTH
- removed copper zone on B.Cu, net POUT-
- removed copper zone on F.Cu, net POUT-
Other:
- rule pad_to_mask_clearance: 0.2 -> 0.05

Commit message: Modified PCB file
My repairs left a trace dangling where it shouldn't have, corrected.
Parts:
- removed the C156 at (128.0, 175.6)
- removed the C156 at (166.9, 173.6)
- removed the C156 at (311.6, 159.0)
- removed HCPL-181, K_PAR, K_SER: Relay_DPDT_Schrack-RT2-FormC_RM5mm, Relays_ThroughHole:Relay_DPDT_Schrack-RT2-FormC_RM5mm
- removed REF**: Pin_Header_Straight_2x18_Pitch2.54mm, Pin_Headers:Pin_Header_Straight_2x18_Pitch2.54mm
- removed REF** (x5): Pin_Header_Straight_1x08_Pitch2.54mm, Pin_Headers:Pin_Header_Straight_1x08_Pitch2.54mm
- removed REF**: Pin_Header_Straight_1x06_Pitch2.54mm, Pin_Headers:Pin_Header_Straight_1x06_Pitch2.54mm
- removed REF**: Pin_Header_Straight_2x03_Pitch2.54mm, Pin_Headers:Pin_Header_Straight_2x03_Pitch2.54mm
- added K_DOUT1: RT424005, EEZ PSU consolidated r5B13a:RT-C_016A5_ROUND, F.Cu at (78.1, 149.2)
- added K_PAR1: RT424005, EEZ PSU consolidated r5B13a:RT-C_016A5_ROUND, F.Cu at (136.2, 133.6)
- added K_SER1: RT424005, EEZ PSU consolidated r5B13a:RT-C_016A5_ROUND, F.Cu at (160.9, 156.3)
- added LED_PWR1: HSMD-C170, EEZ PSU consolidated r5B13a:LED_0805, B.Cu at (311.5, 158.9)
- added LED_SP1: HSMH-C170, EEZ PSU consolidated r5B13a:LED_HSMH-C170, B.Cu at (149.0, 162.0)
- added MCU1: Arduino Due, EEZ PSU consolidated r5B13a:ARDUINO+ICSP_MIRROR, F.Cu at (326.3, 106.1)
- added R136A1: 1R, EEZ PSU consolidated r5B13a:R0805, F.Cu at (166.2, 175.5)
- added R140A1: 1R, EEZ PSU consolidated r5B13a:R0805, F.Cu at (128.0, 175.6)
- R78A1, R78B1: footprint EEZ PSU consolidated r5B13a:C0805 -> EEZ PSU consolidated r5B13a:R0805
- moved C34 4.94 mm to (38.7, 59.7)
- moved R40 4.94 mm to (44.1, 59.7)
- moved R113 4.12 mm to (64.5, 173.8)
- moved C104A1 2.92 mm to (170.2, 175.5), turned to 180 degrees
- moved R57 2.47 mm to (49.1, 61.8)
- moved R44 2.04 mm to (38.7, 61.8)
- moved R43 2.04 mm to (44.1, 61.8)
- moved R32 1.97 mm to (38.7, 63.9)
- moved C40 1.97 mm to (49.1, 63.9), turned to 180 degrees
- moved C36 1.96 mm to (44.1, 63.9)
- moved R112 1.39 mm to (62.5, 173.8), turned to 270 degrees
- moved C126 0.84 mm to (238.5, 175.3)
- moved R148 0.77 mm to (228.9, 176.2)
- moved R147 0.69 mm to (228.9, 174.3)
- moved C125 0.58 mm to (240.2, 175.3)
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- renumbered C156 to C104A1, C156 to C109A1, R65A to R65A1, R65 to R65B1
Connections:
- C104A1 pad 1: (no net) -> /Binding posts relays, LED driver/OUT1+
- C104A1 pad 2: /Binding posts relays, LED driver/OUT1+ -> Net-(C104A1-Pad2)
- C109A1 pad 1: (no net) -> /Binding posts relays, LED driver/OUT2+
- C109A1 pad 2: /Binding posts relays, LED driver/OUT2+ -> Net-(C109A1-Pad2)
- C11 pad 2: GND -> POUT-
- C12 pad 2: GND -> POUT-
- C13 pad 2: GND -> POUT-
- C15 pad 2: GND -> POUT-
- R65 pad 1: GND -> POUT-
- R65A1 pad 1: Net-(Q14-Pad3) -> POUT-
- R65A1 pad 1S: Net-(R63-Pad1) -> Net-(R65A1-Pad1S)
- R65A1 pad 2: GND -> Net-(Q14-Pad3)
- R65A1 pad 2S: Net-(R65A1-Pad1S) -> Net-(R63-Pad1)
- R65B1 pad 1: GND -> POUT-
- R78A1 pad 1: /Digital control, voltage reference/AUX_USET_IN -> Net-(R78A1-Pad1)
- R78A1 pad 2: (no net) -> /Digital control, voltage reference/AUX_USET_IN
- R78B1 pad 1: (no net) -> Net-(C62-Pad2)
- R78B1 pad 2: Net-(C62-Pad2) -> Net-(R78A1-Pad1)
Routing:
- net GND: track 528.1 -> 436.4 mm, vias 401 -> 392
- net POUT-: track 0.00 -> 83.5 mm, vias 0 -> 12
- net DC_OUT: track 112.3 -> 95.7 mm
- net /Binding posts relays, LED driver/OUT1+: track 16.7 -> 25.1 mm
- net OUT+: track 256.4 -> 264.2 mm
- net (no net): track 6.13 -> 0.00 mm, vias 1 -> 0
- net Net-(K_S1-Pad3): track 34.9 -> 30.4 mm
- net OUT-: track 128.2 -> 132.5 mm
- net /AC soft-start, +5V power/AUX_PWR_SSTART: track 33.0 -> 37.1 mm
- net Net-(IC5-Pad5): track 19.3 -> 15.3 mm, vias 2 -> 0
- net /Binding posts relays, LED driver/OUT1-: track 49.5 -> 53.4 mm
- net +5V: track 969.6 -> 972.6 mm
- net Net-(OK2-Pad4): track 21.9 -> 24.1 mm
- net Net-(C104A1-Pad2): track 0.00 -> 2.10 mm
- net Net-(C109A1-Pad2): track 0.00 -> 2.04 mm
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- added copper zone on F.Cu, net Net-(K_PAR1-Pad12A)
- added copper zone on B.Cu, net Net-(K_PAR1-Pad12B)
- added copper zone on B.Cu, net Net-(K_SER1-Pad14A)
- added copper zone on F.Cu, net POUT-
- removed copper zone on F.Cu, net Net-(K_PAR-Pad12A)
- removed copper zone on B.Cu, net Net-(K_PAR-Pad12B)
- removed copper zone on B.Cu, net Net-(K_SER-Pad14A)
Other:
- net class Default: via_dia 0.8 -> 1; via_drill 0.4 -> 0.6
- net class Mains added: clearance 1.5, trace_width 0.25, via_dia 0.8, via_drill 0.4
- board text added: "!INT! 8"
- board text added: "+5V 10"
- board text added: "+5V 8"
- board text added: "+Sense 22"
- board text added: "+Vout 24"
- board text added: "+Vout 26"
- board text added: "-Sense 21"
- board text added: "-Vout 18"
- board text added: "-Vout 20"
- board text added: "1"
- board text added: "1 Fan+ (Red)"
- board text added: "1 Gnd"
- board text added: "1 MOSI"
- board text added: "10"
- board text added: "11 AUX_USET"
- board text added: "13 TEMP_NTC"
- board text added: "15 MCU_VCC"
- board text added: "17 Vout-"
- board text added: "18 Vout-"
- board text added: "19 Vout-"
- board text added: "2"
- board text added: "2 Fan- (Black)"
- board text added: "20 Vout-"
- board text added: "21 Sense-"
- board text added: "23"
- board text added: "23 Vout+"
- board text added: "24 Vout+"
- board text added: "25"
- board text added: "25 Vout +"
- board text added: "26"
- board text added: "26 Vout+"
- board text added: "27"
- board text added: "29"
- board text added: "3"
- board text added: "3 CS_EXP"
- board text added: "3 PWR_DIRECT"
- board text added: "3 Sense (Yellow)"
- board text added: "5"
- board text added: "5 !RESET!"
- board text added: "5 FAN_SENSE"
- board text added: "7 DOUT2"
- board text added: "7 Dout2"
- board text added: "7 SCLK"
- board text added: "8"
- board text added: "9"
- board text added: "9 Gnd"
- board text added: "9 MISO"
- board text added: "A1"
- board text added: "A2"
- board text added: "CH1+"
- board text added: "CH1-"
- board text added: "CH2+"
- board text added: "CH2-"
- board text added: "CS_ADC 6"
- board text added: "CS_DAC 4"
- board text added: "D"
- board text added: "EARTH"
- board text added: "FAN_PWM 6"
- board text added: "G"
- board text added: "GND"
- board text added: "Gnd 10"
- board text added: "Gnd 12"
- board text added: "Gnd 14"
- board text added: "Gnd 16"
- board text added: "Gnd 2"
- board text added: "NC"
- board text added: "PWR_SSTART 4"
- board text added: "S"
- board text added: "Standby"
- board text added: "Vdd 2"
- board text added: "X16"
- board text removed: "10 +5V"
- board text removed: "18 -Vout"
- board text removed: "2 Gnd"
- board text removed: "20 -Vout"
- board text removed: "24 +Vout"
- board text removed: "26 +Vout"
- board text removed: "4 PWR_SSTART"
- board text removed: "6 FAN_PWM"
- board text removed: "8 +5V"
- board text removed: "DOUT2 7"
- board text removed: "Dout2 7"
- board text removed: "FAN_SENSE 5"
- board text removed: "Fan+ (Red) 1"
- board text removed: "Fan- (Black) 2"
- board text removed: "Gnd 1"
- board text removed: "Gnd 9"
- board text removed: "PWR_DIRECT 3"
- board text removed: "Sense (Yellow) 3"
- board text removed: "Sense- 21"
